File: packages/scoring-circuit/pcb/scoring-prototype-board.kicad_sch (KiCad schematic)
At the start: 36 parts

Commit message: refactor(scoring-circuit): remove retired prototype architecture
Parts:
- removed V5 (x4): V5, symbol Custom:rail_up
- added V5 (x4): V5, symbol Custom:rail_up
Connections:
- net at C_V5_BULK.1, C_V5_BYPASS.1: now also V5.1
- net at J_DISPLAY.1 (V5): now also V5.1
- net at J_BUZZER.1 (V5): now also V5.1
Changed lines of the file:
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@@
     (instances
       (project ""
-        (path "/eee25254-a44a-4b13-b51d-3b4898075f6b"
+        (path "/9fc84f56-b1b9-44d4-ad87-6d632362281d"
           (reference "J_CONTROLLER_LEFT")
           (unit 1)
@@
     (instances
       (project ""
-        (path "/eee25254-a44a-4b13-b51d-3b4898075f6b"
+        (path "/9fc84f56-b1b9-44d4-ad87-6d632362281d"
           (reference "J_CONTROLLER_RIGHT")
           (unit 1)
@@
     (instances
       (project ""
-        (path "/eee25254-a44a-4b13-b51d-3b4898075f6b"
+        (path "/9fc84f56-b1b9-44d4-ad87-6d632362281d"
           (reference "J_WEAPON_LEFT")
           (unit 1)
@@
     (instances
       (project ""
-        (path "/eee25254-a44a-4b13-b51d-3b4898075f6b"
+        (path "/9fc84f56-b1b9-44d4-ad87-6d632362281d"
           (reference "J_WEAPON_RIGHT")
           (unit 1)
@@
     (instances
       (project ""
-        (path "/eee25254-a44a-4b13-b51d-3b4898075f6b"
+        (path "/9fc84f56-b1b9-44d4-ad87-6d632362281d"
           (reference "J_PISTE")
           (unit 1)
@@
     (instances
       (project ""
-        (path "/eee25254-a44a-4b13-b51d-3b4898075f6b"
+        (path "/9fc84f56-b1b9-44d4-ad87-6d632362281d"
           (reference "J_POWER_INPUT")
           (unit 1)
@@
     (instances
       (project ""
-        (path "/eee25254-a44a-4b13-b51d-3b4898075f6b"
+        (path "/9fc84f56-b1b9-44d4-ad87-6d632362281d"
           (reference "U_ETHERNET")
           (unit 1)
@@
     (instances
       (project ""
-        (path "/eee25254-a44a-4b13-b51d-3b4898075f6b"
+        (path "/9fc84f56-b1b9-44d4-ad87-6d632362281d"
           (reference "R_ETH_CS_PULLUP")
           (unit 1)
@@
     (instances
       (project ""
-        (path "/eee25254-a44a-4b13-b51d-3b4898075f6b"
+        (path "/9fc84f56-b1b9-44d4-ad87-6d632362281d"
           (reference "R_LEFT_A_DRIVE")
           (unit 1)
@@
     (instances
       (project ""
-        (path "/eee25254-a44a-4b13-b51d-3b4898075f6b"
+        (path "/9fc84f56-b1b9-44d4-ad87-6d632362281d"
           (reference "R_LEFT_B_DRIVE")
           (unit 1)
@@
     (instances
       (project ""
-        (path "/eee25254-a44a-4b13-b51d-3b4898075f6b"
+        (path "/9fc84f56-b1b9-44d4-ad87-6d632362281d"
           (reference "R_LEFT_B_SENSE")
           (unit 1)
@@
     (instances
       (project ""
-        (path "/eee25254-a44a-4b13-b51d-3b4898075f6b"
+        (path "/9fc84f56-b1b9-44d4-ad87-6d632362281d"
           (reference "R_LEFT_C_DRIVE")
           (unit 1)
@@
     (instances
       (project ""
-        (path "/eee25254-a44a-4b13-b51d-3b4898075f6b"
+        (path "/9fc84f56-b1b9-44d4-ad87-6d632362281d"
           (reference "R_LEFT_C_SENSE")
           (unit 1)
@@
     (instances
       (project ""
-        (path "/eee25254-a44a-4b13-b51d-3b4898075f6b"
+        (path "/9fc84f56-b1b9-44d4-ad87-6d632362281d"
           (reference "R_RIGHT_A_DRIVE")
           (unit 1)
@@
     (instances
       (project ""
-        (path "/eee25254-a44a-4b13-b51d-3b4898075f6b"
+        (path "/9fc84f56-b1b9-44d4-ad87-6d632362281d"
           (reference "R_RIGHT_B_DRIVE")
           (unit 1)
@@
     (instances
       (project ""
-        (path "/eee25254-a44a-4b13-b51d-3b4898075f6b"
+        (path "/9fc84f56-b1b9-44d4-ad87-6d632362281d"
           (reference "R_RIGHT_B_SENSE")
           (unit 1)
@@
     (instances
       (project ""
-        (path "/eee25254-a44a-4b13-b51d-3b4898075f6b"
+        (path "/9fc84f56-b1b9-44d4-ad87-6d632362281d"
           (reference "R_RIGHT_C_DRIVE")
           (unit 1)
@@
     (instances
       (project ""
-        (path "/eee25254-a44a-4b13-b51d-3b4898075f6b"
+        (path "/9fc84f56-b1b9-44d4-ad87-6d632362281d"
           (reference "R_RIGHT_C_SENSE")
           (unit 1)
@@
     (instances
       (project ""
-        (path "/eee25254-a44a-4b13-b51d-3b4898075f6b"
+        (path "/9fc84f56-b1b9-44d4-ad87-6d632362281d"
           (reference "R_PISTE_DRIVE")
           (unit 1)
@@
     (instances
       (project ""
-        (path "/eee25254-a44a-4b13-b51d-3b4898075f6b"
+        (path "/9fc84f56-b1b9-44d4-ad87-6d632362281d"
           (reference "R_PISTE_SENSE")
           (unit 1)
@@
     (instances
       (project ""
-        (path "/eee25254-a44a-4b13-b51d-3b4898075f6b"
+        (path "/9fc84f56-b1b9-44d4-ad87-6d632362281d"
           (reference "U_IR_RECEIVER")
           (unit 1)
@@
     (instances
       (project ""
-        (path "/eee25254-a44a-4b13-b51d-3b4898075f6b"
+        (path "/9fc84f56-b1b9-44d4-ad87-6d632362281d"
           (reference "R_IR_SUPPLY")
           (unit 1)
@@
     (instances
       (project ""
-        (path "/eee25254-a44a-4b13-b51d-3b4898075f6b"
+        (path "/9fc84f56-b1b9-44d4-ad87-6d632362281d"
           (reference "C_IR_SUPPLY")
           (unit 1)
@@
     (instances
       (project ""
-        (path "/eee25254-a44a-4b13-b51d-3b4898075f6b"
+        (path "/9fc84f56-b1b9-44d4-ad87-6d632362281d"
           (reference "R_IR_PULLUP")
           (unit 1)
@@
     (instances
       (project ""
-        (path "/eee25254-a44a-4b13-b51d-3b4898075f6b"
+        (path "/9fc84f56-b1b9-44d4-ad87-6d632362281d"
           (reference "J_DISPLAY")
           (unit 1)
@@
     (instances
       (project ""
-        (path "/eee25254-a44a-4b13-b51d-3b4898075f6b"
+        (path "/9fc84f56-b1b9-44d4-ad87-6d632362281d"
           (reference "R_DISPLAY_DATA")
           (unit 1)
@@
     (instances
       (project ""
-        (path "/eee25254-a44a-4b13-b51d-3b4898075f6b"
+        (path "/9fc84f56-b1b9-44d4-ad87-6d632362281d"
           (reference "J_BUZZER")
           (unit 1)
@@
     (instances
       (project ""
-        (path "/eee25254-a44a-4b13-b51d-3b4898075f6b"
+        (path "/9fc84f56-b1b9-44d4-ad87-6d632362281d"
           (reference "Q_BUZZER")
           (unit 1)
@@
     (instances
       (project ""
-        (path "/eee25254-a44a-4b13-b51d-3b4898075f6b"
+        (path "/9fc84f56-b1b9-44d4-ad87-6d632362281d"
           (reference "R_BUZZER_GATE")
           (unit 1)
@@
     (instances
       (project ""
-        (path "/eee25254-a44a-4b13-b51d-3b4898075f6b"
+        (path "/9fc84f56-b1b9-44d4-ad87-6d632362281d"
           (reference "R_BUZZER_GATE_PULLDOWN")
           (unit 1)
@@
     (instances
       (project ""
-        (path "/eee25254-a44a-4b13-b51d-3b4898075f6b"
+        (path "/9fc84f56-b1b9-44d4-ad87-6d632362281d"
           (reference "C_V5_BULK")
           (unit 1)
@@
     (instances
       (project ""
-        (path "/eee25254-a44a-4b13-b51d-3b4898075f6b"
+        (path "/9fc84f56-b1b9-44d4-ad87-6d632362281d"
           (reference "C_V5_BYPASS")
           (unit 1)
@@
     (instances
       (project ""
-        (path "/eee25254-a44a-4b13-b51d-3b4898075f6b"
+        (path "/9fc84f56-b1b9-44d4-ad87-6d632362281d"
           (reference "V5")
           (unit 1)
@@
     (instances
       (project ""
-        (path "/eee25254-a44a-4b13-b51d-3b4898075f6b"
+        (path "/9fc84f56-b1b9-44d4-ad87-6d632362281d"
           (reference "V5")
           (unit 1)
@@
     (instances
       (project ""
-        (path "/eee25254-a44a-4b13-b51d-3b4898075f6b"
+        (path "/9fc84f56-b1b9-44d4-ad87-6d632362281d"
           (reference "V5")
           (unit 1)
@@
     (instances
       (project ""
-        (path "/eee25254-a44a-4b13-b51d-3b4898075f6b"
+        (path "/9fc84f56-b1b9-44d4-ad87-6d632362281d"
           (reference "V5")
           (unit 1)

Commit message: feat(scoring-circuit): add usb-c prototype power
Parts:
- removed J_POWER_INPUT: J_POWER_INPUT, symbol Connector_Generic:Conn_01x2
- removed V5 (x4): V5, symbol Custom:rail_up
- added U_USB_C_PD: 5991, symbol Device:U_5991
- added U_V5_REGULATOR: D36V50F5, symbol Device:U_D36V50F5
- added V5 (x3): V5, symbol Custom:rail_up
Connections:
- net APP_GND: now also U_V5_REGULATOR.3 (GND_OUT_1), U_V5_REGULATOR.4 (GND_OUT_2)
- net at J_BUZZER.1 (V5): now also V5.1
- net at C_V5_BULK.1, C_V5_BYPASS.1: now also V5.1
- net V5: now reaches J_DISPLAY.1 (V5)
- new net: U_USB_C_PD.1 (PD_20V), U_V5_REGULATOR.11 (EN), U_V5_REGULATOR.7 (VIN_1), U_V5_REGULATOR.8 (VIN_2)
- new net: U_V5_REGULATOR.1 (VOUT_1), U_V5_REGULATOR.2 (VOUT_2), V5.1
- new net U_V5_REGULATOR_GND_IN_1: U_USB_C_PD.2 (APP_GND), U_V5_REGULATOR.5 (GND_IN_1), U_V5_REGULATOR.6 (GND_IN_2)

Commit message: feat(scoring-circuit): add scoring indicators
Parts:
- removed V5 (x3): V5, symbol Custom:rail_up
- added LED_LEFT_RED: WP7113ID, symbol Device:led_up
- added LED_RIGHT_GREEN: WP7113GD, symbol Device:led_up
- added R_LEFT_RED_LED, R_RIGHT_GREEN_LED: 330Ω, symbol Device:boxresistor_right
- added V5 (x5): V5, symbol Custom:rail_up
Connections:
- net APP_GND: now also LED_LEFT_RED.1, LED_RIGHT_GREEN.1
- net at C_V5_BULK.1, C_V5_BYPASS.1: now also V5.1
- net at J_BUZZER.1 (V5): now also V5.1
- net at U_V5_REGULATOR.1 (VOUT_1), U_V5_REGULATOR.2 (VOUT_2): now also V5.1
- net J_CONTROLLER_RIGHT_GPIO42: now reaches J_CONTROLLER_RIGHT.6 (GPIO42)
- net J_CONTROLLER_RIGHT_GPIO42: now also R_LEFT_RED_LED.1
- net J_CONTROLLER_RIGHT_GPIO41: now reaches J_CONTROLLER_RIGHT.7 (GPIO41)
- net J_CONTROLLER_RIGHT_GPIO41: now also R_RIGHT_GREEN_LED.1
- net V5: no longer names the net of J_DISPLAY.1 (V5)
- net V5: now also V5.1
- new net: LED_LEFT_RED.2, R_LEFT_RED_LED.2
- new net: LED_RIGHT_GREEN.2, R_RIGHT_GREEN_LED.2

Commit message: feat(scoring-circuit): add prototype sounder
Parts:
- removed J_BUZZER: J_BUZZER, symbol Connector_Generic:Conn_01x2
- removed R_BUZZER_GATE_PULLDOWN: 100kΩ, symbol Device:boxresistor_up
- removed V5 (x5): V5, symbol Custom:rail_up
- added BZ_SCORING: PS1240P02BT, symbol Device:U_PS1240P02BT
- added R_BUZZER_GATE_PULLDOWN: 100kΩ, symbol Device:boxresistor_down
- added V5 (x4): V5, symbol Custom:rail_up
Connections:
- net APP_3V3: now also BZ_SCORING.1 (POSITIVE)
- net APP_GND: now also R_BUZZER_GATE_PULLDOWN.2
- net at Q_BUZZER.3 (DRAIN): now also BZ_SCORING.2 (SWITCHED_GROUND)
- net at C_V5_BULK.1, C_V5_BYPASS.1: now also V5.1
- net at J_DISPLAY.1 (V5): now also V5.1
- net at U_V5_REGULATOR.1 (VOUT_1), U_V5_REGULATOR.2 (VOUT_2): now also V5.1
- net Q_BUZZER_GATE: no longer names the net of Q_BUZZER.1 (GATE), R_BUZZER_GATE.2
- net Q_BUZZER_GATE: now also R_BUZZER_GATE_PULLDOWN.1

Commit message: feat(scoring-circuit): add repeater outputs
Parts:
- removed V5 (x4): V5, symbol Custom:rail_up
- added C_FPA_DRIVER_BYPASS: 100nF, symbol Device:capacitor_right
- added J_FPA_REPEATER_1, J_FPA_REPEATER_2: 182-009-113R161, symbol Device:U_182-009-113R161
- added U_FPA_DRIVER: AM26LV31EIPWR, symbol Device:U_AM26LV31EIPWR
- added V5 (x2): V5, symbol Custom:rail_up
Connections:
- net APP_3V3: now also C_FPA_DRIVER_BYPASS.1, U_FPA_DRIVER.16 (APP_3V3), U_FPA_DRIVER.4 (ENABLE_HIGH)
- net APP_GND: now also C_FPA_DRIVER_BYPASS.2, J_FPA_REPEATER_1.6 (APP_GND_6), J_FPA_REPEATER_1.7 (APP_GND_7), J_FPA_REPEATER_2.6 (APP_GND_6), J_FPA_REPEATER_2.7 (APP_GND_7), U_FPA_DRIVER.12 (ENABLE_LOW), U_FPA_DRIVER.15 (DRIVER_4_INPUT), U_FPA_DRIVER.8 (APP_GND), U_FPA_DRIVER.9 (DRIVER_3_INPUT)
- net at C_V5_BULK.1, C_V5_BYPASS.1: now also V5.1
- net V5: now reaches J_DISPLAY.1 (V5)
- net FPA_TX: now reaches J_CONTROLLER_RIGHT.2 (GPIO43_UART_TX)
- net FPA_TX: now also U_FPA_DRIVER.1 (DRIVER_1_INPUT), U_FPA_DRIVER.7 (DRIVER_2_INPUT)
- net at U_V5_REGULATOR.1 (VOUT_1), U_V5_REGULATOR.2 (VOUT_2): now also V5.1
- new net: J_FPA_REPEATER_1.4 (TX_POS), U_FPA_DRIVER.2 (DRIVER_1_POSITIVE)
- new net U_FPA_DRIVER_DRIVER_1_NEGATIVE: J_FPA_REPEATER_1.3 (TX_NEG), U_FPA_DRIVER.3 (DRIVER_1_NEGATIVE)
- new net U_FPA_DRIVER_DRIVER_2_NEGATIVE: J_FPA_REPEATER_2.3 (TX_NEG), U_FPA_DRIVER.5 (DRIVER_2_NEGATIVE)
- new net U_FPA_DRIVER_DRIVER_2_POSITIVE: J_FPA_REPEATER_2.4 (TX_POS), U_FPA_DRIVER.6 (DRIVER_2_POSITIVE)

Commit message: feat(scoring-circuit): add FA-05 outputs and scoring lamps
Parts:
- removed C_FPA_DRIVER_BYPASS: 100nF, symbol Device:capacitor_right
- removed J_FPA_REPEATER_1, J_FPA_REPEATER_2: 182-009-113R161, symbol Device:U_182-009-113R161
- removed U_FPA_DRIVER: AM26LV31EIPWR, symbol Device:U_AM26LV31EIPWR
- removed U_USB_C_PD: 5991, symbol Device:U_5991
- removed V5 (x2): V5, symbol Custom:rail_up
- added D_FAVERO_DATA_1, D_FAVERO_DATA_2: 1N4004-E3/54, symbol Device:U_1N4004-E3_54
- added J_FAVERO_DATA_1, J_FAVERO_DATA_2: 5520250-2, symbol Device:U_5520250-2
- added LED_LEFT_WHITE, LED_RIGHT_WHITE: WP7113QWC/D, symbol Device:led_down
- added Q_LEFT_WHITE_LED, Q_RIGHT_WHITE_LED: BSS138-7-F, symbol Device:U_BSS138-7-F
- added R_FAVERO_DATA_1_BASE, R_FAVERO_DATA_2_BASE: 680kΩ, symbol Device:boxresistor_right
- added R_FAVERO_DATA_1_INPUT, R_FAVERO_DATA_2_INPUT: 330Ω, symbol Device:boxresistor_up
- added R_FAVERO_DATA_1_LOOP, R_FAVERO_DATA_2_LOOP: 82Ω, symbol Device:boxresistor_right
- added R_LEFT_WHITE_LED, R_RIGHT_WHITE_LED: 330Ω, symbol Device:boxresistor_down
- added R_LEFT_WHITE_LED_PULLDOWN, R_RIGHT_WHITE_LED_PULLDOWN: 100kΩ, symbol Device:boxresistor_up
- added U_FAVERO_DATA_1, U_FAVERO_DATA_2: 4N32M, symbol Device:U_4N32M
- added U_USB_C_PD: 5807, symbol Device:U_5807
- added V5 (x4): V5, symbol Custom:rail_up
Connections:
- net APP_GND: now also Q_LEFT_WHITE_LED.2 (SOURCE), Q_RIGHT_WHITE_LED.2 (SOURCE), R_LEFT_WHITE_LED_PULLDOWN.2, R_RIGHT_WHITE_LED_PULLDOWN.2, U_FAVERO_DATA_1.2 (LED_CATHODE), U_FAVERO_DATA_2.2 (LED_CATHODE); no longer U_V5_REGULATOR.4 (GND_OUT_2)
- net U_V5_REGULATOR_GND_IN_1: now also U_USB_C_PD.2 (APP_GND); no longer U_V5_REGULATOR.6 (GND_IN_2)
- net at U_V5_REGULATOR.11 (EN), U_V5_REGULATOR.7 (VIN_1): now also U_USB_C_PD.1 (PD_VOUT); no longer U_V5_REGULATOR.8 (VIN_2)
- net at U_V5_REGULATOR.1 (VOUT_1): now also V5.1; no longer U_V5_REGULATOR.2 (VOUT_2)
- net at C_V5_BULK.1, C_V5_BYPASS.1: now also V5.1
- net LED_RIGHT_WHITE_DRIVE: now reaches J_CONTROLLER_RIGHT.17 (GPIO47)
- net LED_RIGHT_WHITE_DRIVE: now also Q_RIGHT_WHITE_LED.1 (GATE), R_RIGHT_WHITE_LED_PULLDOWN.1
- net LED_LEFT_WHITE_DRIVE: now reaches J_CONTROLLER_RIGHT.8 (GPIO40)
- net LED_LEFT_WHITE_DRIVE: now also Q_LEFT_WHITE_LED.1 (GATE), R_LEFT_WHITE_LED_PULLDOWN.1
- net FPA_TX renamed FAVERO_DATA_TX
- net FAVERO_DATA_TX: now also R_FAVERO_DATA_1_INPUT.1, R_FAVERO_DATA_2_INPUT.1
- new net: R_LEFT_WHITE_LED.1, V5.1
- new net: LED_LEFT_WHITE.1, Q_LEFT_WHITE_LED.3 (DRAIN)
- new net: J_FAVERO_DATA_1.3 (DATA_A), U_FAVERO_DATA_1.4 (EMITTER)
- new net: R_FAVERO_DATA_1_BASE.1, U_FAVERO_DATA_1.6 (BASE)
- new net: J_FAVERO_DATA_2.2 (OUTER_A), R_FAVERO_DATA_2_LOOP.2
- new net: LED_LEFT_WHITE.2, R_LEFT_WHITE_LED.2
- new net: J_FAVERO_DATA_1.2 (OUTER_A), R_FAVERO_DATA_1_LOOP.2
- new net: LED_RIGHT_WHITE.1, Q_RIGHT_WHITE_LED.3 (DRAIN)
- new net: LED_RIGHT_WHITE.2, R_RIGHT_WHITE_LED.2
- new net: R_RIGHT_WHITE_LED.1, V5.1
- new net: J_FAVERO_DATA_2.3 (DATA_A), U_FAVERO_DATA_2.4 (EMITTER)
- new net: D_FAVERO_DATA_2.2 (ANODE), J_FAVERO_DATA_2.4 (DATA_B)
- new net: J_FAVERO_DATA_2.5 (OUTER_B), R_FAVERO_DATA_2_BASE.2
- new net: R_FAVERO_DATA_2_BASE.1, U_FAVERO_DATA_2.6 (BASE)
- new net: J_FAVERO_DATA_1.5 (OUTER_B), R_FAVERO_DATA_1_BASE.2
- new net: D_FAVERO_DATA_1.2 (ANODE), J_FAVERO_DATA_1.4 (DATA_B)
- new net U_FAVERO_DATA_1_COLLECTOR: D_FAVERO_DATA_1.1 (CATHODE), R_FAVERO_DATA_1_LOOP.1, U_FAVERO_DATA_1.5 (COLLECTOR)
- new net U_FAVERO_DATA_1_LED_ANODE: R_FAVERO_DATA_1_INPUT.2, U_FAVERO_DATA_1.1 (LED_ANODE)
- new net U_FAVERO_DATA_2_COLLECTOR: D_FAVERO_DATA_2.1 (CATHODE), R_FAVERO_DATA_2_LOOP.1, U_FAVERO_DATA_2.5 (COLLECTOR)
- new net U_FAVERO_DATA_2_LED_ANODE: R_FAVERO_DATA_2_INPUT.2, U_FAVERO_DATA_2.1 (LED_ANODE)

Commit message: fix(scoring-circuit): attach board component models
Parts:
- removed V5 (x4): V5, symbol Custom:rail_up
- added V5 (x4): V5, symbol Custom:rail_up
Connections:
- net at R_LEFT_WHITE_LED.1: now also V5.1
- net at U_V5_REGULATOR.1 (VOUT_1): now also V5.1
- net at C_V5_BULK.1, C_V5_BYPASS.1: now also V5.1
- net at R_RIGHT_WHITE_LED.1: now also V5.1

Commit message: fix(scoring-circuit): remove unused prototype circuitry
Parts:
- removed R_ETH_CS_PULLUP: 10kΩ, symbol Device:boxresistor_right
- removed R_IR_PULLUP: 10kΩ, symbol Device:boxresistor_up
- removed V5 (x4): V5, symbol Custom:rail_up
- added V5 (x5): V5, symbol Custom:rail_up
Connections:
- net U_V5_REGULATOR_GND_IN_1 is gone; now on an unnamed net: U_USB_C_PD.2 (APP_GND), U_V5_REGULATOR.5 (GND_IN_1)
- net APP_GND: now also U_V5_REGULATOR.4 (GND_OUT_2)
- net at U_USB_C_PD.1 (PD_VOUT), U_V5_REGULATOR.7 (VIN_1): now also U_V5_REGULATOR.8 (VIN_2); no longer U_V5_REGULATOR.11 (EN)
- net at R_LEFT_WHITE_LED.1: now also V5.1
- net at C_V5_BULK.1, C_V5_BYPASS.1: now also V5.1
- net at U_V5_REGULATOR.1 (VOUT_1): now also U_V5_REGULATOR.2 (VOUT_2), V5.1
- net at R_RIGHT_WHITE_LED.1: now also V5.1
- net V5: no longer names the net of J_DISPLAY.1 (V5)
- net V5: now also V5.1
