File: packages/scoring-circuit/pcb/scoring-prototype-board.kicad_sch (KiCad schematic)
At the start: 60 parts

Commit message: feat(scoring-circuit): align prototype display and conductors
Parts:
- removed J_DISPLAY: J_DISPLAY, symbol Connector_Generic:Conn_01x3
- removed R_DISPLAY_DATA: 330Ω, symbol Device:boxresistor_up
- removed R_LEFT_A_DRIVE, R_RIGHT_A_DRIVE: 33Ω, symbol Device:boxresistor_right
- removed R_LEFT_B_DRIVE, R_LEFT_C_DRIVE, R_PISTE_DRIVE, R_RIGHT_B_DRIVE, R_RIGHT_C_DRIVE: 470Ω, symbol Device:boxresistor_right
- removed R_LEFT_B_SENSE, R_LEFT_C_SENSE, R_PISTE_SENSE, R_RIGHT_B_SENSE, R_RIGHT_C_SENSE: 1kΩ, symbol Device:boxresistor_right
- removed V5 (x5): V5, symbol Custom:rail_up
- added J_HUB75_DATA: TST-108-02-G-D, symbol Device:U_TST-108-02-G-D
- added J_HUB75_POWER: 645004114822, symbol Device:U_645004114822
- added R_LEFT_A_SERIES, R_RIGHT_A_SERIES: 33Ω, symbol Device:boxresistor_right
- added R_LEFT_B_SERIES, R_LEFT_C_SERIES, R_PISTE_SERIES, R_RIGHT_B_SERIES, R_RIGHT_C_SERIES: 470Ω, symbol Device:boxresistor_right
- added V5 (x6): V5, symbol Custom:rail_up
Connections:
- net DISPLAY_DATA is gone; now on net APP_SPI_MOSI: J_CONTROLLER_RIGHT.18 (GPIO21)
- net APP_GND: now also J_HUB75_DATA.16 (GND_3), J_HUB75_DATA.4 (GND_1), J_HUB75_DATA.8 (GND_2); no longer U_IR_RECEIVER.2 (GND)
- net APP_SPI_MISO: now also J_CONTROLLER_RIGHT.13 (GPIO35)
- net BUZZER_DRIVE: now also J_CONTROLLER_RIGHT.16 (GPIO48); no longer J_CONTROLLER_RIGHT.9 (GPIO39)
- net ETH_CS_N: now also J_CONTROLLER_RIGHT.12 (GPIO36)
- net ETH_INT_N: now also J_CONTROLLER_RIGHT.11 (GPIO37)
- net IR_RX: now also J_CONTROLLER_RIGHT.10 (GPIO38_RGB)
- net LED_LEFT_WHITE_DRIVE: now also J_CONTROLLER_RIGHT.17 (GPIO47); no longer J_CONTROLLER_RIGHT.8 (GPIO40)
- net LED_RIGHT_WHITE_DRIVE: now also J_CONTROLLER_RIGHT.19 (GPIO20_USB_D_PLUS); no longer J_CONTROLLER_RIGHT.17 (GPIO47)
- net LEFT_A: now also R_LEFT_A_SERIES.2
- net LEFT_B: now also R_LEFT_B_SERIES.2
- net LEFT_C: now also R_LEFT_C_SERIES.2
- net PISTE: now also R_PISTE_SERIES.2
- net RIGHT_A: now also J_WEAPON_RIGHT.1 (RIGHT_A), R_RIGHT_A_SERIES.2
- net RIGHT_B: now also J_WEAPON_RIGHT.2 (RIGHT_B), R_RIGHT_B_SERIES.2
- net RIGHT_C: now also J_WEAPON_RIGHT.3 (RIGHT_C), R_RIGHT_C_SERIES.2
- net at R_LEFT_WHITE_LED.1: now also V5.1
- net at R_RIGHT_WHITE_LED.1: now also V5.1
- net at C_V5_BULK.1, C_V5_BYPASS.1: now also V5.1
- net at U_V5_REGULATOR.1 (VOUT_1), U_V5_REGULATOR.2 (VOUT_2): now also V5.1
- net at J_CONTROLLER_RIGHT.20 (GPIO19_USB_D_MINUS): now also R_RIGHT_GREEN_LED.1
- net J_CONTROLLER_RIGHT_GPIO41 renamed HUB75_CLK
- net HUB75_CLK: now also J_HUB75_DATA.13 (CLK); no longer R_RIGHT_GREEN_LED.1
- net J_CONTROLLER_RIGHT_GPIO42 renamed HUB75_D
- net HUB75_D: now also J_HUB75_DATA.12 (D); no longer R_LEFT_RED_LED.1
- net SENSE_LEFT_B renamed SCORING_PISTE
- net SCORING_PISTE: now also R_PISTE_SERIES.1
- net SENSE_LEFT_C renamed HUB75_OE
- net HUB75_OE: now also J_HUB75_DATA.15 (OE)
- new net: J_HUB75_POWER.3 (GND_1), J_HUB75_POWER.4 (GND_2), U_IR_RECEIVER.2 (GND)
- new net: J_HUB75_POWER.1 (V5_1), J_HUB75_POWER.2 (V5_2), V5.1
- new net HUB75_A: J_HUB75_DATA.9 (A)
- new net HUB75_B: J_HUB75_DATA.10 (B)
- new net HUB75_B1: J_HUB75_DATA.3 (B1)
- new net HUB75_B2: J_HUB75_DATA.7 (B2)
- new net HUB75_C: J_HUB75_DATA.11 (C)
- new net HUB75_G1: J_HUB75_DATA.2 (G1)
- new net HUB75_G2: J_HUB75_DATA.6 (G2)
- new net HUB75_LAT: J_CONTROLLER_RIGHT.8 (GPIO40), J_HUB75_DATA.14 (LAT)
- new net HUB75_R1: J_HUB75_DATA.1 (R1)
- new net HUB75_R2: J_HUB75_DATA.5 (R2)
- new net J_CONTROLLER_RIGHT_GPIO39: J_CONTROLLER_RIGHT.9 (GPIO39), R_LEFT_RED_LED.1
- new net SCORING_LEFT_A: R_LEFT_A_SERIES.1
- new net SCORING_LEFT_B: R_LEFT_B_SERIES.1
- new net SCORING_LEFT_C: R_LEFT_C_SERIES.1
- new net SCORING_RIGHT_A: R_RIGHT_A_SERIES.1
- new net SCORING_RIGHT_B: R_RIGHT_B_SERIES.1
- new net SCORING_RIGHT_C: R_RIGHT_C_SERIES.1

Commit message: feat(scoring-circuit): remove redundant scoring lamps
Parts:
- removed LED_LEFT_RED: WP7113ID, symbol Device:led_up
- removed LED_LEFT_WHITE, LED_RIGHT_WHITE: WP7113QWC/D, symbol Device:led_down
- removed LED_RIGHT_GREEN: WP7113GD, symbol Device:led_up
- removed Q_LEFT_WHITE_LED, Q_RIGHT_WHITE_LED: BSS138-7-F, symbol Device:U_BSS138-7-F
- removed R_LEFT_RED_LED, R_RIGHT_GREEN_LED: 330Ω, symbol Device:boxresistor_right
- removed R_LEFT_WHITE_LED, R_RIGHT_WHITE_LED: 330Ω, symbol Device:boxresistor_down
- removed R_LEFT_WHITE_LED_PULLDOWN, R_RIGHT_WHITE_LED_PULLDOWN: 100kΩ, symbol Device:boxresistor_up
- removed V5 (x6): V5, symbol Custom:rail_up
- added V5 (x4): V5, symbol Custom:rail_up
Connections:
- net APP_GND: now also J_HUB75_POWER.3 (GND_1), J_HUB75_POWER.4 (GND_2), U_IR_RECEIVER.2 (GND)
- net at U_V5_REGULATOR.1 (VOUT_1), U_V5_REGULATOR.2 (VOUT_2): now also V5.1
- net at C_V5_BULK.1, C_V5_BYPASS.1: now also V5.1
- net at J_HUB75_POWER.1 (V5_1), J_HUB75_POWER.2 (V5_2): now also V5.1
- net J_CONTROLLER_RIGHT_GPIO39: no longer names the net of J_CONTROLLER_RIGHT.9 (GPIO39)
- net LED_LEFT_WHITE_DRIVE: no longer names the net of J_CONTROLLER_RIGHT.17 (GPIO47)
- net LED_RIGHT_WHITE_DRIVE: no longer names the net of J_CONTROLLER_RIGHT.19 (GPIO20_USB_D_PLUS)

Commit message: feat(scoring-circuit): price the prototype order BOM
Parts:
- removed V5 (x4): V5, symbol Custom:rail_up
- added V5 (x4): V5, symbol Custom:rail_up
Connections:
- net APP_SPI_MISO: now also J_CONTROLLER_RIGHT.19 (GPIO20_USB_D_PLUS); no longer J_CONTROLLER_RIGHT.13 (GPIO35)
- net ETH_CS_N: now also J_CONTROLLER_RIGHT.17 (GPIO47); no longer J_CONTROLLER_RIGHT.12 (GPIO36)
- net ETH_INT_N: now also J_CONTROLLER_RIGHT.9 (GPIO39); no longer J_CONTROLLER_RIGHT.11 (GPIO37)
- net at U_V5_REGULATOR.1 (VOUT_1), U_V5_REGULATOR.2 (VOUT_2): now also V5.1
- net at C_V5_BULK.1, C_V5_BYPASS.1: now also V5.1
- net at J_HUB75_POWER.1 (V5_1), J_HUB75_POWER.2 (V5_2): now also V5.1

Commit message: fix(scoring-circuit): space the ESP32 assembly
Parts:
- removed V5 (x4): V5, symbol Custom:rail_up
- added V5 (x4): V5, symbol Custom:rail_up
Connections:
- net at U_V5_REGULATOR.1 (VOUT_1), U_V5_REGULATOR.2 (VOUT_2): now also V5.1
- net at J_HUB75_POWER.1 (V5_1), J_HUB75_POWER.2 (V5_2): now also V5.1
- net at C_V5_BULK.1, C_V5_BYPASS.1: now also V5.1
Changed lines of the file:
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@@
     (instances
       (project ""
-        (path "/92ddeb7f-a395-446c-b72f-0c4e7e4411e3"
+        (path "/eb320af9-d762-4703-a09f-589b08a6cdf5"
           (reference "J_CONTROLLER_LEFT")
           (unit 1)
@@
     (instances
       (project ""
-        (path "/92ddeb7f-a395-446c-b72f-0c4e7e4411e3"
+        (path "/eb320af9-d762-4703-a09f-589b08a6cdf5"
           (reference "J_CONTROLLER_RIGHT")
           (unit 1)
@@
     (instances
       (project ""
-        (path "/92ddeb7f-a395-446c-b72f-0c4e7e4411e3"
+        (path "/eb320af9-d762-4703-a09f-589b08a6cdf5"
           (reference "J_WEAPON_LEFT")
           (unit 1)
@@
     (instances
       (project ""
-        (path "/92ddeb7f-a395-446c-b72f-0c4e7e4411e3"
+        (path "/eb320af9-d762-4703-a09f-589b08a6cdf5"
           (reference "J_WEAPON_RIGHT")
           (unit 1)
@@
     (instances
       (project ""
-        (path "/92ddeb7f-a395-446c-b72f-0c4e7e4411e3"
+        (path "/eb320af9-d762-4703-a09f-589b08a6cdf5"
           (reference "J_PISTE")
           (unit 1)
@@
     (instances
       (project ""
-        (path "/92ddeb7f-a395-446c-b72f-0c4e7e4411e3"
+        (path "/eb320af9-d762-4703-a09f-589b08a6cdf5"
           (reference "U_USB_C_PD")
           (unit 1)
@@
     (instances
       (project ""
-        (path "/92ddeb7f-a395-446c-b72f-0c4e7e4411e3"
+        (path "/eb320af9-d762-4703-a09f-589b08a6cdf5"
           (reference "U_V5_REGULATOR")
           (unit 1)
@@
     (instances
       (project ""
-        (path "/92ddeb7f-a395-446c-b72f-0c4e7e4411e3"
+        (path "/eb320af9-d762-4703-a09f-589b08a6cdf5"
           (reference "U_ETHERNET")
           (unit 1)
@@
     (instances
       (project ""
-        (path "/92ddeb7f-a395-446c-b72f-0c4e7e4411e3"
+        (path "/eb320af9-d762-4703-a09f-589b08a6cdf5"
           (reference "R_LEFT_A_SERIES")
           (unit 1)
@@
     (instances
       (project ""
-        (path "/92ddeb7f-a395-446c-b72f-0c4e7e4411e3"
+        (path "/eb320af9-d762-4703-a09f-589b08a6cdf5"
           (reference "R_LEFT_B_SERIES")
           (unit 1)
@@
     (instances
       (project ""
-        (path "/92ddeb7f-a395-446c-b72f-0c4e7e4411e3"
+        (path "/eb320af9-d762-4703-a09f-589b08a6cdf5"
           (reference "R_LEFT_C_SERIES")
           (unit 1)
@@
     (instances
       (project ""
-        (path "/92ddeb7f-a395-446c-b72f-0c4e7e4411e3"
+        (path "/eb320af9-d762-4703-a09f-589b08a6cdf5"
           (reference "R_RIGHT_A_SERIES")
           (unit 1)
@@
     (instances
       (project ""
-        (path "/92ddeb7f-a395-446c-b72f-0c4e7e4411e3"
+        (path "/eb320af9-d762-4703-a09f-589b08a6cdf5"
           (reference "R_RIGHT_B_SERIES")
           (unit 1)
@@
     (instances
       (project ""
-        (path "/92ddeb7f-a395-446c-b72f-0c4e7e4411e3"
+        (path "/eb320af9-d762-4703-a09f-589b08a6cdf5"
           (reference "R_RIGHT_C_SERIES")
           (unit 1)
@@
     (instances
       (project ""
-        (path "/92ddeb7f-a395-446c-b72f-0c4e7e4411e3"
+        (path "/eb320af9-d762-4703-a09f-589b08a6cdf5"
           (reference "R_PISTE_SERIES")
           (unit 1)
@@
     (instances
       (project ""
-        (path "/92ddeb7f-a395-446c-b72f-0c4e7e4411e3"
+        (path "/eb320af9-d762-4703-a09f-589b08a6cdf5"
           (reference "U_IR_RECEIVER")
           (unit 1)
@@
     (instances
       (project ""
-        (path "/92ddeb7f-a395-446c-b72f-0c4e7e4411e3"
+        (path "/eb320af9-d762-4703-a09f-589b08a6cdf5"
           (reference "R_IR_SUPPLY")
           (unit 1)
@@
     (instances
       (project ""
-        (path "/92ddeb7f-a395-446c-b72f-0c4e7e4411e3"
+        (path "/eb320af9-d762-4703-a09f-589b08a6cdf5"
           (reference "C_IR_SUPPLY")
           (unit 1)
@@
     (instances
       (project ""
-        (path "/92ddeb7f-a395-446c-b72f-0c4e7e4411e3"
+        (path "/eb320af9-d762-4703-a09f-589b08a6cdf5"
           (reference "J_HUB75_DATA")
           (unit 1)
@@
     (instances
       (project ""
-        (path "/92ddeb7f-a395-446c-b72f-0c4e7e4411e3"
+        (path "/eb320af9-d762-4703-a09f-589b08a6cdf5"
           (reference "J_HUB75_POWER")
           (unit 1)
@@
     (instances
       (project ""
-        (path "/92ddeb7f-a395-446c-b72f-0c4e7e4411e3"
+        (path "/eb320af9-d762-4703-a09f-589b08a6cdf5"
           (reference "BZ_SCORING")
           (unit 1)
@@
     (instances
       (project ""
-        (path "/92ddeb7f-a395-446c-b72f-0c4e7e4411e3"
+        (path "/eb320af9-d762-4703-a09f-589b08a6cdf5"
           (reference "Q_BUZZER")
           (unit 1)
@@
     (instances
       (project ""
-        (path "/92ddeb7f-a395-446c-b72f-0c4e7e4411e3"
+        (path "/eb320af9-d762-4703-a09f-589b08a6cdf5"
           (reference "R_BUZZER_GATE")
           (unit 1)
@@
     (instances
       (project ""
-        (path "/92ddeb7f-a395-446c-b72f-0c4e7e4411e3"
+        (path "/eb320af9-d762-4703-a09f-589b08a6cdf5"
           (reference "R_BUZZER_GATE_PULLDOWN")
           (unit 1)
@@
     (instances
       (project ""
-        (path "/92ddeb7f-a395-446c-b72f-0c4e7e4411e3"
+        (path "/eb320af9-d762-4703-a09f-589b08a6cdf5"
           (reference "C_V5_BULK")
           (unit 1)
@@
     (instances
       (project ""
-        (path "/92ddeb7f-a395-446c-b72f-0c4e7e4411e3"
+        (path "/eb320af9-d762-4703-a09f-589b08a6cdf5"
           (reference "C_V5_BYPASS")
           (unit 1)
@@
     (instances
       (project ""
-        (path "/92ddeb7f-a395-446c-b72f-0c4e7e4411e3"
+        (path "/eb320af9-d762-4703-a09f-589b08a6cdf5"
           (reference "J_FAVERO_DATA_1")
           (unit 1)
@@
     (instances
       (project ""
-        (path "/92ddeb7f-a395-446c-b72f-0c4e7e4411e3"
+        (path "/eb320af9-d762-4703-a09f-589b08a6cdf5"
           (reference "U_FAVERO_DATA_1")
           (unit 1)
@@
     (instances
       (project ""
-        (path "/92ddeb7f-a395-446c-b72f-0c4e7e4411e3"
+        (path "/eb320af9-d762-4703-a09f-589b08a6cdf5"
           (reference "R_FAVERO_DATA_1_INPUT")
           (unit 1)
@@
     (instances
       (project ""
-        (path "/92ddeb7f-a395-446c-b72f-0c4e7e4411e3"
+        (path "/eb320af9-d762-4703-a09f-589b08a6cdf5"
           (reference "R_FAVERO_DATA_1_LOOP")
           (unit 1)
@@
     (instances
       (project ""
-        (path "/92ddeb7f-a395-446c-b72f-0c4e7e4411e3"
+        (path "/eb320af9-d762-4703-a09f-589b08a6cdf5"
           (reference "R_FAVERO_DATA_1_BASE")
           (unit 1)
@@
     (instances
       (project ""
-        (path "/92ddeb7f-a395-446c-b72f-0c4e7e4411e3"
+        (path "/eb320af9-d762-4703-a09f-589b08a6cdf5"
           (reference "D_FAVERO_DATA_1")
           (unit 1)
@@
     (instances
       (project ""
-        (path "/92ddeb7f-a395-446c-b72f-0c4e7e4411e3"
+        (path "/eb320af9-d762-4703-a09f-589b08a6cdf5"
           (reference "J_FAVERO_DATA_2")
           (unit 1)
@@
     (instances
       (project ""
-        (path "/92ddeb7f-a395-446c-b72f-0c4e7e4411e3"
+        (path "/eb320af9-d762-4703-a09f-589b08a6cdf5"
           (reference "U_FAVERO_DATA_2")
           (unit 1)
@@
     (instances
       (project ""
-        (path "/92ddeb7f-a395-446c-b72f-0c4e7e4411e3"
+        (path "/eb320af9-d762-4703-a09f-589b08a6cdf5"
           (reference "R_FAVERO_DATA_2_INPUT")
           (unit 1)
@@
     (instances
       (project ""
-        (path "/92ddeb7f-a395-446c-b72f-0c4e7e4411e3"
+        (path "/eb320af9-d762-4703-a09f-589b08a6cdf5"
           (reference "R_FAVERO_DATA_2_LOOP")
           (unit 1)
@@
     (instances
       (project ""
-        (path "/92ddeb7f-a395-446c-b72f-0c4e7e4411e3"
+        (path "/eb320af9-d762-4703-a09f-589b08a6cdf5"
           (reference "R_FAVERO_DATA_2_BASE")
           (unit 1)
@@
     (instances
       (project ""
-        (path "/92ddeb7f-a395-446c-b72f-0c4e7e4411e3"
+        (path "/eb320af9-d762-4703-a09f-589b08a6cdf5"
           (reference "D_FAVERO_DATA_2")
           (unit 1)
@@
     (instances
       (project ""
-        (path "/92ddeb7f-a395-446c-b72f-0c4e7e4411e3"
+        (path "/eb320af9-d762-4703-a09f-589b08a6cdf5"
           (reference "V5")
           (unit 1)
@@
     (instances
       (project ""
-        (path "/92ddeb7f-a395-446c-b72f-0c4e7e4411e3"
+        (path "/eb320af9-d762-4703-a09f-589b08a6cdf5"
           (reference "V5")
           (unit 1)
@@
     (instances
       (project ""
-        (path "/92ddeb7f-a395-446c-b72f-0c4e7e4411e3"
+        (path "/eb320af9-d762-4703-a09f-589b08a6cdf5"
           (reference "V5")
           (unit 1)
@@
     (instances
       (project ""
-        (path "/92ddeb7f-a395-446c-b72f-0c4e7e4411e3"
+        (path "/eb320af9-d762-4703-a09f-589b08a6cdf5"
           (reference "V5")
           (unit 1)
