File: packages/scoring-circuit/pcb/scoring-prototype-board.kicad_sch (KiCad schematic)
At the start: 42 parts

Commit message: feat(scoring-circuit): validate prototype electronics with ngspice
Parts:
- removed V5 (x4): V5, symbol Custom:rail_up
- added V5 (x4): V5, symbol Custom:rail_up
- R_FAVERO_DATA_1_INPUT, R_FAVERO_DATA_2_INPUT: value 330Ω -> 82Ω
Connections:
- net at J_HUB75_POWER.1 (V5_1), J_HUB75_POWER.2 (V5_2): now also V5.1
- net at U_V5_REGULATOR.1 (VOUT_1), U_V5_REGULATOR.2 (VOUT_2): now also V5.1
- net at C_V5_BULK.1, C_V5_BYPASS.1: now also V5.1
Changed lines of the file:
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@@
     (instances
       (project ""
-        (path "/eb320af9-d762-4703-a09f-589b08a6cdf5"
+        (path "/8779ccd1-5db7-433f-9d16-b3e561d3270b"
           (reference "J_CONTROLLER_LEFT")
           (unit 1)
@@
     (instances
       (project ""
-        (path "/eb320af9-d762-4703-a09f-589b08a6cdf5"
+        (path "/8779ccd1-5db7-433f-9d16-b3e561d3270b"
           (reference "J_CONTROLLER_RIGHT")
           (unit 1)
@@
     (instances
       (project ""
-        (path "/eb320af9-d762-4703-a09f-589b08a6cdf5"
+        (path "/8779ccd1-5db7-433f-9d16-b3e561d3270b"
           (reference "J_WEAPON_LEFT")
           (unit 1)
@@
     (instances
       (project ""
-        (path "/eb320af9-d762-4703-a09f-589b08a6cdf5"
+        (path "/8779ccd1-5db7-433f-9d16-b3e561d3270b"
           (reference "J_WEAPON_RIGHT")
           (unit 1)
@@
     (instances
       (project ""
-        (path "/eb320af9-d762-4703-a09f-589b08a6cdf5"
+        (path "/8779ccd1-5db7-433f-9d16-b3e561d3270b"
           (reference "J_PISTE")
           (unit 1)
@@
     (instances
       (project ""
-        (path "/eb320af9-d762-4703-a09f-589b08a6cdf5"
+        (path "/8779ccd1-5db7-433f-9d16-b3e561d3270b"
           (reference "U_USB_C_PD")
           (unit 1)
@@
     (instances
       (project ""
-        (path "/eb320af9-d762-4703-a09f-589b08a6cdf5"
+        (path "/8779ccd1-5db7-433f-9d16-b3e561d3270b"
           (reference "U_V5_REGULATOR")
           (unit 1)
@@
     (instances
       (project ""
-        (path "/eb320af9-d762-4703-a09f-589b08a6cdf5"
+        (path "/8779ccd1-5db7-433f-9d16-b3e561d3270b"
           (reference "U_ETHERNET")
           (unit 1)
@@
     (instances
       (project ""
-        (path "/eb320af9-d762-4703-a09f-589b08a6cdf5"
+        (path "/8779ccd1-5db7-433f-9d16-b3e561d3270b"
           (reference "R_LEFT_A_SERIES")
           (unit 1)
@@
     (instances
       (project ""
-        (path "/eb320af9-d762-4703-a09f-589b08a6cdf5"
+        (path "/8779ccd1-5db7-433f-9d16-b3e561d3270b"
           (reference "R_LEFT_B_SERIES")
           (unit 1)
@@
     (instances
       (project ""
-        (path "/eb320af9-d762-4703-a09f-589b08a6cdf5"
+        (path "/8779ccd1-5db7-433f-9d16-b3e561d3270b"
           (reference "R_LEFT_C_SERIES")
           (unit 1)
@@
     (instances
       (project ""
-        (path "/eb320af9-d762-4703-a09f-589b08a6cdf5"
+        (path "/8779ccd1-5db7-433f-9d16-b3e561d3270b"
           (reference "R_RIGHT_A_SERIES")
           (unit 1)
@@
     (instances
       (project ""
-        (path "/eb320af9-d762-4703-a09f-589b08a6cdf5"
+        (path "/8779ccd1-5db7-433f-9d16-b3e561d3270b"
           (reference "R_RIGHT_B_SERIES")
           (unit 1)
@@
     (instances
       (project ""
-        (path "/eb320af9-d762-4703-a09f-589b08a6cdf5"
+        (path "/8779ccd1-5db7-433f-9d16-b3e561d3270b"
           (reference "R_RIGHT_C_SERIES")
           (unit 1)
@@
     (instances
       (project ""
-        (path "/eb320af9-d762-4703-a09f-589b08a6cdf5"
+        (path "/8779ccd1-5db7-433f-9d16-b3e561d3270b"
           (reference "R_PISTE_SERIES")
           (unit 1)
@@
     (instances
       (project ""
-        (path "/eb320af9-d762-4703-a09f-589b08a6cdf5"
+        (path "/8779ccd1-5db7-433f-9d16-b3e561d3270b"
           (reference "U_IR_RECEIVER")
           (unit 1)
@@
     (instances
       (project ""
-        (path "/eb320af9-d762-4703-a09f-589b08a6cdf5"
+        (path "/8779ccd1-5db7-433f-9d16-b3e561d3270b"
           (reference "R_IR_SUPPLY")
           (unit 1)
@@
     (instances
       (project ""
-        (path "/eb320af9-d762-4703-a09f-589b08a6cdf5"
+        (path "/8779ccd1-5db7-433f-9d16-b3e561d3270b"
           (reference "C_IR_SUPPLY")
           (unit 1)
@@
     (instances
       (project ""
-        (path "/eb320af9-d762-4703-a09f-589b08a6cdf5"
+        (path "/8779ccd1-5db7-433f-9d16-b3e561d3270b"
           (reference "J_HUB75_DATA")
           (unit 1)
@@
     (instances
       (project ""
-        (path "/eb320af9-d762-4703-a09f-589b08a6cdf5"
+        (path "/8779ccd1-5db7-433f-9d16-b3e561d3270b"
           (reference "J_HUB75_POWER")
           (unit 1)
@@
     (instances
       (project ""
-        (path "/eb320af9-d762-4703-a09f-589b08a6cdf5"
+        (path "/8779ccd1-5db7-433f-9d16-b3e561d3270b"
           (reference "BZ_SCORING")
           (unit 1)
@@
     (instances
       (project ""
-        (path "/eb320af9-d762-4703-a09f-589b08a6cdf5"
+        (path "/8779ccd1-5db7-433f-9d16-b3e561d3270b"
           (reference "Q_BUZZER")
           (unit 1)
@@
     (instances
       (project ""
-        (path "/eb320af9-d762-4703-a09f-589b08a6cdf5"
+        (path "/8779ccd1-5db7-433f-9d16-b3e561d3270b"
           (reference "R_BUZZER_GATE")
           (unit 1)
@@
     (instances
       (project ""
-        (path "/eb320af9-d762-4703-a09f-589b08a6cdf5"
+        (path "/8779ccd1-5db7-433f-9d16-b3e561d3270b"
           (reference "R_BUZZER_GATE_PULLDOWN")
           (unit 1)
@@
     (instances
       (project ""
-        (path "/eb320af9-d762-4703-a09f-589b08a6cdf5"
+        (path "/8779ccd1-5db7-433f-9d16-b3e561d3270b"
           (reference "C_V5_BULK")
           (unit 1)
@@
     (instances
       (project ""
-        (path "/eb320af9-d762-4703-a09f-589b08a6cdf5"
+        (path "/8779ccd1-5db7-433f-9d16-b3e561d3270b"
           (reference "C_V5_BYPASS")
           (unit 1)
@@
     (instances
       (project ""
-        (path "/eb320af9-d762-4703-a09f-589b08a6cdf5"
+        (path "/8779ccd1-5db7-433f-9d16-b3e561d3270b"
           (reference "J_FAVERO_DATA_1")
           (unit 1)
@@
     (instances
       (project ""
-        (path "/eb320af9-d762-4703-a09f-589b08a6cdf5"
+        (path "/8779ccd1-5db7-433f-9d16-b3e561d3270b"
           (reference "U_FAVERO_DATA_1")
           (unit 1)
@@
       )
     )
-    (property "Value" "330Ω"
+    (property "Value" "82Ω"
       (id 1)
       (at 432.2425 93.37499999999991 0)
@@
     (instances
       (project ""
-        (path "/eb320af9-d762-4703-a09f-589b08a6cdf5"
+        (path "/8779ccd1-5db7-433f-9d16-b3e561d3270b"
           (reference "R_FAVERO_DATA_1_INPUT")
           (unit 1)
@@
     (instances
       (project ""
-        (path "/eb320af9-d762-4703-a09f-589b08a6cdf5"
+        (path "/8779ccd1-5db7-433f-9d16-b3e561d3270b"
           (reference "R_FAVERO_DATA_1_LOOP")
           (unit 1)
@@
     (instances
       (project ""
-        (path "/eb320af9-d762-4703-a09f-589b08a6cdf5"
+        (path "/8779ccd1-5db7-433f-9d16-b3e561d3270b"
           (reference "R_FAVERO_DATA_1_BASE")
           (unit 1)
@@
     (instances
       (project ""
-        (path "/eb320af9-d762-4703-a09f-589b08a6cdf5"
+        (path "/8779ccd1-5db7-433f-9d16-b3e561d3270b"
           (reference "D_FAVERO_DATA_1")
           (unit 1)
@@
     (instances
       (project ""
-        (path "/eb320af9-d762-4703-a09f-589b08a6cdf5"
+        (path "/8779ccd1-5db7-433f-9d16-b3e561d3270b"
           (reference "J_FAVERO_DATA_2")
           (unit 1)
@@
     (instances
       (project ""
-        (path "/eb320af9-d762-4703-a09f-589b08a6cdf5"
+        (path "/8779ccd1-5db7-433f-9d16-b3e561d3270b"
           (reference "U_FAVERO_DATA_2")
           (unit 1)
@@
       )
     )
-    (property "Value" "330Ω"
+    (property "Value" "82Ω"
       (id 1)
       (at 432.2425 178.57499999999993 0)
@@
     (instances
       (project ""
-        (path "/eb320af9-d762-4703-a09f-589b08a6cdf5"
+        (path "/8779ccd1-5db7-433f-9d16-b3e561d3270b"
           (reference "R_FAVERO_DATA_2_INPUT")
           (unit 1)
@@
     (instances
       (project ""
-        (path "/eb320af9-d762-4703-a09f-589b08a6cdf5"
+        (path "/8779ccd1-5db7-433f-9d16-b3e561d3270b"
           (reference "R_FAVERO_DATA_2_LOOP")
           (unit 1)
@@
     (instances
       (project ""
-        (path "/eb320af9-d762-4703-a09f-589b08a6cdf5"
+        (path "/8779ccd1-5db7-433f-9d16-b3e561d3270b"
           (reference "R_FAVERO_DATA_2_BASE")
           (unit 1)
@@
     (instances
       (project ""
-        (path "/eb320af9-d762-4703-a09f-589b08a6cdf5"
+        (path "/8779ccd1-5db7-433f-9d16-b3e561d3270b"
           (reference "D_FAVERO_DATA_2")
           (unit 1)
@@
     (instances
       (project ""
-        (path "/eb320af9-d762-4703-a09f-589b08a6cdf5"
+        (path "/8779ccd1-5db7-433f-9d16-b3e561d3270b"
           (reference "V5")
           (unit 1)
@@
     (instances
       (project ""
-        (path "/eb320af9-d762-4703-a09f-589b08a6cdf5"
+        (path "/8779ccd1-5db7-433f-9d16-b3e561d3270b"
           (reference "V5")
           (unit 1)
@@
     (instances
       (project ""
-        (path "/eb320af9-d762-4703-a09f-589b08a6cdf5"
+        (path "/8779ccd1-5db7-433f-9d16-b3e561d3270b"
           (reference "V5")
           (unit 1)
@@
     (instances
       (project ""
-        (path "/eb320af9-d762-4703-a09f-589b08a6cdf5"
+        (path "/8779ccd1-5db7-433f-9d16-b3e561d3270b"
           (reference "V5")
           (unit 1)

Commit message: fix(scoring-circuit): align all prototype CAD models
Parts:
- removed V5 (x4): V5, symbol Custom:rail_up
- added V5 (x4): V5, symbol Custom:rail_up
Connections:
- net at C_V5_BULK.1, C_V5_BYPASS.1: now also V5.1
- net at J_HUB75_POWER.1 (V5_1), J_HUB75_POWER.2 (V5_2): now also V5.1
- net at U_V5_REGULATOR.1 (VOUT_1), U_V5_REGULATOR.2 (VOUT_2): now also V5.1
Changed lines of the file:
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@@
     (instances
       (project ""
-        (path "/8779ccd1-5db7-433f-9d16-b3e561d3270b"
+        (path "/37108faa-7298-4e6c-a552-10776871d6b1"
           (reference "J_CONTROLLER_LEFT")
           (unit 1)
@@
     (instances
       (project ""
-        (path "/8779ccd1-5db7-433f-9d16-b3e561d3270b"
+        (path "/37108faa-7298-4e6c-a552-10776871d6b1"
           (reference "J_CONTROLLER_RIGHT")
           (unit 1)
@@
     (instances
       (project ""
-        (path "/8779ccd1-5db7-433f-9d16-b3e561d3270b"
+        (path "/37108faa-7298-4e6c-a552-10776871d6b1"
           (reference "J_WEAPON_LEFT")
           (unit 1)
@@
     (instances
       (project ""
-        (path "/8779ccd1-5db7-433f-9d16-b3e561d3270b"
+        (path "/37108faa-7298-4e6c-a552-10776871d6b1"
           (reference "J_WEAPON_RIGHT")
           (unit 1)
@@
     (instances
       (project ""
-        (path "/8779ccd1-5db7-433f-9d16-b3e561d3270b"
+        (path "/37108faa-7298-4e6c-a552-10776871d6b1"
           (reference "J_PISTE")
           (unit 1)
@@
     (instances
       (project ""
-        (path "/8779ccd1-5db7-433f-9d16-b3e561d3270b"
+        (path "/37108faa-7298-4e6c-a552-10776871d6b1"
           (reference "U_USB_C_PD")
           (unit 1)
@@
     (instances
       (project ""
-        (path "/8779ccd1-5db7-433f-9d16-b3e561d3270b"
+        (path "/37108faa-7298-4e6c-a552-10776871d6b1"
           (reference "U_V5_REGULATOR")
           (unit 1)
@@
     (instances
       (project ""
-        (path "/8779ccd1-5db7-433f-9d16-b3e561d3270b"
+        (path "/37108faa-7298-4e6c-a552-10776871d6b1"
           (reference "U_ETHERNET")
           (unit 1)
@@
     (instances
       (project ""
-        (path "/8779ccd1-5db7-433f-9d16-b3e561d3270b"
+        (path "/37108faa-7298-4e6c-a552-10776871d6b1"
           (reference "R_LEFT_A_SERIES")
           (unit 1)
@@
     (instances
       (project ""
-        (path "/8779ccd1-5db7-433f-9d16-b3e561d3270b"
+        (path "/37108faa-7298-4e6c-a552-10776871d6b1"
           (reference "R_LEFT_B_SERIES")
           (unit 1)
@@
     (instances
       (project ""
-        (path "/8779ccd1-5db7-433f-9d16-b3e561d3270b"
+        (path "/37108faa-7298-4e6c-a552-10776871d6b1"
           (reference "R_LEFT_C_SERIES")
           (unit 1)
@@
     (instances
       (project ""
-        (path "/8779ccd1-5db7-433f-9d16-b3e561d3270b"
+        (path "/37108faa-7298-4e6c-a552-10776871d6b1"
           (reference "R_RIGHT_A_SERIES")
           (unit 1)
@@
     (instances
       (project ""
-        (path "/8779ccd1-5db7-433f-9d16-b3e561d3270b"
+        (path "/37108faa-7298-4e6c-a552-10776871d6b1"
           (reference "R_RIGHT_B_SERIES")
           (unit 1)
@@
     (instances
       (project ""
-        (path "/8779ccd1-5db7-433f-9d16-b3e561d3270b"
+        (path "/37108faa-7298-4e6c-a552-10776871d6b1"
           (reference "R_RIGHT_C_SERIES")
           (unit 1)
@@
     (instances
       (project ""
-        (path "/8779ccd1-5db7-433f-9d16-b3e561d3270b"
+        (path "/37108faa-7298-4e6c-a552-10776871d6b1"
           (reference "R_PISTE_SERIES")
           (unit 1)
@@
     (instances
       (project ""
-        (path "/8779ccd1-5db7-433f-9d16-b3e561d3270b"
+        (path "/37108faa-7298-4e6c-a552-10776871d6b1"
           (reference "U_IR_RECEIVER")
           (unit 1)
@@
     (instances
       (project ""
-        (path "/8779ccd1-5db7-433f-9d16-b3e561d3270b"
+        (path "/37108faa-7298-4e6c-a552-10776871d6b1"
           (reference "R_IR_SUPPLY")
           (unit 1)
@@
     (instances
       (project ""
-        (path "/8779ccd1-5db7-433f-9d16-b3e561d3270b"
+        (path "/37108faa-7298-4e6c-a552-10776871d6b1"
           (reference "C_IR_SUPPLY")
           (unit 1)
@@
     (instances
       (project ""
-        (path "/8779ccd1-5db7-433f-9d16-b3e561d3270b"
+        (path "/37108faa-7298-4e6c-a552-10776871d6b1"
           (reference "J_HUB75_DATA")
           (unit 1)
@@
     (instances
       (project ""
-        (path "/8779ccd1-5db7-433f-9d16-b3e561d3270b"
+        (path "/37108faa-7298-4e6c-a552-10776871d6b1"
           (reference "J_HUB75_POWER")
           (unit 1)
@@
     (instances
       (project ""
-        (path "/8779ccd1-5db7-433f-9d16-b3e561d3270b"
+        (path "/37108faa-7298-4e6c-a552-10776871d6b1"
           (reference "BZ_SCORING")
           (unit 1)
@@
     (instances
       (project ""
-        (path "/8779ccd1-5db7-433f-9d16-b3e561d3270b"
+        (path "/37108faa-7298-4e6c-a552-10776871d6b1"
           (reference "Q_BUZZER")
           (unit 1)
@@
     (instances
       (project ""
-        (path "/8779ccd1-5db7-433f-9d16-b3e561d3270b"
+        (path "/37108faa-7298-4e6c-a552-10776871d6b1"
           (reference "R_BUZZER_GATE")
           (unit 1)
@@
     (instances
       (project ""
-        (path "/8779ccd1-5db7-433f-9d16-b3e561d3270b"
+        (path "/37108faa-7298-4e6c-a552-10776871d6b1"
           (reference "R_BUZZER_GATE_PULLDOWN")
           (unit 1)
@@
     (instances
       (project ""
-        (path "/8779ccd1-5db7-433f-9d16-b3e561d3270b"
+        (path "/37108faa-7298-4e6c-a552-10776871d6b1"
           (reference "C_V5_BULK")
           (unit 1)
@@
     (instances
       (project ""
-        (path "/8779ccd1-5db7-433f-9d16-b3e561d3270b"
+        (path "/37108faa-7298-4e6c-a552-10776871d6b1"
           (reference "C_V5_BYPASS")
           (unit 1)
@@
     (instances
       (project ""
-        (path "/8779ccd1-5db7-433f-9d16-b3e561d3270b"
+        (path "/37108faa-7298-4e6c-a552-10776871d6b1"
           (reference "J_FAVERO_DATA_1")
           (unit 1)
@@
     (instances
       (project ""
-        (path "/8779ccd1-5db7-433f-9d16-b3e561d3270b"
+        (path "/37108faa-7298-4e6c-a552-10776871d6b1"
           (reference "U_FAVERO_DATA_1")
           (unit 1)
@@
     (instances
       (project ""
-        (path "/8779ccd1-5db7-433f-9d16-b3e561d3270b"
+        (path "/37108faa-7298-4e6c-a552-10776871d6b1"
           (reference "R_FAVERO_DATA_1_INPUT")
           (unit 1)
@@
     (instances
       (project ""
-        (path "/8779ccd1-5db7-433f-9d16-b3e561d3270b"
+        (path "/37108faa-7298-4e6c-a552-10776871d6b1"
           (reference "R_FAVERO_DATA_1_LOOP")
           (unit 1)
@@
     (instances
       (project ""
-        (path "/8779ccd1-5db7-433f-9d16-b3e561d3270b"
+        (path "/37108faa-7298-4e6c-a552-10776871d6b1"
           (reference "R_FAVERO_DATA_1_BASE")
           (unit 1)
@@
     (instances
       (project ""
-        (path "/8779ccd1-5db7-433f-9d16-b3e561d3270b"
+        (path "/37108faa-7298-4e6c-a552-10776871d6b1"
           (reference "D_FAVERO_DATA_1")
           (unit 1)
@@
     (instances
       (project ""
-        (path "/8779ccd1-5db7-433f-9d16-b3e561d3270b"
+        (path "/37108faa-7298-4e6c-a552-10776871d6b1"
           (reference "J_FAVERO_DATA_2")
           (unit 1)
@@
     (instances
       (project ""
-        (path "/8779ccd1-5db7-433f-9d16-b3e561d3270b"
+        (path "/37108faa-7298-4e6c-a552-10776871d6b1"
           (reference "U_FAVERO_DATA_2")
           (unit 1)
@@
     (instances
       (project ""
-        (path "/8779ccd1-5db7-433f-9d16-b3e561d3270b"
+        (path "/37108faa-7298-4e6c-a552-10776871d6b1"
           (reference "R_FAVERO_DATA_2_INPUT")
           (unit 1)
@@
     (instances
       (project ""
-        (path "/8779ccd1-5db7-433f-9d16-b3e561d3270b"
+        (path "/37108faa-7298-4e6c-a552-10776871d6b1"
           (reference "R_FAVERO_DATA_2_LOOP")
           (unit 1)
@@
     (instances
       (project ""
-        (path "/8779ccd1-5db7-433f-9d16-b3e561d3270b"
+        (path "/37108faa-7298-4e6c-a552-10776871d6b1"
           (reference "R_FAVERO_DATA_2_BASE")
           (unit 1)
@@
     (instances
       (project ""
-        (path "/8779ccd1-5db7-433f-9d16-b3e561d3270b"
+        (path "/37108faa-7298-4e6c-a552-10776871d6b1"
           (reference "D_FAVERO_DATA_2")
           (unit 1)
@@
     (instances
       (project ""
-        (path "/8779ccd1-5db7-433f-9d16-b3e561d3270b"
+        (path "/37108faa-7298-4e6c-a552-10776871d6b1"
           (reference "V5")
           (unit 1)
@@
     (instances
       (project ""
-        (path "/8779ccd1-5db7-433f-9d16-b3e561d3270b"
+        (path "/37108faa-7298-4e6c-a552-10776871d6b1"
           (reference "V5")
           (unit 1)
@@
     (instances
       (project ""
-        (path "/8779ccd1-5db7-433f-9d16-b3e561d3270b"
+        (path "/37108faa-7298-4e6c-a552-10776871d6b1"
           (reference "V5")
           (unit 1)
@@
     (instances
       (project ""
-        (path "/8779ccd1-5db7-433f-9d16-b3e561d3270b"
+        (path "/37108faa-7298-4e6c-a552-10776871d6b1"
           (reference "V5")
           (unit 1)
