File: packages/scoring-circuit/pcb/scoring-prototype-board.kicad_sch (KiCad schematic)
At the start: 42 parts

Commit message: fix(scoring-circuit): clear repeater support placement
Parts:
- removed V5 (x4): V5, symbol Custom:rail_up
- added V5 (x4): V5, symbol Custom:rail_up
Connections:
- net at J_HUB75_POWER.1 (V5_1), J_HUB75_POWER.2 (V5_2): now also V5.1
- net at U_V5_REGULATOR.1 (VOUT_1), U_V5_REGULATOR.2 (VOUT_2): now also V5.1
- net at C_V5_BULK.1, C_V5_BYPASS.1: now also V5.1
Changed lines of the file:
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@@
     (instances
       (project ""
-        (path "/2e0f7609-671f-4aa5-9de8-e48290b9d466"
+        (path "/253667d2-eebf-4ec3-a193-9fc7a8d1f262"
           (reference "J_CONTROLLER_LEFT")
           (unit 1)
@@
     (instances
       (project ""
-        (path "/2e0f7609-671f-4aa5-9de8-e48290b9d466"
+        (path "/253667d2-eebf-4ec3-a193-9fc7a8d1f262"
           (reference "J_CONTROLLER_RIGHT")
           (unit 1)
@@
     (instances
       (project ""
-        (path "/2e0f7609-671f-4aa5-9de8-e48290b9d466"
+        (path "/253667d2-eebf-4ec3-a193-9fc7a8d1f262"
           (reference "J_WEAPON_LEFT")
           (unit 1)
@@
     (instances
       (project ""
-        (path "/2e0f7609-671f-4aa5-9de8-e48290b9d466"
+        (path "/253667d2-eebf-4ec3-a193-9fc7a8d1f262"
           (reference "J_WEAPON_RIGHT")
           (unit 1)
@@
     (instances
       (project ""
-        (path "/2e0f7609-671f-4aa5-9de8-e48290b9d466"
+        (path "/253667d2-eebf-4ec3-a193-9fc7a8d1f262"
           (reference "J_PISTE")
           (unit 1)
@@
     (instances
       (project ""
-        (path "/2e0f7609-671f-4aa5-9de8-e48290b9d466"
+        (path "/253667d2-eebf-4ec3-a193-9fc7a8d1f262"
           (reference "U_USB_C_PD")
           (unit 1)
@@
     (instances
       (project ""
-        (path "/2e0f7609-671f-4aa5-9de8-e48290b9d466"
+        (path "/253667d2-eebf-4ec3-a193-9fc7a8d1f262"
           (reference "U_V5_REGULATOR")
           (unit 1)
@@
     (instances
       (project ""
-        (path "/2e0f7609-671f-4aa5-9de8-e48290b9d466"
+        (path "/253667d2-eebf-4ec3-a193-9fc7a8d1f262"
           (reference "U_ETHERNET")
           (unit 1)
@@
     (instances
       (project ""
-        (path "/2e0f7609-671f-4aa5-9de8-e48290b9d466"
+        (path "/253667d2-eebf-4ec3-a193-9fc7a8d1f262"
           (reference "R_LEFT_A_SERIES")
           (unit 1)
@@
     (instances
       (project ""
-        (path "/2e0f7609-671f-4aa5-9de8-e48290b9d466"
+        (path "/253667d2-eebf-4ec3-a193-9fc7a8d1f262"
           (reference "R_LEFT_B_SERIES")
           (unit 1)
@@
     (instances
       (project ""
-        (path "/2e0f7609-671f-4aa5-9de8-e48290b9d466"
+        (path "/253667d2-eebf-4ec3-a193-9fc7a8d1f262"
           (reference "R_LEFT_C_SERIES")
           (unit 1)
@@
     (instances
       (project ""
-        (path "/2e0f7609-671f-4aa5-9de8-e48290b9d466"
+        (path "/253667d2-eebf-4ec3-a193-9fc7a8d1f262"
           (reference "R_RIGHT_A_SERIES")
           (unit 1)
@@
     (instances
       (project ""
-        (path "/2e0f7609-671f-4aa5-9de8-e48290b9d466"
+        (path "/253667d2-eebf-4ec3-a193-9fc7a8d1f262"
           (reference "R_RIGHT_B_SERIES")
           (unit 1)
@@
     (instances
       (project ""
-        (path "/2e0f7609-671f-4aa5-9de8-e48290b9d466"
+        (path "/253667d2-eebf-4ec3-a193-9fc7a8d1f262"
           (reference "R_RIGHT_C_SERIES")
           (unit 1)
@@
     (instances
       (project ""
-        (path "/2e0f7609-671f-4aa5-9de8-e48290b9d466"
+        (path "/253667d2-eebf-4ec3-a193-9fc7a8d1f262"
           (reference "R_PISTE_SERIES")
           (unit 1)
@@
     (instances
       (project ""
-        (path "/2e0f7609-671f-4aa5-9de8-e48290b9d466"
+        (path "/253667d2-eebf-4ec3-a193-9fc7a8d1f262"
           (reference "U_IR_RECEIVER")
           (unit 1)
@@
     (instances
       (project ""
-        (path "/2e0f7609-671f-4aa5-9de8-e48290b9d466"
+        (path "/253667d2-eebf-4ec3-a193-9fc7a8d1f262"
           (reference "R_IR_SUPPLY")
           (unit 1)
@@
     (instances
       (project ""
-        (path "/2e0f7609-671f-4aa5-9de8-e48290b9d466"
+        (path "/253667d2-eebf-4ec3-a193-9fc7a8d1f262"
           (reference "C_IR_SUPPLY")
           (unit 1)
@@
     (instances
       (project ""
-        (path "/2e0f7609-671f-4aa5-9de8-e48290b9d466"
+        (path "/253667d2-eebf-4ec3-a193-9fc7a8d1f262"
           (reference "J_HUB75_DATA")
           (unit 1)
@@
     (instances
       (project ""
-        (path "/2e0f7609-671f-4aa5-9de8-e48290b9d466"
+        (path "/253667d2-eebf-4ec3-a193-9fc7a8d1f262"
           (reference "J_HUB75_POWER")
           (unit 1)
@@
     (instances
       (project ""
-        (path "/2e0f7609-671f-4aa5-9de8-e48290b9d466"
+        (path "/253667d2-eebf-4ec3-a193-9fc7a8d1f262"
           (reference "BZ_SCORING")
           (unit 1)
@@
     (instances
       (project ""
-        (path "/2e0f7609-671f-4aa5-9de8-e48290b9d466"
+        (path "/253667d2-eebf-4ec3-a193-9fc7a8d1f262"
           (reference "Q_BUZZER")
           (unit 1)
@@
     (instances
       (project ""
-        (path "/2e0f7609-671f-4aa5-9de8-e48290b9d466"
+        (path "/253667d2-eebf-4ec3-a193-9fc7a8d1f262"
           (reference "R_BUZZER_GATE")
           (unit 1)
@@
     (instances
       (project ""
-        (path "/2e0f7609-671f-4aa5-9de8-e48290b9d466"
+        (path "/253667d2-eebf-4ec3-a193-9fc7a8d1f262"
           (reference "R_BUZZER_GATE_PULLDOWN")
           (unit 1)
@@
     (instances
       (project ""
-        (path "/2e0f7609-671f-4aa5-9de8-e48290b9d466"
+        (path "/253667d2-eebf-4ec3-a193-9fc7a8d1f262"
           (reference "C_V5_BULK")
           (unit 1)
@@
     (instances
       (project ""
-        (path "/2e0f7609-671f-4aa5-9de8-e48290b9d466"
+        (path "/253667d2-eebf-4ec3-a193-9fc7a8d1f262"
           (reference "C_V5_BYPASS")
           (unit 1)
@@
     (instances
       (project ""
-        (path "/2e0f7609-671f-4aa5-9de8-e48290b9d466"
+        (path "/253667d2-eebf-4ec3-a193-9fc7a8d1f262"
           (reference "J_FAVERO_DATA_1")
           (unit 1)
@@
     (instances
       (project ""
-        (path "/2e0f7609-671f-4aa5-9de8-e48290b9d466"
+        (path "/253667d2-eebf-4ec3-a193-9fc7a8d1f262"
           (reference "U_FAVERO_DATA_1")
           (unit 1)
@@
     (instances
       (project ""
-        (path "/2e0f7609-671f-4aa5-9de8-e48290b9d466"
+        (path "/253667d2-eebf-4ec3-a193-9fc7a8d1f262"
           (reference "R_FAVERO_DATA_1_INPUT")
           (unit 1)
@@
     (instances
       (project ""
-        (path "/2e0f7609-671f-4aa5-9de8-e48290b9d466"
+        (path "/253667d2-eebf-4ec3-a193-9fc7a8d1f262"
           (reference "R_FAVERO_DATA_1_LOOP")
           (unit 1)
@@
     (instances
       (project ""
-        (path "/2e0f7609-671f-4aa5-9de8-e48290b9d466"
+        (path "/253667d2-eebf-4ec3-a193-9fc7a8d1f262"
           (reference "R_FAVERO_DATA_1_BASE")
           (unit 1)
@@
     (instances
       (project ""
-        (path "/2e0f7609-671f-4aa5-9de8-e48290b9d466"
+        (path "/253667d2-eebf-4ec3-a193-9fc7a8d1f262"
           (reference "D_FAVERO_DATA_1")
           (unit 1)
@@
     (instances
       (project ""
-        (path "/2e0f7609-671f-4aa5-9de8-e48290b9d466"
+        (path "/253667d2-eebf-4ec3-a193-9fc7a8d1f262"
           (reference "J_FAVERO_DATA_2")
           (unit 1)
@@
     (instances
       (project ""
-        (path "/2e0f7609-671f-4aa5-9de8-e48290b9d466"
+        (path "/253667d2-eebf-4ec3-a193-9fc7a8d1f262"
           (reference "U_FAVERO_DATA_2")
           (unit 1)
@@
     (instances
       (project ""
-        (path "/2e0f7609-671f-4aa5-9de8-e48290b9d466"
+        (path "/253667d2-eebf-4ec3-a193-9fc7a8d1f262"
           (reference "R_FAVERO_DATA_2_INPUT")
           (unit 1)
@@
     (instances
       (project ""
-        (path "/2e0f7609-671f-4aa5-9de8-e48290b9d466"
+        (path "/253667d2-eebf-4ec3-a193-9fc7a8d1f262"
           (reference "R_FAVERO_DATA_2_LOOP")
           (unit 1)
@@
     (instances
       (project ""
-        (path "/2e0f7609-671f-4aa5-9de8-e48290b9d466"
+        (path "/253667d2-eebf-4ec3-a193-9fc7a8d1f262"
           (reference "R_FAVERO_DATA_2_BASE")
           (unit 1)
@@
     (instances
       (project ""
-        (path "/2e0f7609-671f-4aa5-9de8-e48290b9d466"
+        (path "/253667d2-eebf-4ec3-a193-9fc7a8d1f262"
           (reference "D_FAVERO_DATA_2")
           (unit 1)
@@
     (instances
       (project ""
-        (path "/2e0f7609-671f-4aa5-9de8-e48290b9d466"
+        (path "/253667d2-eebf-4ec3-a193-9fc7a8d1f262"
           (reference "V5")
           (unit 1)
@@
     (instances
       (project ""
-        (path "/2e0f7609-671f-4aa5-9de8-e48290b9d466"
+        (path "/253667d2-eebf-4ec3-a193-9fc7a8d1f262"
           (reference "V5")
           (unit 1)
@@
     (instances
       (project ""
-        (path "/2e0f7609-671f-4aa5-9de8-e48290b9d466"
+        (path "/253667d2-eebf-4ec3-a193-9fc7a8d1f262"
           (reference "V5")
           (unit 1)
@@
     (instances
       (project ""
-        (path "/2e0f7609-671f-4aa5-9de8-e48290b9d466"
+        (path "/253667d2-eebf-4ec3-a193-9fc7a8d1f262"
           (reference "V5")
           (unit 1)
