File: packages/scoring-circuit/pcb/scoring-prototype-board.kicad_pcb (KiCad board)
At the start: 2 copper layers, 160 x 100 mm, 43 parts

Commit message: feat(scoring-circuit): validate prototype electronics with ngspice
Parts:
- R_FAVERO_DATA_1_INPUT, R_FAVERO_DATA_2_INPUT: value 330Ω -> 82Ω; footprint tscircuit:RC0805FR-07330RL -> tscircuit:RC0805FR-0782RL
Changed lines of the file:
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@@
   )
   (footprint
-    "tscircuit:RC0805FR-07330RL"
+    "tscircuit:RC0805FR-0782RL"
     (layer F.Cu)
     (at 148 118 0)
@@
       )
     )
-    (property "Value" "330Ω"
+    (property "Value" "82Ω"
       (at 0 3 0)
       (layer F.Fab)
@@
   )
   (footprint
-    "tscircuit:RC0805FR-07330RL"
+    "tscircuit:RC0805FR-0782RL"
     (layer F.Cu)
     (at 168 118 0)
@@
       )
     )
-    (property "Value" "330Ω"
+    (property "Value" "82Ω"
       (at 0 3 0)
       (layer F.Fab)
