File: packages/scoring-circuit/usb-scoring-platform/usb-and-power.kicad_sch (KiCad schematic)
At the start: 16 parts, among them J1 GCT USB4105-GF-A, U3 TPD2E2U06DCKR, U4 AP2112K-3.3TRG1, U7 AP63203WU-7

Commit message: fix(scoring-circuit): clear USB locating holes without moving connector
Parts:
- J1: footprint Connector_USB:USB_C_Receptacle_GCT_USB4105-xx-A_16P_TopMnt_Horizontal -> ScoringPlatform:USB4105_GF_A
Changed lines of the file:
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@@
 (paper "A3")
 (title_block (title "USB-C computer connection and PD power") (rev "Engineering draft") (comment 1 "NOT FOR FABRICATION"))
-(symbol (lib_id "Connector:USB_C_Receptacle_USB2.0_16P") (at 49.53 64.77 0) (unit 1) (in_bom yes) (on_board yes) (dnp no) (property "Reference" "J1" (at 49.53 40.53 0) (effects (font (size 1.2 1.2)))) (property "Value" "GCT USB4105-GF-A" (at 49.53 42.53 0) (effects (font (size 1.1 1.1)))) (property "Footprint" "Connector_USB:USB_C_Receptacle_GCT_USB4105-xx-A_16P_TopMnt_Horizontal" (at 49.53 64.77 0) (effects (font (size 1 1)) (hide yes))) (pin "A1") (pin "A4") (pin "A5") (pin "A6") (pin "A7") (pin "A8") (pin "A9") (pin "A12") (pin "B1") (pin "B4") (pin "B5") (pin "B6") (pin "B7") (pin "B8") (pin "B9") (pin "B12") (pin "SH") (instances (project "usb-scoring-platform" (path "/20cc8167-128c-446a-a106-f942323e143f/36d13c9b-c278-4925-a3f2-4480b5a41043" (reference "J1") (unit 1)))))
+(symbol (lib_id "Connector:USB_C_Receptacle_USB2.0_16P") (at 49.53 64.77 0) (unit 1) (in_bom yes) (on_board yes) (dnp no) (property "Reference" "J1" (at 49.53 40.53 0) (effects (font (size 1.2 1.2)))) (property "Value" "GCT USB4105-GF-A" (at 49.53 42.53 0) (effects (font (size 1.1 1.1)))) (property "Footprint" "ScoringPlatform:USB4105_GF_A" (at 49.53 64.77 0) (effects (font (size 1 1)) (hide yes))) (pin "A1") (pin "A4") (pin "A5") (pin "A6") (pin "A7") (pin "A8") (pin "A9") (pin "A12") (pin "B1") (pin "B4") (pin "B5") (pin "B6") (pin "B7") (pin "B8") (pin "B9") (pin "B12") (pin "SH") (instances (project "usb-scoring-platform" (path "/20cc8167-128c-446a-a106-f942323e143f/36d13c9b-c278-4925-a3f2-4480b5a41043" (reference "J1") (unit 1)))))
 (wire (pts (xy 49.53 87.63) (xy 49.53 92.71)) (stroke (width 0) (type default)))
 (global_label "USB_GND" (shape bidirectional) (at 49.53 92.71 0) (effects (font (size 0.9 0.9)) (justify left)) (property "Intersheetrefs" "" (at 49.53 92.71 0) (effects (font (size 1 1)) (hide yes))))

Commit message: feat(scoring-circuit): select exact prototype resistor parts
Parts:
- R3: MPN (none) -> RC0603FR-07100KL; Manufacturer (none) -> YAGEO
- R4: MPN (none) -> RC0603FR-07150KL; Manufacturer (none) -> YAGEO
Changed lines of the file:
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@@
 (wire (pts (xy 275.59 114.3) (xy 275.59 119.38)) (stroke (width 0) (type default)))
 (global_label "GND" (shape bidirectional) (at 275.59 119.38 0) (effects (font (size 0.9 0.9)) (justify left)) (property "Intersheetrefs" "" (at 275.59 119.38 0) (effects (font (size 1 1)) (hide yes))))
-(symbol (lib_id "Device:R") (at 335.28 49.53 0) (unit 1) (in_bom yes) (on_board yes) (dnp no) (property "Reference" "R3" (at 335.28 35.53 0) (effects (font (size 1.2 1.2)))) (property "Value" "100k 1%" (at 335.28 37.53 0) (effects (font (size 1.1 1.1)))) (property "Footprint" "Resistor_SMD:R_0603_1608Metric" (at 335.28 49.53 0) (effects (font (size 1 1)) (hide yes))) (pin "1") (pin "2") (instances (project "usb-scoring-platform" (path "/20cc8167-128c-446a-a106-f942323e143f/36d13c9b-c278-4925-a3f2-4480b5a41043" (reference "R3") (unit 1)))))
+(symbol (lib_id "Device:R") (at 335.28 49.53 0) (unit 1) (in_bom yes) (on_board yes) (dnp no) (property "Reference" "R3" (at 335.28 35.53 0) (effects (font (size 1.2 1.2)))) (property "Value" "100k 1%" (at 335.28 37.53 0) (effects (font (size 1.1 1.1)))) (property "Footprint" "Resistor_SMD:R_0603_1608Metric" (at 335.28 49.53 0) (effects (font (size 1 1)) (hide yes))) (pin "1") (pin "2") (property "Manufacturer" "YAGEO" (at 335.28 49.53 0) (effects (font (size 1 1)) (hide yes))) (property "MPN" "RC0603FR-07100KL" (at 335.28 49.53 0) (effects (font (size 1 1)) (hide yes))) (property "Datasheet" "https://www.yageogroup.com/component-documentation/download/specsheet/RC0603FR-07100KL" (at 335.28 49.53 0) (effects (font (size 1 1)) (hide yes))) (instances (project "usb-scoring-platform" (path "/20cc8167-128c-446a-a106-f942323e143f/36d13c9b-c278-4925-a3f2-4480b5a41043" (reference "R3") (unit 1)))))
 (wire (pts (xy 335.28 45.72) (xy 335.28 40.64)) (stroke (width 0) (type default)))
 (global_label "USB_ISOLATED_5V" (shape bidirectional) (at 335.28 40.64 0) (effects (font (size 0.9 0.9)) (justify left)) (property "Intersheetrefs" "" (at 335.28 40.64 0) (effects (font (size 1 1)) (hide yes))))
 (wire (pts (xy 335.28 53.34) (xy 335.28 58.42)) (stroke (width 0) (type default)))
 (global_label "USB_PRESENT" (shape bidirectional) (at 335.28 58.42 0) (effects (font (size 0.9 0.9)) (justify left)) (property "Intersheetrefs" "" (at 335.28 58.42 0) (effects (font (size 1 1)) (hide yes))))
-(symbol (lib_id "Device:R") (at 379.73 49.53 0) (unit 1) (in_bom yes) (on_board yes) (dnp no) (property "Reference" "R4" (at 379.73 35.53 0) (effects (font (size 1.2 1.2)))) (property "Value" "150k 1%" (at 379.73 37.53 0) (effects (font (size 1.1 1.1)))) (property "Footprint" "Resistor_SMD:R_0603_1608Metric" (at 379.73 49.53 0) (effects (font (size 1 1)) (hide yes))) (pin "1") (pin "2") (instances (project "usb-scoring-platform" (path "/20cc8167-128c-446a-a106-f942323e143f/36d13c9b-c278-4925-a3f2-4480b5a41043" (reference "R4") (unit 1)))))
+(symbol (lib_id "Device:R") (at 379.73 49.53 0) (unit 1) (in_bom yes) (on_board yes) (dnp no) (property "Reference" "R4" (at 379.73 35.53 0) (effects (font (size 1.2 1.2)))) (property "Value" "150k 1%" (at 379.73 37.53 0) (effects (font (size 1.1 1.1)))) (property "Footprint" "Resistor_SMD:R_0603_1608Metric" (at 379.73 49.53 0) (effects (font (size 1 1)) (hide yes))) (pin "1") (pin "2") (property "Manufacturer" "YAGEO" (at 379.73 49.53 0) (effects (font (size 1 1)) (hide yes))) (property "MPN" "RC0603FR-07150KL" (at 379.73 49.53 0) (effects (font (size 1 1)) (hide yes))) (property "Datasheet" "https://www.yageogroup.com/component-documentation/download/specsheet/RC0603FR-07150KL" (at 379.73 49.53 0) (effects (font (size 1 1)) (hide yes))) (instances (project "usb-scoring-platform" (path "/20cc8167-128c-446a-a106-f942323e143f/36d13c9b-c278-4925-a3f2-4480b5a41043" (reference "R4") (unit 1)))))
 (wire (pts (xy 379.73 45.72) (xy 379.73 40.64)) (stroke (width 0) (type default)))
 (global_label "USB_PRESENT" (shape bidirectional) (at 379.73 40.64 0) (effects (font (size 0.9 0.9)) (justify left)) (property "Intersheetrefs" "" (at 379.73 40.64 0) (effects (font (size 1 1)) (hide yes))))

Commit message: feat(scoring-circuit): select bypass and timing capacitors
Parts:
- C4: MPN (none) -> C1608X7R1H104K080AA; Manufacturer (none) -> TDK
Changed lines of the file:
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@@
 (wire (pts (xy 320.04 179.07) (xy 320.04 184.15)) (stroke (width 0) (type default)))
 (global_label "APP_3V3" (shape bidirectional) (at 320.04 184.15 0) (effects (font (size 0.9 0.9)) (justify left)) (property "Intersheetrefs" "" (at 320.04 184.15 0) (effects (font (size 1 1)) (hide yes))))
-(symbol (lib_id "Device:C") (at 255.27 219.71 0) (unit 1) (in_bom yes) (on_board yes) (dnp no) (property "Reference" "C4" (at 255.27 205.71 0) (effects (font (size 1.2 1.2)))) (property "Value" "100nF 16V" (at 255.27 207.71 0) (effects (font (size 1.1 1.1)))) (property "Footprint" "Capacitor_SMD:C_0603_1608Metric" (at 255.27 219.71 0) (effects (font (size 1 1)) (hide yes))) (pin "1") (pin "2") (instances (project "usb-scoring-platform" (path "/20cc8167-128c-446a-a106-f942323e143f/36d13c9b-c278-4925-a3f2-4480b5a41043" (reference "C4") (unit 1)))))
+(symbol (lib_id "Device:C") (at 255.27 219.71 0) (unit 1) (in_bom yes) (on_board yes) (dnp no) (property "Reference" "C4" (at 255.27 205.71 0) (effects (font (size 1.2 1.2)))) (property "Value" "100nF 16V" (at 255.27 207.71 0) (effects (font (size 1.1 1.1)))) (property "Footprint" "Capacitor_SMD:C_0603_1608Metric" (at 255.27 219.71 0) (effects (font (size 1 1)) (hide yes))) (pin "1") (pin "2") (property "Manufacturer" "TDK" (at 255.27 219.71 0) (effects (font (size 1 1)) (hide yes))) (property "MPN" "C1608X7R1H104K080AA" (at 255.27 219.71 0) (effects (font (size 1 1)) (hide yes))) (property "Datasheet" "https://product.tdk.com/en/search/capacitor/ceramic/mlcc/info?part_no=C1608X7R1H104K080AA" (at 255.27 219.71 0) (effects (font (size 1 1)) (hide yes))) (instances (project "usb-scoring-platform" (path "/20cc8167-128c-446a-a106-f942323e143f/36d13c9b-c278-4925-a3f2-4480b5a41043" (reference "C4") (unit 1)))))
 (wire (pts (xy 255.27 215.9) (xy 255.27 210.82)) (stroke (width 0) (type default)))
 (global_label "BUCK_BOOT" (shape bidirectional) (at 255.27 210.82 0) (effects (font (size 0.9 0.9)) (justify left)) (property "Intersheetrefs" "" (at 255.27 210.82 0) (effects (font (size 1 1)) (hide yes))))
