File: packages/scoring-circuit/usb-scoring-platform/usb-and-power.kicad_sch (KiCad schematic)
At the start: 16 parts, among them J1 GCT USB4105-GF-A, U3 TPD2E2U06DCKR, U4 AP2112K-3.3TRG1, U7 AP63203WU-7

Commit message: feat(scoring-circuit): select local supply capacitors
Parts:
- C2, C3: MPN (none) -> C1608X7R1H105K080AB; Manufacturer (none) -> TDK
Changed lines of the file:
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@@
 (wire (pts (xy 273.05 57.15) (xy 278.13 57.15)) (stroke (width 0) (type default)))
 (global_label "CORE_3V3" (shape bidirectional) (at 278.13 57.15 0) (effects (font (size 0.9 0.9)) (justify left)) (property "Intersheetrefs" "" (at 278.13 57.15 0) (effects (font (size 1 1)) (hide yes))))
-(symbol (lib_id "Device:C") (at 229.87 110.49 0) (unit 1) (in_bom yes) (on_board yes) (dnp no) (property "Reference" "C2" (at 229.87 96.49 0) (effects (font (size 1.2 1.2)))) (property "Value" "1uF 10V" (at 229.87 98.49 0) (effects (font (size 1.1 1.1)))) (property "Footprint" "Capacitor_SMD:C_0603_1608Metric" (at 229.87 110.49 0) (effects (font (size 1 1)) (hide yes))) (pin "1") (pin "2") (instances (project "usb-scoring-platform" (path "/20cc8167-128c-446a-a106-f942323e143f/36d13c9b-c278-4925-a3f2-4480b5a41043" (reference "C2") (unit 1)))))
+(symbol (lib_id "Device:C") (at 229.87 110.49 0) (unit 1) (in_bom yes) (on_board yes) (dnp no) (property "Reference" "C2" (at 229.87 96.49 0) (effects (font (size 1.2 1.2)))) (property "Value" "1uF 10V" (at 229.87 98.49 0) (effects (font (size 1.1 1.1)))) (property "Footprint" "Capacitor_SMD:C_0603_1608Metric" (at 229.87 110.49 0) (effects (font (size 1 1)) (hide yes))) (pin "1") (pin "2") (property "Manufacturer" "TDK" (at 229.87 110.49 0) (effects (font (size 1 1)) (hide yes))) (property "MPN" "C1608X7R1H105K080AB" (at 229.87 110.49 0) (effects (font (size 1 1)) (hide yes))) (property "Datasheet" "https://product.tdk.com/en/search/capacitor/ceramic/mlcc/info?part_no=C1608X7R1H105K080AB" (at 229.87 110.49 0) (effects (font (size 1 1)) (hide yes))) (instances (project "usb-scoring-platform" (path "/20cc8167-128c-446a-a106-f942323e143f/36d13c9b-c278-4925-a3f2-4480b5a41043" (reference "C2") (unit 1)))))
 (wire (pts (xy 229.87 106.68) (xy 229.87 101.6)) (stroke (width 0) (type default)))
 (global_label "CORE_5V" (shape bidirectional) (at 229.87 101.6 0) (effects (font (size 0.9 0.9)) (justify left)) (property "Intersheetrefs" "" (at 229.87 101.6 0) (effects (font (size 1 1)) (hide yes))))
 (wire (pts (xy 229.87 114.3) (xy 229.87 119.38)) (stroke (width 0) (type default)))
 (global_label "GND" (shape bidirectional) (at 229.87 119.38 0) (effects (font (size 0.9 0.9)) (justify left)) (property "Intersheetrefs" "" (at 229.87 119.38 0) (effects (font (size 1 1)) (hide yes))))
-(symbol (lib_id "Device:C") (at 275.59 110.49 0) (unit 1) (in_bom yes) (on_board yes) (dnp no) (property "Reference" "C3" (at 275.59 96.49 0) (effects (font (size 1.2 1.2)))) (property "Value" "1uF 10V" (at 275.59 98.49 0) (effects (font (size 1.1 1.1)))) (property "Footprint" "Capacitor_SMD:C_0603_1608Metric" (at 275.59 110.49 0) (effects (font (size 1 1)) (hide yes))) (pin "1") (pin "2") (instances (project "usb-scoring-platform" (path "/20cc8167-128c-446a-a106-f942323e143f/36d13c9b-c278-4925-a3f2-4480b5a41043" (reference "C3") (unit 1)))))
+(symbol (lib_id "Device:C") (at 275.59 110.49 0) (unit 1) (in_bom yes) (on_board yes) (dnp no) (property "Reference" "C3" (at 275.59 96.49 0) (effects (font (size 1.2 1.2)))) (property "Value" "1uF 10V" (at 275.59 98.49 0) (effects (font (size 1.1 1.1)))) (property "Footprint" "Capacitor_SMD:C_0603_1608Metric" (at 275.59 110.49 0) (effects (font (size 1 1)) (hide yes))) (pin "1") (pin "2") (property "Manufacturer" "TDK" (at 275.59 110.49 0) (effects (font (size 1 1)) (hide yes))) (property "MPN" "C1608X7R1H105K080AB" (at 275.59 110.49 0) (effects (font (size 1 1)) (hide yes))) (property "Datasheet" "https://product.tdk.com/en/search/capacitor/ceramic/mlcc/info?part_no=C1608X7R1H105K080AB" (at 275.59 110.49 0) (effects (font (size 1 1)) (hide yes))) (instances (project "usb-scoring-platform" (path "/20cc8167-128c-446a-a106-f942323e143f/36d13c9b-c278-4925-a3f2-4480b5a41043" (reference "C3") (unit 1)))))
 (wire (pts (xy 275.59 106.68) (xy 275.59 101.6)) (stroke (width 0) (type default)))
 (global_label "CORE_3V3" (shape bidirectional) (at 275.59 101.6 0) (effects (font (size 0.9 0.9)) (justify left)) (property "Intersheetrefs" "" (at 275.59 101.6 0) (effects (font (size 1 1)) (hide yes))))

Commit message: feat(scoring-circuit): complete nominal capacitor selections
Parts:
- C5: MPN (none) -> C1608X5R1C106M080AB; Manufacturer (none) -> TDK
- C6, C7: MPN (none) -> GRM32ER71E226KE15L; Manufacturer (none) -> Murata
Changed lines of the file:
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@@
 (wire (pts (xy 255.27 223.52) (xy 255.27 228.6)) (stroke (width 0) (type default)))
 (global_label "BUCK_SW" (shape bidirectional) (at 255.27 228.6 0) (effects (font (size 0.9 0.9)) (justify left)) (property "Intersheetrefs" "" (at 255.27 228.6 0) (effects (font (size 1 1)) (hide yes))))
-(symbol (lib_id "Device:C") (at 204.47 219.71 0) (unit 1) (in_bom yes) (on_board yes) (dnp no) (property "Reference" "C5" (at 204.47 205.71 0) (effects (font (size 1.2 1.2)))) (property "Value" "10uF 16V" (at 204.47 207.71 0) (effects (font (size 1.1 1.1)))) (property "Footprint" "Capacitor_SMD:C_0603_1608Metric" (at 204.47 219.71 0) (effects (font (size 1 1)) (hide yes))) (pin "1") (pin "2") (instances (project "usb-scoring-platform" (path "/20cc8167-128c-446a-a106-f942323e143f/36d13c9b-c278-4925-a3f2-4480b5a41043" (reference "C5") (unit 1)))))
+(symbol (lib_id "Device:C") (at 204.47 219.71 0) (unit 1) (in_bom yes) (on_board yes) (dnp no) (property "Reference" "C5" (at 204.47 205.71 0) (effects (font (size 1.2 1.2)))) (property "Value" "10uF 16V" (at 204.47 207.71 0) (effects (font (size 1.1 1.1)))) (property "Footprint" "Capacitor_SMD:C_0603_1608Metric" (at 204.47 219.71 0) (effects (font (size 1 1)) (hide yes))) (pin "1") (pin "2") (property "Manufacturer" "TDK" (at 0 0 0) (effects (font (size 1 1)) (hide yes))) (property "MPN" "C1608X5R1C106M080AB" (at 0 0 0) (effects (font (size 1 1)) (hide yes))) (property "Datasheet" "https://product.tdk.com/en/search/capacitor/ceramic/mlcc/info?part_no=C1608X5R1C106M080AB" (at 0 0 0) (effects (font (size 1 1)) (hide yes))) (instances (project "usb-scoring-platform" (path "/20cc8167-128c-446a-a106-f942323e143f/36d13c9b-c278-4925-a3f2-4480b5a41043" (reference "C5") (unit 1)))))
 (wire (pts (xy 204.47 215.9) (xy 204.47 210.82)) (stroke (width 0) (type default)))
 (global_label "PANEL_5V" (shape bidirectional) (at 204.47 210.82 0) (effects (font (size 0.9 0.9)) (justify left)) (property "Intersheetrefs" "" (at 204.47 210.82 0) (effects (font (size 1 1)) (hide yes))))
 (wire (pts (xy 204.47 223.52) (xy 204.47 228.6)) (stroke (width 0) (type default)))
 (global_label "GND" (shape bidirectional) (at 204.47 228.6 0) (effects (font (size 0.9 0.9)) (justify left)) (property "Intersheetrefs" "" (at 204.47 228.6 0) (effects (font (size 1 1)) (hide yes))))
-(symbol (lib_id "Device:C") (at 320.04 219.71 0) (unit 1) (in_bom yes) (on_board yes) (dnp no) (property "Reference" "C6" (at 320.04 205.71 0) (effects (font (size 1.2 1.2)))) (property "Value" "22uF 10V X7R" (at 320.04 207.71 0) (effects (font (size 1.1 1.1)))) (property "Footprint" "Capacitor_SMD:C_1210_3225Metric" (at 320.04 219.71 0) (effects (font (size 1 1)) (hide yes))) (pin "1") (pin "2") (instances (project "usb-scoring-platform" (path "/20cc8167-128c-446a-a106-f942323e143f/36d13c9b-c278-4925-a3f2-4480b5a41043" (reference "C6") (unit 1)))))
+(symbol (lib_id "Device:C") (at 320.04 219.71 0) (unit 1) (in_bom yes) (on_board yes) (dnp no) (property "Reference" "C6" (at 320.04 205.71 0) (effects (font (size 1.2 1.2)))) (property "Value" "22uF 10V X7R" (at 320.04 207.71 0) (effects (font (size 1.1 1.1)))) (property "Footprint" "Capacitor_SMD:C_1210_3225Metric" (at 320.04 219.71 0) (effects (font (size 1 1)) (hide yes))) (pin "1") (pin "2") (property "Manufacturer" "Murata" (at 0 0 0) (effects (font (size 1 1)) (hide yes))) (property "MPN" "GRM32ER71E226KE15L" (at 0 0 0) (effects (font (size 1 1)) (hide yes))) (property "Datasheet" "https://www.murata.com/en-global/api/pdfdownloadapi?cate=luCeramicCapacitorsSMD&partno=GRM32ER71E226KE15%23" (at 0 0 0) (effects (font (size 1 1)) (hide yes))) (instances (project "usb-scoring-platform" (path "/20cc8167-128c-446a-a106-f942323e143f/36d13c9b-c278-4925-a3f2-4480b5a41043" (reference "C6") (unit 1)))))
 (wire (pts (xy 320.04 215.9) (xy 320.04 210.82)) (stroke (width 0) (type default)))
 (global_label "APP_3V3" (shape bidirectional) (at 320.04 210.82 0) (effects (font (size 0.9 0.9)) (justify left)) (property "Intersheetrefs" "" (at 320.04 210.82 0) (effects (font (size 1 1)) (hide yes))))
 (wire (pts (xy 320.04 223.52) (xy 320.04 228.6)) (stroke (width 0) (type default)))
 (global_label "GND" (shape bidirectional) (at 320.04 228.6 0) (effects (font (size 0.9 0.9)) (justify left)) (property "Intersheetrefs" "" (at 320.04 228.6 0) (effects (font (size 1 1)) (hide yes))))
-(symbol (lib_id "Device:C") (at 364.49 219.71 0) (unit 1) (in_bom yes) (on_board yes) (dnp no) (property "Reference" "C7" (at 364.49 205.71 0) (effects (font (size 1.2 1.2)))) (property "Value" "22uF 10V X7R" (at 364.49 207.71 0) (effects (font (size 1.1 1.1)))) (property "Footprint" "Capacitor_SMD:C_1210_3225Metric" (at 364.49 219.71 0) (effects (font (size 1 1)) (hide yes))) (pin "1") (pin "2") (instances (project "usb-scoring-platform" (path "/20cc8167-128c-446a-a106-f942323e143f/36d13c9b-c278-4925-a3f2-4480b5a41043" (reference "C7") (unit 1)))))
+(symbol (lib_id "Device:C") (at 364.49 219.71 0) (unit 1) (in_bom yes) (on_board yes) (dnp no) (property "Reference" "C7" (at 364.49 205.71 0) (effects (font (size 1.2 1.2)))) (property "Value" "22uF 10V X7R" (at 364.49 207.71 0) (effects (font (size 1.1 1.1)))) (property "Footprint" "Capacitor_SMD:C_1210_3225Metric" (at 364.49 219.71 0) (effects (font (size 1 1)) (hide yes))) (pin "1") (pin "2") (property "Manufacturer" "Murata" (at 0 0 0) (effects (font (size 1 1)) (hide yes))) (property "MPN" "GRM32ER71E226KE15L" (at 0 0 0) (effects (font (size 1 1)) (hide yes))) (property "Datasheet" "https://www.murata.com/en-global/api/pdfdownloadapi?cate=luCeramicCapacitorsSMD&partno=GRM32ER71E226KE15%23" (at 0 0 0) (effects (font (size 1 1)) (hide yes))) (instances (project "usb-scoring-platform" (path "/20cc8167-128c-446a-a106-f942323e143f/36d13c9b-c278-4925-a3f2-4480b5a41043" (reference "C7") (unit 1)))))
 (wire (pts (xy 364.49 215.9) (xy 364.49 210.82)) (stroke (width 0) (type default)))
 (global_label "APP_3V3" (shape bidirectional) (at 364.49 210.82 0) (effects (font (size 0.9 0.9)) (justify left)) (property "Intersheetrefs" "" (at 364.49 210.82 0) (effects (font (size 1 1)) (hide yes))))

Commit message: feat(scoring-circuit): bind diode selections and review polarity
Parts:
- D1, D2: MPN (none) -> SS14-E3/61T; Manufacturer (none) -> Vishay
Changed lines of the file:
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@@
 (wire (pts (xy 90.17 128.27) (xy 90.17 133.35)) (stroke (width 0) (type default)))
 (global_label "USB_GND" (shape bidirectional) (at 90.17 133.35 0) (effects (font (size 0.9 0.9)) (justify left)) (property "Intersheetrefs" "" (at 90.17 133.35 0) (effects (font (size 1 1)) (hide yes))))
-(symbol (lib_id "Diode:SS14") (at 195.58 44.45 0) (unit 1) (in_bom yes) (on_board yes) (dnp no) (property "Reference" "D1" (at 195.58 30.45 0) (effects (font (size 1.2 1.2)))) (property "Value" "SS14" (at 195.58 32.45 0) (effects (font (size 1.1 1.1)))) (property "Footprint" "Diode_SMD:D_SMA" (at 195.58 44.45 0) (effects (font (size 1 1)) (hide yes))) (pin "1") (pin "2") (instances (project "usb-scoring-platform" (path "/20cc8167-128c-446a-a106-f942323e143f/36d13c9b-c278-4925-a3f2-4480b5a41043" (reference "D1") (unit 1)))))
+(symbol (lib_id "Diode:SS14") (at 195.58 44.45 0) (unit 1) (in_bom yes) (on_board yes) (dnp no) (property "Reference" "D1" (at 195.58 30.45 0) (effects (font (size 1.2 1.2)))) (property "Value" "SS14" (at 195.58 32.45 0) (effects (font (size 1.1 1.1)))) (property "Footprint" "Diode_SMD:D_SMA" (at 195.58 44.45 0) (effects (font (size 1 1)) (hide yes))) (pin "1") (pin "2") (property "Manufacturer" "Vishay" (at 0 0 0) (effects (font (size 1 1)) (hide yes))) (property "MPN" "SS14-E3/61T" (at 0 0 0) (effects (font (size 1 1)) (hide yes))) (property "Datasheet" "https://www.vishay.com/doc?88746" (at 0 0 0) (effects (font (size 1 1)) (hide yes))) (instances (project "usb-scoring-platform" (path "/20cc8167-128c-446a-a106-f942323e143f/36d13c9b-c278-4925-a3f2-4480b5a41043" (reference "D1") (unit 1)))))
 (wire (pts (xy 191.77 44.45) (xy 186.69 44.45)) (stroke (width 0) (type default)))
 (global_label "CORE_5V" (shape bidirectional) (at 186.69 44.45 180) (effects (font (size 0.9 0.9)) (justify right)) (property "Intersheetrefs" "" (at 186.69 44.45 180) (effects (font (size 1 1)) (hide yes))))
 (wire (pts (xy 199.39 44.45) (xy 204.47 44.45)) (stroke (width 0) (type default)))
 (global_label "USB_ISOLATED_5V" (shape bidirectional) (at 204.47 44.45 0) (effects (font (size 0.9 0.9)) (justify left)) (property "Intersheetrefs" "" (at 204.47 44.45 0) (effects (font (size 1 1)) (hide yes))))
-(symbol (lib_id "Diode:SS14") (at 195.58 90.17 0) (unit 1) (in_bom yes) (on_board yes) (dnp no) (property "Reference" "D2" (at 195.58 76.17 0) (effects (font (size 1.2 1.2)))) (property "Value" "SS14" (at 195.58 78.17 0) (effects (font (size 1.1 1.1)))) (property "Footprint" "Diode_SMD:D_SMA" (at 195.58 90.17 0) (effects (font (size 1 1)) (hide yes))) (pin "1") (pin "2") (instances (project "usb-scoring-platform" (path "/20cc8167-128c-446a-a106-f942323e143f/36d13c9b-c278-4925-a3f2-4480b5a41043" (reference "D2") (unit 1)))))
+(symbol (lib_id "Diode:SS14") (at 195.58 90.17 0) (unit 1) (in_bom yes) (on_board yes) (dnp no) (property "Reference" "D2" (at 195.58 76.17 0) (effects (font (size 1.2 1.2)))) (property "Value" "SS14" (at 195.58 78.17 0) (effects (font (size 1.1 1.1)))) (property "Footprint" "Diode_SMD:D_SMA" (at 195.58 90.17 0) (effects (font (size 1 1)) (hide yes))) (pin "1") (pin "2") (property "Manufacturer" "Vishay" (at 0 0 0) (effects (font (size 1 1)) (hide yes))) (property "MPN" "SS14-E3/61T" (at 0 0 0) (effects (font (size 1 1)) (hide yes))) (property "Datasheet" "https://www.vishay.com/doc?88746" (at 0 0 0) (effects (font (size 1 1)) (hide yes))) (instances (project "usb-scoring-platform" (path "/20cc8167-128c-446a-a106-f942323e143f/36d13c9b-c278-4925-a3f2-4480b5a41043" (reference "D2") (unit 1)))))
 (wire (pts (xy 191.77 90.17) (xy 186.69 90.17)) (stroke (width 0) (type default)))
 (global_label "CORE_5V" (shape bidirectional) (at 186.69 90.17 180) (effects (font (size 0.9 0.9)) (justify right)) (property "Intersheetrefs" "" (at 186.69 90.17 180) (effects (font (size 1 1)) (hide yes))))

Commit message: chore(scoring-circuit): bind reviewed power inductor ordering codes
Parts:
- L1: MPN (none) -> XAL5030-472MEC; Manufacturer (none) -> Coilcraft
Changed lines of the file:
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@@
 (wire (pts (xy 265.43 175.26) (xy 270.51 175.26)) (stroke (width 0) (type default)))
 (global_label "BUCK_BOOT" (shape bidirectional) (at 270.51 175.26 0) (effects (font (size 0.9 0.9)) (justify left)) (property "Intersheetrefs" "" (at 270.51 175.26 0) (effects (font (size 1 1)) (hide yes))))
-(symbol (lib_id "Device:L") (at 320.04 175.26 0) (unit 1) (in_bom yes) (on_board yes) (dnp no) (property "Reference" "L1" (at 320.04 161.26 0) (effects (font (size 1.2 1.2)))) (property "Value" "XAL5030-472MEC 4.7uH" (at 320.04 163.26 0) (effects (font (size 1.1 1.1)))) (property "Footprint" "Inductor_SMD:L_Coilcraft_XAL5030-XXX" (at 320.04 175.26 0) (effects (font (size 1 1)) (hide yes))) (pin "1") (pin "2") (instances (project "usb-scoring-platform" (path "/20cc8167-128c-446a-a106-f942323e143f/36d13c9b-c278-4925-a3f2-4480b5a41043" (reference "L1") (unit 1)))))
+(symbol (lib_id "Device:L") (at 320.04 175.26 0) (unit 1) (in_bom yes) (on_board yes) (dnp no) (property "Reference" "L1" (at 320.04 161.26 0) (effects (font (size 1.2 1.2)))) (property "Value" "XAL5030-472MEC 4.7uH" (at 320.04 163.26 0) (effects (font (size 1.1 1.1)))) (property "Footprint" "Inductor_SMD:L_Coilcraft_XAL5030-XXX" (at 320.04 175.26 0) (effects (font (size 1 1)) (hide yes))) (pin "1") (pin "2") (instances (project "usb-scoring-platform" (path "/20cc8167-128c-446a-a106-f942323e143f/36d13c9b-c278-4925-a3f2-4480b5a41043" (reference "L1") (unit 1)))) (property "Manufacturer" "Coilcraft" (at 0 0 0) (effects (font (size 1 1)) (hide yes))) (property "MPN" "XAL5030-472MEC" (at 0 0 0) (effects (font (size 1 1)) (hide yes))) (property "Datasheet" "https://www.coilcraft.com/getmedia/49bc46c8-4b2c-45b9-9b6c-2eaa235ea698/xal50xx.pdf" (at 0 0 0) (effects (font (size 1 1)) (hide yes))))
 (wire (pts (xy 320.04 171.45) (xy 320.04 166.37)) (stroke (width 0) (type default)))
 (global_label "BUCK_SW" (shape bidirectional) (at 320.04 166.37 0) (effects (font (size 0.9 0.9)) (justify left)) (property "Intersheetrefs" "" (at 320.04 166.37 0) (effects (font (size 1 1)) (hide yes))))
