File: packages/scoring-circuit/usb-scoring-platform/usb-and-power.kicad_sch (KiCad schematic)
At the start: 16 parts, among them J1 GCT USB4105-GF-A, U3 TPD2E2U06DCKR, U4 AP2112K-3.3TRG1, U7 AP63203WU-7

Commit message: chore(scoring-circuit): complete assembly BOM ordering fields
Parts:
- J1: MPN (none) -> USB4105-GF-A; Manufacturer (none) -> GCT
- U3: MPN (none) -> TPD2E2U06DCKR; Manufacturer (none) -> Texas Instruments
- U4: MPN (none) -> AP2112K-3.3TRG1; Manufacturer (none) -> Diodes Incorporated
- U7: MPN (none) -> AP63203WU-7; Manufacturer (none) -> Diodes Incorporated
Changed lines of the file:
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@@
 (paper "A3")
 (title_block (title "USB-C computer connection and PD power") (rev "Engineering draft") (comment 1 "NOT FOR FABRICATION"))
-(symbol (lib_id "Connector:USB_C_Receptacle_USB2.0_16P") (at 49.53 64.77 0) (unit 1) (in_bom yes) (on_board yes) (dnp no) (property "Reference" "J1" (at 49.53 40.53 0) (effects (font (size 1.2 1.2)))) (property "Value" "GCT USB4105-GF-A" (at 49.53 42.53 0) (effects (font (size 1.1 1.1)))) (property "Footprint" "ScoringPlatform:USB4105_GF_A" (at 49.53 64.77 0) (effects (font (size 1 1)) (hide yes))) (pin "A1") (pin "A4") (pin "A5") (pin "A6") (pin "A7") (pin "A8") (pin "A9") (pin "A12") (pin "B1") (pin "B4") (pin "B5") (pin "B6") (pin "B7") (pin "B8") (pin "B9") (pin "B12") (pin "SH") (instances (project "usb-scoring-platform" (path "/20cc8167-128c-446a-a106-f942323e143f/36d13c9b-c278-4925-a3f2-4480b5a41043" (reference "J1") (unit 1)))))
+(symbol (lib_id "Connector:USB_C_Receptacle_USB2.0_16P") (at 49.53 64.77 0) (unit 1) (in_bom yes) (on_board yes) (dnp no) (property "Reference" "J1" (at 49.53 40.53 0) (effects (font (size 1.2 1.2)))) (property "Value" "GCT USB4105-GF-A" (at 49.53 42.53 0) (effects (font (size 1.1 1.1)))) (property "Footprint" "ScoringPlatform:USB4105_GF_A" (at 49.53 64.77 0) (effects (font (size 1 1)) (hide yes))) (pin "A1") (pin "A4") (pin "A5") (pin "A6") (pin "A7") (pin "A8") (pin "A9") (pin "A12") (pin "B1") (pin "B4") (pin "B5") (pin "B6") (pin "B7") (pin "B8") (pin "B9") (pin "B12") (pin "SH") (instances (project "usb-scoring-platform" (path "/20cc8167-128c-446a-a106-f942323e143f/36d13c9b-c278-4925-a3f2-4480b5a41043" (reference "J1") (unit 1)))) (property "Manufacturer" "GCT" (at 0 0 0) (effects (font (size 1 1)) (hide yes))) (property "MPN" "USB4105-GF-A" (at 0 0 0) (effects (font (size 1 1)) (hide yes))))
 (wire (pts (xy 49.53 87.63) (xy 49.53 92.71)) (stroke (width 0) (type default)))
 (global_label "USB_GND" (shape bidirectional) (at 49.53 92.71 0) (effects (font (size 0.9 0.9)) (justify left)) (property "Intersheetrefs" "" (at 49.53 92.71 0) (effects (font (size 1 1)) (hide yes))))
@@
 (wire (pts (xy 41.91 87.63) (xy 41.91 92.71)) (stroke (width 0) (type default)))
 (global_label "USB_GND" (shape bidirectional) (at 41.91 92.71 0) (effects (font (size 0.9 0.9)) (justify left)) (property "Intersheetrefs" "" (at 41.91 92.71 0) (effects (font (size 1 1)) (hide yes))))
-(symbol (lib_id "Power_Protection:TPD2E2U06DCK") (at 124.46 90.17 0) (unit 1) (in_bom yes) (on_board yes) (dnp no) (property "Reference" "U3" (at 124.46 76.09 0) (effects (font (size 1.2 1.2)))) (property "Value" "TPD2E2U06DCKR" (at 124.46 78.09 0) (effects (font (size 1.1 1.1)))) (property "Footprint" "ScoringPlatform:TPD2E2U06DCKR" (at 124.46 90.17 0) (effects (font (size 1 1)) (hide yes))) (instances (project "usb-scoring-platform" (path "/20cc8167-128c-446a-a106-f942323e143f/36d13c9b-c278-4925-a3f2-4480b5a41043" (reference "U3") (unit 1)))) (property "Datasheet" "https://www.ti.com/lit/ds/symlink/tpd2e2u06.pdf" (at 124.46 90.17 0) (effects (font (size 1 1)) (hide yes))) (pin "1") (pin "2") (pin "3"))
+(symbol (lib_id "Power_Protection:TPD2E2U06DCK") (at 124.46 90.17 0) (unit 1) (in_bom yes) (on_board yes) (dnp no) (property "Reference" "U3" (at 124.46 76.09 0) (effects (font (size 1.2 1.2)))) (property "Value" "TPD2E2U06DCKR" (at 124.46 78.09 0) (effects (font (size 1.1 1.1)))) (property "Footprint" "ScoringPlatform:TPD2E2U06DCKR" (at 124.46 90.17 0) (effects (font (size 1 1)) (hide yes))) (instances (project "usb-scoring-platform" (path "/20cc8167-128c-446a-a106-f942323e143f/36d13c9b-c278-4925-a3f2-4480b5a41043" (reference "U3") (unit 1)))) (property "Datasheet" "https://www.ti.com/lit/ds/symlink/tpd2e2u06.pdf" (at 124.46 90.17 0) (effects (font (size 1 1)) (hide yes))) (pin "1") (pin "2") (pin "3") (property "Manufacturer" "Texas Instruments" (at 0 0 0) (effects (font (size 1 1)) (hide yes))) (property "MPN" "TPD2E2U06DCKR" (at 0 0 0) (effects (font (size 1 1)) (hide yes))))
 (symbol (lib_id "Device:C") (at 90.17 124.46 0) (unit 1) (in_bom yes) (on_board yes) (dnp no) (property "Reference" "C1" (at 90.17 110.46 0) (effects (font (size 1.2 1.2)))) (property "Value" "1uF 50V" (at 90.17 112.46 0) (effects (font (size 1.1 1.1)))) (property "Footprint" "Capacitor_SMD:C_0603_1608Metric" (at 90.17 124.46 0) (effects (font (size 1 1)) (hide yes))) (property "Manufacturer" "TDK" (at 90.17 124.46 0) (effects (font (size 1 1)) (hide yes))) (property "MPN" "C1608X7R1H105K080AB" (at 90.17 124.46 0) (effects (font (size 1 1)) (hide yes))) (property "Datasheet" "https://product.tdk.com/en/search/capacitor/ceramic/mlcc/info?part_no=C1608X7R1H105K080AB" (at 90.17 124.46 0) (effects (font (size 1 1)) (hide yes))) (pin "1") (pin "2") (instances (project "usb-scoring-platform" (path "/20cc8167-128c-446a-a106-f942323e143f/36d13c9b-c278-4925-a3f2-4480b5a41043" (reference "C1") (unit 1)))))
 (wire (pts (xy 90.17 120.65) (xy 90.17 115.57)) (stroke (width 0) (type default)))
@@
 (wire (pts (xy 199.39 90.17) (xy 204.47 90.17)) (stroke (width 0) (type default)))
 (global_label "PANEL_5V" (shape bidirectional) (at 204.47 90.17 0) (effects (font (size 0.9 0.9)) (justify left)) (property "Intersheetrefs" "" (at 204.47 90.17 0) (effects (font (size 1 1)) (hide yes))))
-(symbol (lib_id "Regulator_Linear:AP2112K-3.3") (at 265.43 59.69 0) (unit 1) (in_bom yes) (on_board yes) (dnp no) (property "Reference" "U4" (at 265.43 45.69 0) (effects (font (size 1.2 1.2)))) (property "Value" "AP2112K-3.3TRG1" (at 265.43 47.69 0) (effects (font (size 1.1 1.1)))) (property "Footprint" "Package_TO_SOT_SMD:SOT-23-5" (at 265.43 59.69 0) (effects (font (size 1 1)) (hide yes))) (pin "1") (pin "2") (pin "3") (pin "4") (pin "5") (instances (project "usb-scoring-platform" (path "/20cc8167-128c-446a-a106-f942323e143f/36d13c9b-c278-4925-a3f2-4480b5a41043" (reference "U4") (unit 1)))))
+(symbol (lib_id "Regulator_Linear:AP2112K-3.3") (at 265.43 59.69 0) (unit 1) (in_bom yes) (on_board yes) (dnp no) (property "Reference" "U4" (at 265.43 45.69 0) (effects (font (size 1.2 1.2)))) (property "Value" "AP2112K-3.3TRG1" (at 265.43 47.69 0) (effects (font (size 1.1 1.1)))) (property "Footprint" "Package_TO_SOT_SMD:SOT-23-5" (at 265.43 59.69 0) (effects (font (size 1 1)) (hide yes))) (pin "1") (pin "2") (pin "3") (pin "4") (pin "5") (instances (project "usb-scoring-platform" (path "/20cc8167-128c-446a-a106-f942323e143f/36d13c9b-c278-4925-a3f2-4480b5a41043" (reference "U4") (unit 1)))) (property "Manufacturer" "Diodes Incorporated" (at 0 0 0) (effects (font (size 1 1)) (hide yes))) (property "MPN" "AP2112K-3.3TRG1" (at 0 0 0) (effects (font (size 1 1)) (hide yes))))
 (wire (pts (xy 257.81 57.15) (xy 252.73 57.15)) (stroke (width 0) (type default)))
 (global_label "CORE_5V" (shape bidirectional) (at 252.73 57.15 180) (effects (font (size 0.9 0.9)) (justify right)) (property "Intersheetrefs" "" (at 252.73 57.15 180) (effects (font (size 1 1)) (hide yes))))
@@
 (global_label "GND" (shape bidirectional) (at 379.73 58.42 0) (effects (font (size 0.9 0.9)) (justify left)) (property "Intersheetrefs" "" (at 379.73 58.42 0) (effects (font (size 1 1)) (hide yes))))
 (text "D1/D2 OR the isolated USB supply and PD-derived 5V without backfeeding either source. PB5 senses only the isolated side." (at 195 135 0) (effects (font (size 0.95 0.95)) (justify left top)))
-(symbol (lib_id "Regulator_Switching:AP63203WU") (at 255.27 175.26 0) (unit 1) (in_bom yes) (on_board yes) (dnp no) (property "Reference" "U7" (at 255.27 161.26 0) (effects (font (size 1.2 1.2)))) (property "Value" "AP63203WU-7" (at 255.27 163.26 0) (effects (font (size 1.1 1.1)))) (property "Footprint" "Package_TO_SOT_SMD:TSOT-23-6" (at 255.27 175.26 0) (effects (font (size 1 1)) (hide yes))) (pin "1") (pin "2") (pin "3") (pin "4") (pin "5") (pin "6") (instances (project "usb-scoring-platform" (path "/20cc8167-128c-446a-a106-f942323e143f/36d13c9b-c278-4925-a3f2-4480b5a41043" (reference "U7") (unit 1)))))
+(symbol (lib_id "Regulator_Switching:AP63203WU") (at 255.27 175.26 0) (unit 1) (in_bom yes) (on_board yes) (dnp no) (property "Reference" "U7" (at 255.27 161.26 0) (effects (font (size 1.2 1.2)))) (property "Value" "AP63203WU-7" (at 255.27 163.26 0) (effects (font (size 1.1 1.1)))) (property "Footprint" "Package_TO_SOT_SMD:TSOT-23-6" (at 255.27 175.26 0) (effects (font (size 1 1)) (hide yes))) (pin "1") (pin "2") (pin "3") (pin "4") (pin "5") (pin "6") (instances (project "usb-scoring-platform" (path "/20cc8167-128c-446a-a106-f942323e143f/36d13c9b-c278-4925-a3f2-4480b5a41043" (reference "U7") (unit 1)))) (property "Manufacturer" "Diodes Incorporated" (at 0 0 0) (effects (font (size 1 1)) (hide yes))) (property "MPN" "AP63203WU-7" (at 0 0 0) (effects (font (size 1 1)) (hide yes))))
 (wire (pts (xy 265.43 177.8) (xy 270.51 177.8)) (stroke (width 0) (type default)))
 (global_label "APP_3V3" (shape bidirectional) (at 270.51 177.8 0) (effects (font (size 0.9 0.9)) (justify left)) (property "Intersheetrefs" "" (at 270.51 177.8 0) (effects (font (size 1 1)) (hide yes))))

Commit message: fix(scoring-circuit): source stocked bypass and reservoir capacitors
Parts:
- C4: MPN C1608X7R1H104K080AA -> CC0603KRX7R9BB104; Manufacturer TDK -> Yageo
Changed lines of the file:
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@@
 (wire (pts (xy 320.04 179.07) (xy 320.04 184.15)) (stroke (width 0) (type default)))
 (global_label "APP_3V3" (shape bidirectional) (at 320.04 184.15 0) (effects (font (size 0.9 0.9)) (justify left)) (property "Intersheetrefs" "" (at 320.04 184.15 0) (effects (font (size 1 1)) (hide yes))))
-(symbol (lib_id "Device:C") (at 255.27 219.71 0) (unit 1) (in_bom yes) (on_board yes) (dnp no) (property "Reference" "C4" (at 255.27 205.71 0) (effects (font (size 1.2 1.2)))) (property "Value" "100nF 16V" (at 255.27 207.71 0) (effects (font (size 1.1 1.1)))) (property "Footprint" "Capacitor_SMD:C_0603_1608Metric" (at 255.27 219.71 0) (effects (font (size 1 1)) (hide yes))) (pin "1") (pin "2") (property "Manufacturer" "TDK" (at 255.27 219.71 0) (effects (font (size 1 1)) (hide yes))) (property "MPN" "C1608X7R1H104K080AA" (at 255.27 219.71 0) (effects (font (size 1 1)) (hide yes))) (property "Datasheet" "https://product.tdk.com/en/search/capacitor/ceramic/mlcc/info?part_no=C1608X7R1H104K080AA" (at 255.27 219.71 0) (effects (font (size 1 1)) (hide yes))) (instances (project "usb-scoring-platform" (path "/20cc8167-128c-446a-a106-f942323e143f/36d13c9b-c278-4925-a3f2-4480b5a41043" (reference "C4") (unit 1)))))
+(symbol (lib_id "Device:C") (at 255.27 219.71 0) (unit 1) (in_bom yes) (on_board yes) (dnp no) (property "Reference" "C4" (at 255.27 205.71 0) (effects (font (size 1.2 1.2)))) (property "Value" "100nF 16V" (at 255.27 207.71 0) (effects (font (size 1.1 1.1)))) (property "Footprint" "Capacitor_SMD:C_0603_1608Metric" (at 255.27 219.71 0) (effects (font (size 1 1)) (hide yes))) (pin "1") (pin "2") (property "Manufacturer" "Yageo" (at 255.27 219.71 0) (effects (font (size 1 1)) (hide yes))) (property "MPN" "CC0603KRX7R9BB104" (at 255.27 219.71 0) (effects (font (size 1 1)) (hide yes))) (property "Datasheet" "https://www.yageogroup.com/download/specsheet/CC0603KRX7R9BB104" (at 255.27 219.71 0) (effects (font (size 1 1)) (hide yes))) (instances (project "usb-scoring-platform" (path "/20cc8167-128c-446a-a106-f942323e143f/36d13c9b-c278-4925-a3f2-4480b5a41043" (reference "C4") (unit 1)))))
 (wire (pts (xy 255.27 215.9) (xy 255.27 210.82)) (stroke (width 0) (type default)))
 (global_label "BUCK_BOOT" (shape bidirectional) (at 255.27 210.82 0) (effects (font (size 0.9 0.9)) (justify left)) (property "Intersheetrefs" "" (at 255.27 210.82 0) (effects (font (size 1 1)) (hide yes))))
