File: packages/scoring-circuit/usb-scoring-platform/acquisition-controller.kicad_sch (KiCad schematic)
At the start: 19 parts, among them J2 STM SWD 3.3V, SW1 STM RESET, U1 STM32G474RET6, Y1 ABM3B-8.000MHZ-B2-T

Commit message: feat(scoring-circuit): select bypass and timing capacitors
Parts:
- C10, C11, C13, C16, C34, C8, C9: MPN (none) -> C1608X7R1H104K080AA; Manufacturer (none) -> TDK
- C12: MPN (none) -> C1608X7R1H103K080AA; Manufacturer (none) -> TDK
- C17, C18: MPN (none) -> CGA3E2C0G1H270J080AA; Manufacturer (none) -> TDK

Commit message: feat(scoring-circuit): select local supply capacitors
Parts:
- C15, C33: MPN (none) -> C1608X7R1H105K080AB; Manufacturer (none) -> TDK
