File: packages/scoring-circuit/usb-scoring-platform/acquisition-controller.kicad_sch (KiCad schematic)
At the start: 19 parts, among them J2 STM SWD 3.3V, SW1 STM RESET, U1 STM32G474RET6, Y1 ABM3B-8.000MHZ-B2-T

Commit message: feat(scoring-circuit): complete nominal capacitor selections
Parts:
- C14: MPN (none) -> C1608X7S1A475K080AC; Manufacturer (none) -> TDK

Commit message: chore(scoring-circuit): select reset and boot service buttons
Parts:
- SW1: MPN (none) -> TL3342F160QG; Manufacturer (none) -> E-Switch

Commit message: chore(scoring-circuit): bind crystal and peripheral ordering details
Parts:
- Y1: MPN (none) -> ABM3B-8.000MHZ-B2-T; Manufacturer (none) -> Abracon

Commit message: fix(scoring-circuit): select service headers and correct drill sizes
Parts:
- J2: footprint Connector_PinHeader_2.54mm:PinHeader_1x05_P2.54mm_Vertical -> ScoringPlatform:Samtec_HTSW-105-07-L-S; MPN (none) -> HTSW-105-07-L-S; Manufacturer (none) -> Samtec

Commit message: chore(scoring-circuit): complete assembly BOM ordering fields
Parts:
- U1: MPN (none) -> STM32G474RET6; Manufacturer (none) -> STMicroelectronics

Commit message: fix(scoring-circuit): source stocked bypass and reservoir capacitors
Parts:
- C10, C11, C13, C16, C34, C8, C9: MPN C1608X7R1H104K080AA -> CC0603KRX7R9BB104; Manufacturer TDK -> Yageo
