File: packages/scoring-circuit/usb-scoring-platform/application-controller.kicad_sch (KiCad schematic)
At the start: 17 parts, among them J6 ESP 3.3V UART recovery, SW2 ESP RESET, SW3 ESP BOOT, U10 SN74AXC1T45DCKR, U11 SN74AXC1T45DCKR, U2 ESP32-S3-WROOM-1-N8R8

Commit message: feat(scoring-circuit): route reset-safe processor UART link
Parts:
- added R72, R73: 10k 1%, Resistor_SMD:R_0603_1608Metric, symbol Device:R
Connections:
- net APP_3V3: now also R73.1
- net CORE_3V3: now also R72.1
- net ESP_TX: now also R73.2
- net STM_TX: now also R72.2
Other:
- note added: "R72/R73 hold each transmitter high during reset; R30/R31 keep receivers idle when the opposite rail is off. Each pull references its own processor supply."

Commit message: feat(scoring-circuit): select exact prototype resistor parts
Parts:
- R28, R29, R72, R73: MPN (none) -> RC0603FR-0710KL; Manufacturer (none) -> YAGEO
- R30, R31: MPN (none) -> RC0603FR-0747KL; Manufacturer (none) -> YAGEO

Commit message: feat(scoring-circuit): select bypass and timing capacitors
Parts:
- C23, C24, C25, C26, C27: MPN (none) -> C1608X7R1H104K080AA; Manufacturer (none) -> TDK

Commit message: feat(scoring-circuit): select local supply capacitors
Parts:
- C21: MPN (none) -> C1608X7R1H105K080AB; Manufacturer (none) -> TDK
Changed lines of the file:
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@@
 (wire (pts (xy 160.02 48.26) (xy 160.02 53.34)) (stroke (width 0) (type default)))
 (global_label "ESP_EN" (shape bidirectional) (at 160.02 53.34 0) (effects (font (size 0.9 0.9)) (justify left)) (property "Intersheetrefs" "" (at 160.02 53.34 0) (effects (font (size 1 1)) (hide yes))))
-(symbol (lib_id "Device:C") (at 199.39 44.45 0) (unit 1) (in_bom yes) (on_board yes) (dnp no) (property "Reference" "C21" (at 199.39 30.45 0) (effects (font (size 1.2 1.2)))) (property "Value" "1uF 10V" (at 199.39 32.45 0) (effects (font (size 1.1 1.1)))) (property "Footprint" "Capacitor_SMD:C_0603_1608Metric" (at 199.39 44.45 0) (effects (font (size 1 1)) (hide yes))) (pin "1") (pin "2") (instances (project "usb-scoring-platform" (path "/20cc8167-128c-446a-a106-f942323e143f/97185045-65e6-4b5b-a06d-6bdd67041229" (reference "C21") (unit 1)))))
+(symbol (lib_id "Device:C") (at 199.39 44.45 0) (unit 1) (in_bom yes) (on_board yes) (dnp no) (property "Reference" "C21" (at 199.39 30.45 0) (effects (font (size 1.2 1.2)))) (property "Value" "1uF 10V" (at 199.39 32.45 0) (effects (font (size 1.1 1.1)))) (property "Footprint" "Capacitor_SMD:C_0603_1608Metric" (at 199.39 44.45 0) (effects (font (size 1 1)) (hide yes))) (pin "1") (pin "2") (property "Manufacturer" "TDK" (at 199.39 44.45 0) (effects (font (size 1 1)) (hide yes))) (property "MPN" "C1608X7R1H105K080AB" (at 199.39 44.45 0) (effects (font (size 1 1)) (hide yes))) (property "Datasheet" "https://product.tdk.com/en/search/capacitor/ceramic/mlcc/info?part_no=C1608X7R1H105K080AB" (at 199.39 44.45 0) (effects (font (size 1 1)) (hide yes))) (instances (project "usb-scoring-platform" (path "/20cc8167-128c-446a-a106-f942323e143f/97185045-65e6-4b5b-a06d-6bdd67041229" (reference "C21") (unit 1)))))
 (wire (pts (xy 199.39 40.64) (xy 199.39 35.56)) (stroke (width 0) (type default)))
 (global_label "ESP_EN" (shape bidirectional) (at 199.39 35.56 0) (effects (font (size 0.9 0.9)) (justify left)) (property "Intersheetrefs" "" (at 199.39 35.56 0) (effects (font (size 1 1)) (hide yes))))

Commit message: feat(scoring-circuit): complete nominal capacitor selections
Parts:
- C22: MPN (none) -> C1608X5R1C106M080AB; Manufacturer (none) -> TDK
Changed lines of the file:
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@@
 (wire (pts (xy 240.03 48.26) (xy 240.03 53.34)) (stroke (width 0) (type default)))
 (global_label "ESP_BOOT0" (shape bidirectional) (at 240.03 53.34 0) (effects (font (size 0.9 0.9)) (justify left)) (property "Intersheetrefs" "" (at 240.03 53.34 0) (effects (font (size 1 1)) (hide yes))))
-(symbol (lib_id "Device:C") (at 160.02 90.17 0) (unit 1) (in_bom yes) (on_board yes) (dnp no) (property "Reference" "C22" (at 160.02 76.17 0) (effects (font (size 1.2 1.2)))) (property "Value" "10uF 10V" (at 160.02 78.17 0) (effects (font (size 1.1 1.1)))) (property "Footprint" "Capacitor_SMD:C_0603_1608Metric" (at 160.02 90.17 0) (effects (font (size 1 1)) (hide yes))) (pin "1") (pin "2") (instances (project "usb-scoring-platform" (path "/20cc8167-128c-446a-a106-f942323e143f/97185045-65e6-4b5b-a06d-6bdd67041229" (reference "C22") (unit 1)))))
+(symbol (lib_id "Device:C") (at 160.02 90.17 0) (unit 1) (in_bom yes) (on_board yes) (dnp no) (property "Reference" "C22" (at 160.02 76.17 0) (effects (font (size 1.2 1.2)))) (property "Value" "10uF 10V" (at 160.02 78.17 0) (effects (font (size 1.1 1.1)))) (property "Footprint" "Capacitor_SMD:C_0603_1608Metric" (at 160.02 90.17 0) (effects (font (size 1 1)) (hide yes))) (pin "1") (pin "2") (property "Manufacturer" "TDK" (at 0 0 0) (effects (font (size 1 1)) (hide yes))) (property "MPN" "C1608X5R1C106M080AB" (at 0 0 0) (effects (font (size 1 1)) (hide yes))) (property "Datasheet" "https://product.tdk.com/en/search/capacitor/ceramic/mlcc/info?part_no=C1608X5R1C106M080AB" (at 0 0 0) (effects (font (size 1 1)) (hide yes))) (instances (project "usb-scoring-platform" (path "/20cc8167-128c-446a-a106-f942323e143f/97185045-65e6-4b5b-a06d-6bdd67041229" (reference "C22") (unit 1)))))
 (wire (pts (xy 160.02 86.36) (xy 160.02 81.28)) (stroke (width 0) (type default)))
 (global_label "APP_3V3" (shape bidirectional) (at 160.02 81.28 0) (effects (font (size 0.9 0.9)) (justify left)) (property "Intersheetrefs" "" (at 160.02 81.28 0) (effects (font (size 1 1)) (hide yes))))

Commit message: chore(scoring-circuit): select reset and boot service buttons
Parts:
- SW2, SW3: MPN (none) -> TL3342F160QG; Manufacturer (none) -> E-Switch
Changed lines of the file:
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@@
 (wire (pts (xy 204.47 93.98) (xy 204.47 99.06)) (stroke (width 0) (type default)))
 (global_label "GND" (shape bidirectional) (at 204.47 99.06 0) (effects (font (size 0.9 0.9)) (justify left)) (property "Intersheetrefs" "" (at 204.47 99.06 0) (effects (font (size 1 1)) (hide yes))))
-(symbol (lib_id "Switch:SW_Push") (at 279.4 74.93 0) (unit 1) (in_bom yes) (on_board yes) (dnp no) (property "Reference" "SW2" (at 279.4 60.93 0) (effects (font (size 1.2 1.2)))) (property "Value" "ESP RESET" (at 279.4 62.93 0) (effects (font (size 1.1 1.1)))) (property "Footprint" "Button_Switch_SMD:SW_SPST_TL3342" (at 279.4 74.93 0) (effects (font (size 1 1)) (hide yes))) (pin "1") (pin "2") (instances (project "usb-scoring-platform" (path "/20cc8167-128c-446a-a106-f942323e143f/97185045-65e6-4b5b-a06d-6bdd67041229" (reference "SW2") (unit 1)))))
+(symbol (lib_id "Switch:SW_Push") (at 279.4 74.93 0) (unit 1) (in_bom yes) (on_board yes) (dnp no) (property "Reference" "SW2" (at 279.4 60.93 0) (effects (font (size 1.2 1.2)))) (property "Value" "ESP RESET" (at 279.4 62.93 0) (effects (font (size 1.1 1.1)))) (property "Footprint" "Button_Switch_SMD:SW_SPST_TL3342" (at 279.4 74.93 0) (effects (font (size 1 1)) (hide yes))) (pin "1") (pin "2") (instances (project "usb-scoring-platform" (path "/20cc8167-128c-446a-a106-f942323e143f/97185045-65e6-4b5b-a06d-6bdd67041229" (reference "SW2") (unit 1)))) (property "Manufacturer" "E-Switch" (at 0 0 0) (effects (font (size 1 1)) (hide yes))) (property "MPN" "TL3342F160QG" (at 0 0 0) (effects (font (size 1 1)) (hide yes))) (property "Datasheet" "https://configured-product-images.s3.amazonaws.com/2D/specs/TL3342F160QG.pdf" (at 0 0 0) (effects (font (size 1 1)) (hide yes))))
 (wire (pts (xy 274.32 74.93) (xy 269.24 74.93)) (stroke (width 0) (type default)))
 (global_label "ESP_EN" (shape bidirectional) (at 269.24 74.93 180) (effects (font (size 0.9 0.9)) (justify right)) (property "Intersheetrefs" "" (at 269.24 74.93 180) (effects (font (size 1 1)) (hide yes))))
 (wire (pts (xy 284.48 74.93) (xy 289.56 74.93)) (stroke (width 0) (type default)))
 (global_label "GND" (shape bidirectional) (at 289.56 74.93 0) (effects (font (size 0.9 0.9)) (justify left)) (property "Intersheetrefs" "" (at 289.56 74.93 0) (effects (font (size 1 1)) (hide yes))))
-(symbol (lib_id "Switch:SW_Push") (at 350.52 74.93 0) (unit 1) (in_bom yes) (on_board yes) (dnp no) (property "Reference" "SW3" (at 350.52 60.93 0) (effects (font (size 1.2 1.2)))) (property "Value" "ESP BOOT" (at 350.52 62.93 0) (effects (font (size 1.1 1.1)))) (property "Footprint" "Button_Switch_SMD:SW_SPST_TL3342" (at 350.52 74.93 0) (effects (font (size 1 1)) (hide yes))) (pin "1") (pin "2") (instances (project "usb-scoring-platform" (path "/20cc8167-128c-446a-a106-f942323e143f/97185045-65e6-4b5b-a06d-6bdd67041229" (reference "SW3") (unit 1)))))
+(symbol (lib_id "Switch:SW_Push") (at 350.52 74.93 0) (unit 1) (in_bom yes) (on_board yes) (dnp no) (property "Reference" "SW3" (at 350.52 60.93 0) (effects (font (size 1.2 1.2)))) (property "Value" "ESP BOOT" (at 350.52 62.93 0) (effects (font (size 1.1 1.1)))) (property "Footprint" "Button_Switch_SMD:SW_SPST_TL3342" (at 350.52 74.93 0) (effects (font (size 1 1)) (hide yes))) (pin "1") (pin "2") (instances (project "usb-scoring-platform" (path "/20cc8167-128c-446a-a106-f942323e143f/97185045-65e6-4b5b-a06d-6bdd67041229" (reference "SW3") (unit 1)))) (property "Manufacturer" "E-Switch" (at 0 0 0) (effects (font (size 1 1)) (hide yes))) (property "MPN" "TL3342F160QG" (at 0 0 0) (effects (font (size 1 1)) (hide yes))) (property "Datasheet" "https://configured-product-images.s3.amazonaws.com/2D/specs/TL3342F160QG.pdf" (at 0 0 0) (effects (font (size 1 1)) (hide yes))))
 (wire (pts (xy 345.44 74.93) (xy 340.36 74.93)) (stroke (width 0) (type default)))
 (global_label "ESP_BOOT0" (shape bidirectional) (at 340.36 74.93 180) (effects (font (size 0.9 0.9)) (justify right)) (property "Intersheetrefs" "" (at 340.36 74.93 180) (effects (font (size 1 1)) (hide yes))))

Commit message: fix(scoring-circuit): select service headers and correct drill sizes
Parts:
- J6: footprint Connector_PinHeader_2.54mm:PinHeader_1x06_P2.54mm_Vertical -> ScoringPlatform:Samtec_HTSW-106-07-L-S; MPN (none) -> HTSW-106-07-L-S; Manufacturer (none) -> Samtec
Changed lines of the file:
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@@
 (wire (pts (xy 355.6 74.93) (xy 360.68 74.93)) (stroke (width 0) (type default)))
 (global_label "GND" (shape bidirectional) (at 360.68 74.93 0) (effects (font (size 0.9 0.9)) (justify left)) (property "Intersheetrefs" "" (at 360.68 74.93 0) (effects (font (size 1 1)) (hide yes))))
-(symbol (lib_id "Connector_Generic:Conn_01x06") (at 320.04 129.54 0) (unit 1) (in_bom yes) (on_board yes) (dnp no) (property "Reference" "J6" (at 320.04 115.46 0) (effects (font (size 1.2 1.2)))) (property "Value" "ESP 3.3V UART recovery" (at 320.04 117.46 0) (effects (font (size 1.1 1.1)))) (property "Footprint" "Connector_PinHeader_2.54mm:PinHeader_1x06_P2.54mm_Vertical" (at 320.04 129.54 0) (effects (font (size 1 1)) (hide yes))) (pin "1") (pin "2") (pin "3") (pin "4") (pin "5") (pin "6") (instances (project "usb-scoring-platform" (path "/20cc8167-128c-446a-a106-f942323e143f/97185045-65e6-4b5b-a06d-6bdd67041229" (reference "J6") (unit 1)))))
+(symbol (lib_id "Connector_Generic:Conn_01x06") (at 320.04 129.54 0) (unit 1) (in_bom yes) (on_board yes) (dnp no) (property "Reference" "J6" (at 320.04 115.46 0) (effects (font (size 1.2 1.2)))) (property "Value" "ESP 3.3V UART recovery" (at 320.04 117.46 0) (effects (font (size 1.1 1.1)))) (property "Footprint" "ScoringPlatform:Samtec_HTSW-106-07-L-S" (at 320.04 129.54 0) (effects (font (size 1 1)) (hide yes))) (pin "1") (pin "2") (pin "3") (pin "4") (pin "5") (pin "6") (instances (project "usb-scoring-platform" (path "/20cc8167-128c-446a-a106-f942323e143f/97185045-65e6-4b5b-a06d-6bdd67041229" (reference "J6") (unit 1)))) (property "Datasheet" "https://suddendocs.samtec.com/prints/htsw-xxx-xx-xxx-x-xx-xx-xx-mkt.pdf" (at 0 0 0) (effects (font (size 1 1)) (hide yes))) (property "Manufacturer" "Samtec" (at 0 0 0) (effects (font (size 1 1)) (hide yes))) (property "MPN" "HTSW-106-07-L-S" (at 0 0 0) (effects (font (size 1 1)) (hide yes))))
 (wire (pts (xy 314.96 124.46) (xy 309.88 124.46)) (stroke (width 0) (type default)))
 (global_label "APP_3V3" (shape bidirectional) (at 309.88 124.46 180) (effects (font (size 0.9 0.9)) (justify right)) (property "Intersheetrefs" "" (at 309.88 124.46 180) (effects (font (size 1 1)) (hide yes))))

Commit message: chore(scoring-circuit): complete assembly BOM ordering fields
Parts:
- U10, U11: MPN (none) -> SN74AXC1T45DCKR; Manufacturer (none) -> Texas Instruments
- U2: MPN (none) -> ESP32-S3-WROOM-1-N8R8; Manufacturer (none) -> Espressif Systems
Changed lines of the file:
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@@
 (paper "A3")
 (title_block (title "ESP32 display, IR and network controller") (rev "Engineering draft") (comment 1 "NOT FOR FABRICATION"))
-(symbol (lib_id "RF_Module:ESP32-S3-WROOM-1") (at 80.01 100.33 0) (unit 1) (in_bom yes) (on_board yes) (dnp no) (property "Reference" "U2" (at 80.01 63.39 0) (effects (font (size 1.2 1.2)))) (property "Value" "ESP32-S3-WROOM-1-N8R8" (at 80.01 65.39 0) (effects (font (size 1.1 1.1)))) (property "Footprint" "RF_Module:ESP32-S3-WROOM-1" (at 80.01 100.33 0) (effects (font (size 1 1)) (hide yes))) (pin "1") (pin "2") (pin "3") (pin "4") (pin "5") (pin "6") (pin "7") (pin "8") (pin "9") (pin "10") (pin "11") (pin "12") (pin "13") (pin "14") (pin "15") (pin "16") (pin "17") (pin "18") (pin "19") (pin "20") (pin "21") (pin "22") (pin "23") (pin "24") (pin "25") (pin "26") (pin "27") (pin "28") (pin "29") (pin "30") (pin "31") (pin "32") (pin "33") (pin "34") (pin "35") (pin "36") (pin "37") (pin "38") (pin "39") (pin "40") (pin "41") (instances (project "usb-scoring-platform" (path "/20cc8167-128c-446a-a106-f942323e143f/97185045-65e6-4b5b-a06d-6bdd67041229" (reference "U2") (unit 1)))))
+(symbol (lib_id "RF_Module:ESP32-S3-WROOM-1") (at 80.01 100.33 0) (unit 1) (in_bom yes) (on_board yes) (dnp no) (property "Reference" "U2" (at 80.01 63.39 0) (effects (font (size 1.2 1.2)))) (property "Value" "ESP32-S3-WROOM-1-N8R8" (at 80.01 65.39 0) (effects (font (size 1.1 1.1)))) (property "Footprint" "RF_Module:ESP32-S3-WROOM-1" (at 80.01 100.33 0) (effects (font (size 1 1)) (hide yes))) (pin "1") (pin "2") (pin "3") (pin "4") (pin "5") (pin "6") (pin "7") (pin "8") (pin "9") (pin "10") (pin "11") (pin "12") (pin "13") (pin "14") (pin "15") (pin "16") (pin "17") (pin "18") (pin "19") (pin "20") (pin "21") (pin "22") (pin "23") (pin "24") (pin "25") (pin "26") (pin "27") (pin "28") (pin "29") (pin "30") (pin "31") (pin "32") (pin "33") (pin "34") (pin "35") (pin "36") (pin "37") (pin "38") (pin "39") (pin "40") (pin "41") (instances (project "usb-scoring-platform" (path "/20cc8167-128c-446a-a106-f942323e143f/97185045-65e6-4b5b-a06d-6bdd67041229" (reference "U2") (unit 1)))) (property "Manufacturer" "Espressif Systems" (at 0 0 0) (effects (font (size 1 1)) (hide yes))) (property "MPN" "ESP32-S3-WROOM-1-N8R8" (at 0 0 0) (effects (font (size 1 1)) (hide yes))))
 (wire (pts (xy 80.01 128.27) (xy 80.01 133.35)) (stroke (width 0) (type default)))
 (global_label "GND" (shape bidirectional) (at 80.01 133.35 0) (effects (font (size 0.9 0.9)) (justify left)) (property "Intersheetrefs" "" (at 80.01 133.35 0) (effects (font (size 1 1)) (hide yes))))
@@
 (wire (pts (xy 314.96 137.16) (xy 309.88 137.16)) (stroke (width 0) (type default)))
 (global_label "ESP_BOOT0" (shape bidirectional) (at 309.88 137.16 180) (effects (font (size 0.9 0.9)) (justify right)) (property "Intersheetrefs" "" (at 309.88 137.16 180) (effects (font (size 1 1)) (hide yes))))
-(symbol (lib_id "ScoringPlatform:SN74AXC1T45DCKR") (at 80.01 195.58 0) (unit 1) (in_bom yes) (on_board yes) (dnp no) (property "Reference" "U10" (at 80.01 181.58 0) (effects (font (size 1.2 1.2)))) (property "Value" "SN74AXC1T45DCKR" (at 80.01 183.58 0) (effects (font (size 1.1 1.1)))) (property "Footprint" "Package_TO_SOT_SMD:SOT-363_SC-70-6" (at 80.01 195.58 0) (effects (font (size 1 1)) (hide yes))) (pin "1") (pin "2") (pin "3") (pin "4") (pin "5") (pin "6") (instances (project "usb-scoring-platform" (path "/20cc8167-128c-446a-a106-f942323e143f/97185045-65e6-4b5b-a06d-6bdd67041229" (reference "U10") (unit 1)))))
+(symbol (lib_id "ScoringPlatform:SN74AXC1T45DCKR") (at 80.01 195.58 0) (unit 1) (in_bom yes) (on_board yes) (dnp no) (property "Reference" "U10" (at 80.01 181.58 0) (effects (font (size 1.2 1.2)))) (property "Value" "SN74AXC1T45DCKR" (at 80.01 183.58 0) (effects (font (size 1.1 1.1)))) (property "Footprint" "Package_TO_SOT_SMD:SOT-363_SC-70-6" (at 80.01 195.58 0) (effects (font (size 1 1)) (hide yes))) (pin "1") (pin "2") (pin "3") (pin "4") (pin "5") (pin "6") (instances (project "usb-scoring-platform" (path "/20cc8167-128c-446a-a106-f942323e143f/97185045-65e6-4b5b-a06d-6bdd67041229" (reference "U10") (unit 1)))) (property "Manufacturer" "Texas Instruments" (at 0 0 0) (effects (font (size 1 1)) (hide yes))) (property "MPN" "SN74AXC1T45DCKR" (at 0 0 0) (effects (font (size 1 1)) (hide yes))))
 (wire (pts (xy 62.23 193.04) (xy 57.15 193.04)) (stroke (width 0) (type default)))
 (global_label "CORE_3V3" (shape bidirectional) (at 57.15 193.04 180) (effects (font (size 0.9 0.9)) (justify right)) (property "Intersheetrefs" "" (at 57.15 193.04 180) (effects (font (size 1 1)) (hide yes))))
@@
 (wire (pts (xy 110.49 243.84) (xy 110.49 248.92)) (stroke (width 0) (type default)))
 (global_label "GND" (shape bidirectional) (at 110.49 248.92 0) (effects (font (size 0.9 0.9)) (justify left)) (property "Intersheetrefs" "" (at 110.49 248.92 0) (effects (font (size 1 1)) (hide yes))))
-(symbol (lib_id "ScoringPlatform:SN74AXC1T45DCKR") (at 229.87 195.58 0) (unit 1) (in_bom yes) (on_board yes) (dnp no) (property "Reference" "U11" (at 229.87 181.58 0) (effects (font (size 1.2 1.2)))) (property "Value" "SN74AXC1T45DCKR" (at 229.87 183.58 0) (effects (font (size 1.1 1.1)))) (property "Footprint" "Package_TO_SOT_SMD:SOT-363_SC-70-6" (at 229.87 195.58 0) (effects (font (size 1 1)) (hide yes))) (pin "1") (pin "2") (pin "3") (pin "4") (pin "5") (pin "6") (instances (project "usb-scoring-platform" (path "/20cc8167-128c-446a-a106-f942323e143f/97185045-65e6-4b5b-a06d-6bdd67041229" (reference "U11") (unit 1)))))
+(symbol (lib_id "ScoringPlatform:SN74AXC1T45DCKR") (at 229.87 195.58 0) (unit 1) (in_bom yes) (on_board yes) (dnp no) (property "Reference" "U11" (at 229.87 181.58 0) (effects (font (size 1.2 1.2)))) (property "Value" "SN74AXC1T45DCKR" (at 229.87 183.58 0) (effects (font (size 1.1 1.1)))) (property "Footprint" "Package_TO_SOT_SMD:SOT-363_SC-70-6" (at 229.87 195.58 0) (effects (font (size 1 1)) (hide yes))) (pin "1") (pin "2") (pin "3") (pin "4") (pin "5") (pin "6") (instances (project "usb-scoring-platform" (path "/20cc8167-128c-446a-a106-f942323e143f/97185045-65e6-4b5b-a06d-6bdd67041229" (reference "U11") (unit 1)))) (property "Manufacturer" "Texas Instruments" (at 0 0 0) (effects (font (size 1 1)) (hide yes))) (property "MPN" "SN74AXC1T45DCKR" (at 0 0 0) (effects (font (size 1 1)) (hide yes))))
 (wire (pts (xy 212.09 193.04) (xy 207.01 193.04)) (stroke (width 0) (type default)))
 (global_label "CORE_3V3" (shape bidirectional) (at 207.01 193.04 180) (effects (font (size 0.9 0.9)) (justify right)) (property "Intersheetrefs" "" (at 207.01 193.04 180) (effects (font (size 1 1)) (hide yes))))
