File: packages/scoring-circuit/usb-scoring-platform/application-controller.kicad_sch (KiCad schematic)
At the start: 19 parts, among them J6 ESP 3.3V UART recovery, SW2 ESP RESET, SW3 ESP BOOT, U10 SN74AXC1T45DCKR, U11 SN74AXC1T45DCKR, U2 ESP32-S3-WROOM-1-N8R8

Commit message: fix(scoring): allow translator package body clearance
Parts:
- U10, U11: footprint Package_TO_SOT_SMD:SOT-363_SC-70-6 -> ScoringPlatform:SN74AXC1T45DCKR
Changed lines of the file:
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@@
 (wire (pts (xy 314.96 137.16) (xy 309.88 137.16)) (stroke (width 0) (type default)))
 (global_label "ESP_BOOT0" (shape bidirectional) (at 309.88 137.16 180) (effects (font (size 0.9 0.9)) (justify right)) (property "Intersheetrefs" "" (at 309.88 137.16 180) (effects (font (size 1 1)) (hide yes))))
-(symbol (lib_id "ScoringPlatform:SN74AXC1T45DCKR") (at 80.01 195.58 0) (unit 1) (in_bom yes) (on_board yes) (dnp no) (property "Reference" "U10" (at 80.01 181.58 0) (effects (font (size 1.2 1.2)))) (property "Value" "SN74AXC1T45DCKR" (at 80.01 183.58 0) (effects (font (size 1.1 1.1)))) (property "Footprint" "Package_TO_SOT_SMD:SOT-363_SC-70-6" (at 80.01 195.58 0) (effects (font (size 1 1)) (hide yes))) (pin "1") (pin "2") (pin "3") (pin "4") (pin "5") (pin "6") (instances (project "usb-scoring-platform" (path "/20cc8167-128c-446a-a106-f942323e143f/97185045-65e6-4b5b-a06d-6bdd67041229" (reference "U10") (unit 1)))) (property "Manufacturer" "Texas Instruments" (at 0 0 0) (effects (font (size 1 1)) (hide yes))) (property "MPN" "SN74AXC1T45DCKR" (at 0 0 0) (effects (font (size 1 1)) (hide yes))))
+(symbol (lib_id "ScoringPlatform:SN74AXC1T45DCKR") (at 80.01 195.58 0) (unit 1) (in_bom yes) (on_board yes) (dnp no) (property "Reference" "U10" (at 80.01 181.58 0) (effects (font (size 1.2 1.2)))) (property "Value" "SN74AXC1T45DCKR" (at 80.01 183.58 0) (effects (font (size 1.1 1.1)))) (property "Footprint" "ScoringPlatform:SN74AXC1T45DCKR" (at 80.01 195.58 0) (effects (font (size 1 1)) (hide yes))) (pin "1") (pin "2") (pin "3") (pin "4") (pin "5") (pin "6") (instances (project "usb-scoring-platform" (path "/20cc8167-128c-446a-a106-f942323e143f/97185045-65e6-4b5b-a06d-6bdd67041229" (reference "U10") (unit 1)))) (property "Manufacturer" "Texas Instruments" (at 0 0 0) (effects (font (size 1 1)) (hide yes))) (property "MPN" "SN74AXC1T45DCKR" (at 0 0 0) (effects (font (size 1 1)) (hide yes))))
 (wire (pts (xy 62.23 193.04) (xy 57.15 193.04)) (stroke (width 0) (type default)))
 (global_label "CORE_3V3" (shape bidirectional) (at 57.15 193.04 180) (effects (font (size 0.9 0.9)) (justify right)) (property "Intersheetrefs" "" (at 57.15 193.04 180) (effects (font (size 1 1)) (hide yes))))
@@
 (wire (pts (xy 110.49 243.84) (xy 110.49 248.92)) (stroke (width 0) (type default)))
 (global_label "GND" (shape bidirectional) (at 110.49 248.92 0) (effects (font (size 0.9 0.9)) (justify left)) (property "Intersheetrefs" "" (at 110.49 248.92 0) (effects (font (size 1 1)) (hide yes))))
-(symbol (lib_id "ScoringPlatform:SN74AXC1T45DCKR") (at 229.87 195.58 0) (unit 1) (in_bom yes) (on_board yes) (dnp no) (property "Reference" "U11" (at 229.87 181.58 0) (effects (font (size 1.2 1.2)))) (property "Value" "SN74AXC1T45DCKR" (at 229.87 183.58 0) (effects (font (size 1.1 1.1)))) (property "Footprint" "Package_TO_SOT_SMD:SOT-363_SC-70-6" (at 229.87 195.58 0) (effects (font (size 1 1)) (hide yes))) (pin "1") (pin "2") (pin "3") (pin "4") (pin "5") (pin "6") (instances (project "usb-scoring-platform" (path "/20cc8167-128c-446a-a106-f942323e143f/97185045-65e6-4b5b-a06d-6bdd67041229" (reference "U11") (unit 1)))) (property "Manufacturer" "Texas Instruments" (at 0 0 0) (effects (font (size 1 1)) (hide yes))) (property "MPN" "SN74AXC1T45DCKR" (at 0 0 0) (effects (font (size 1 1)) (hide yes))))
+(symbol (lib_id "ScoringPlatform:SN74AXC1T45DCKR") (at 229.87 195.58 0) (unit 1) (in_bom yes) (on_board yes) (dnp no) (property "Reference" "U11" (at 229.87 181.58 0) (effects (font (size 1.2 1.2)))) (property "Value" "SN74AXC1T45DCKR" (at 229.87 183.58 0) (effects (font (size 1.1 1.1)))) (property "Footprint" "ScoringPlatform:SN74AXC1T45DCKR" (at 229.87 195.58 0) (effects (font (size 1 1)) (hide yes))) (pin "1") (pin "2") (pin "3") (pin "4") (pin "5") (pin "6") (instances (project "usb-scoring-platform" (path "/20cc8167-128c-446a-a106-f942323e143f/97185045-65e6-4b5b-a06d-6bdd67041229" (reference "U11") (unit 1)))) (property "Manufacturer" "Texas Instruments" (at 0 0 0) (effects (font (size 1 1)) (hide yes))) (property "MPN" "SN74AXC1T45DCKR" (at 0 0 0) (effects (font (size 1 1)) (hide yes))))
 (wire (pts (xy 212.09 193.04) (xy 207.01 193.04)) (stroke (width 0) (type default)))
 (global_label "CORE_3V3" (shape bidirectional) (at 207.01 193.04 180) (effects (font (size 0.9 0.9)) (justify right)) (property "Intersheetrefs" "" (at 207.01 193.04 180) (effects (font (size 1 1)) (hide yes))))

Commit message: fix(scoring-circuit): source stocked bypass and reservoir capacitors
Parts:
- C23, C24, C25, C26, C27: MPN C1608X7R1H104K080AA -> CC0603KRX7R9BB104; Manufacturer TDK -> Yageo
