File: packages/scoring-circuit/usb-scoring-platform/favero-repeaters.kicad_sch (KiCad schematic)
At the start: 14 parts, among them J10 5520250-2, J9 5520250-2, Q3 DMN2056U-7, U16 4N32M, U17 4N32M

Commit message: chore(scoring-circuit): complete assembly BOM ordering fields
Parts:
- J10, J9: MPN (none) -> 5520250-2; Manufacturer (none) -> TE Connectivity
- U16, U17: MPN (none) -> 4N32M; Manufacturer (none) -> onsemi
Changed lines of the file:
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@@
 (paper "A3")
 (title_block (title "Two FA-05 DATA-LINE repeater outputs") (rev "Engineering draft") (comment 1 "NOT FOR FABRICATION"))
-(symbol (lib_id "ScoringPlatform:4N32M") (at 154.94 74.93 0) (unit 1) (in_bom yes) (on_board yes) (dnp no) (property "Reference" "U16" (at 154.94 60.93 0) (effects (font (size 1.2 1.2)))) (property "Value" "4N32M" (at 154.94 62.93 0) (effects (font (size 1.1 1.1)))) (property "Footprint" "ScoringPlatform:4N32M" (at 154.94 74.93 0) (effects (font (size 1 1)) (hide yes))) (pin "1") (pin "2") (pin "3") (pin "4") (pin "5") (pin "6") (instances (project "usb-scoring-platform" (path "/20cc8167-128c-446a-a106-f942323e143f/19a689f6-051a-47d6-a064-26f29b455422" (reference "U16") (unit 1)))))
+(symbol (lib_id "ScoringPlatform:4N32M") (at 154.94 74.93 0) (unit 1) (in_bom yes) (on_board yes) (dnp no) (property "Reference" "U16" (at 154.94 60.93 0) (effects (font (size 1.2 1.2)))) (property "Value" "4N32M" (at 154.94 62.93 0) (effects (font (size 1.1 1.1)))) (property "Footprint" "ScoringPlatform:4N32M" (at 154.94 74.93 0) (effects (font (size 1 1)) (hide yes))) (pin "1") (pin "2") (pin "3") (pin "4") (pin "5") (pin "6") (instances (project "usb-scoring-platform" (path "/20cc8167-128c-446a-a106-f942323e143f/19a689f6-051a-47d6-a064-26f29b455422" (reference "U16") (unit 1)))) (property "Manufacturer" "onsemi" (at 0 0 0) (effects (font (size 1 1)) (hide yes))) (property "MPN" "4N32M" (at 0 0 0) (effects (font (size 1 1)) (hide yes))))
 (wire (pts (xy 137.16 72.39) (xy 132.08 72.39)) (stroke (width 0) (type default)))
 (global_label "FAVERO1_LED" (shape bidirectional) (at 132.08 72.39 180) (effects (font (size 0.9 0.9)) (justify right)) (property "Intersheetrefs" "" (at 132.08 72.39 180) (effects (font (size 1 1)) (hide yes))))
@@
 (wire (pts (xy 172.72 77.47) (xy 177.8 77.47)) (stroke (width 0) (type default)))
 (global_label "FAVERO1_BASE" (shape bidirectional) (at 177.8 77.47 0) (effects (font (size 0.9 0.9)) (justify left)) (property "Intersheetrefs" "" (at 177.8 77.47 0) (effects (font (size 1 1)) (hide yes))))
-(symbol (lib_id "ScoringPlatform:TE_5520250_2") (at 335.28 74.93 0) (unit 1) (in_bom yes) (on_board yes) (dnp no) (property "Reference" "J9" (at 335.28 60.93 0) (effects (font (size 1.2 1.2)))) (property "Value" "5520250-2" (at 335.28 62.93 0) (effects (font (size 1.1 1.1)))) (property "Footprint" "ScoringPlatform:RJ14" (at 335.28 74.93 0) (effects (font (size 1 1)) (hide yes))) (pin "2") (pin "3") (pin "4") (pin "5") (instances (project "usb-scoring-platform" (path "/20cc8167-128c-446a-a106-f942323e143f/19a689f6-051a-47d6-a064-26f29b455422" (reference "J9") (unit 1)))))
+(symbol (lib_id "ScoringPlatform:TE_5520250_2") (at 335.28 74.93 0) (unit 1) (in_bom yes) (on_board yes) (dnp no) (property "Reference" "J9" (at 335.28 60.93 0) (effects (font (size 1.2 1.2)))) (property "Value" "5520250-2" (at 335.28 62.93 0) (effects (font (size 1.1 1.1)))) (property "Footprint" "ScoringPlatform:RJ14" (at 335.28 74.93 0) (effects (font (size 1 1)) (hide yes))) (pin "2") (pin "3") (pin "4") (pin "5") (instances (project "usb-scoring-platform" (path "/20cc8167-128c-446a-a106-f942323e143f/19a689f6-051a-47d6-a064-26f29b455422" (reference "J9") (unit 1)))) (property "Manufacturer" "TE Connectivity" (at 0 0 0) (effects (font (size 1 1)) (hide yes))) (property "MPN" "5520250-2" (at 0 0 0) (effects (font (size 1 1)) (hide yes))))
 (wire (pts (xy 317.5 72.39) (xy 312.42 72.39)) (stroke (width 0) (type default)))
 (global_label "FAVERO1_OUTER_A" (shape bidirectional) (at 312.42 72.39 180) (effects (font (size 0.9 0.9)) (justify right)) (property "Intersheetrefs" "" (at 312.42 72.39 180) (effects (font (size 1 1)) (hide yes))))
@@
 (wire (pts (xy 238.76 124.46) (xy 243.84 124.46)) (stroke (width 0) (type default)))
 (global_label "FAVERO1_EMITTER" (shape bidirectional) (at 243.84 124.46 0) (effects (font (size 0.9 0.9)) (justify left)) (property "Intersheetrefs" "" (at 243.84 124.46 0) (effects (font (size 1 1)) (hide yes))))
-(symbol (lib_id "ScoringPlatform:4N32M") (at 154.94 180.34 0) (unit 1) (in_bom yes) (on_board yes) (dnp no) (property "Reference" "U17" (at 154.94 166.34 0) (effects (font (size 1.2 1.2)))) (property "Value" "4N32M" (at 154.94 168.34 0) (effects (font (size 1.1 1.1)))) (property "Footprint" "ScoringPlatform:4N32M" (at 154.94 180.34 0) (effects (font (size 1 1)) (hide yes))) (pin "1") (pin "2") (pin "3") (pin "4") (pin "5") (pin "6") (instances (project "usb-scoring-platform" (path "/20cc8167-128c-446a-a106-f942323e143f/19a689f6-051a-47d6-a064-26f29b455422" (reference "U17") (unit 1)))))
+(symbol (lib_id "ScoringPlatform:4N32M") (at 154.94 180.34 0) (unit 1) (in_bom yes) (on_board yes) (dnp no) (property "Reference" "U17" (at 154.94 166.34 0) (effects (font (size 1.2 1.2)))) (property "Value" "4N32M" (at 154.94 168.34 0) (effects (font (size 1.1 1.1)))) (property "Footprint" "ScoringPlatform:4N32M" (at 154.94 180.34 0) (effects (font (size 1 1)) (hide yes))) (pin "1") (pin "2") (pin "3") (pin "4") (pin "5") (pin "6") (instances (project "usb-scoring-platform" (path "/20cc8167-128c-446a-a106-f942323e143f/19a689f6-051a-47d6-a064-26f29b455422" (reference "U17") (unit 1)))) (property "Manufacturer" "onsemi" (at 0 0 0) (effects (font (size 1 1)) (hide yes))) (property "MPN" "4N32M" (at 0 0 0) (effects (font (size 1 1)) (hide yes))))
 (wire (pts (xy 137.16 177.8) (xy 132.08 177.8)) (stroke (width 0) (type default)))
 (global_label "FAVERO2_LED" (shape bidirectional) (at 132.08 177.8 180) (effects (font (size 0.9 0.9)) (justify right)) (property "Intersheetrefs" "" (at 132.08 177.8 180) (effects (font (size 1 1)) (hide yes))))
@@
 (wire (pts (xy 172.72 182.88) (xy 177.8 182.88)) (stroke (width 0) (type default)))
 (global_label "FAVERO2_BASE" (shape bidirectional) (at 177.8 182.88 0) (effects (font (size 0.9 0.9)) (justify left)) (property "Intersheetrefs" "" (at 177.8 182.88 0) (effects (font (size 1 1)) (hide yes))))
-(symbol (lib_id "ScoringPlatform:TE_5520250_2") (at 335.28 180.34 0) (unit 1) (in_bom yes) (on_board yes) (dnp no) (property "Reference" "J10" (at 335.28 166.34 0) (effects (font (size 1.2 1.2)))) (property "Value" "5520250-2" (at 335.28 168.34 0) (effects (font (size 1.1 1.1)))) (property "Footprint" "ScoringPlatform:RJ14" (at 335.28 180.34 0) (effects (font (size 1 1)) (hide yes))) (pin "2") (pin "3") (pin "4") (pin "5") (instances (project "usb-scoring-platform" (path "/20cc8167-128c-446a-a106-f942323e143f/19a689f6-051a-47d6-a064-26f29b455422" (reference "J10") (unit 1)))))
+(symbol (lib_id "ScoringPlatform:TE_5520250_2") (at 335.28 180.34 0) (unit 1) (in_bom yes) (on_board yes) (dnp no) (property "Reference" "J10" (at 335.28 166.34 0) (effects (font (size 1.2 1.2)))) (property "Value" "5520250-2" (at 335.28 168.34 0) (effects (font (size 1.1 1.1)))) (property "Footprint" "ScoringPlatform:RJ14" (at 335.28 180.34 0) (effects (font (size 1 1)) (hide yes))) (pin "2") (pin "3") (pin "4") (pin "5") (instances (project "usb-scoring-platform" (path "/20cc8167-128c-446a-a106-f942323e143f/19a689f6-051a-47d6-a064-26f29b455422" (reference "J10") (unit 1)))) (property "Manufacturer" "TE Connectivity" (at 0 0 0) (effects (font (size 1 1)) (hide yes))) (property "MPN" "5520250-2" (at 0 0 0) (effects (font (size 1 1)) (hide yes))))
 (wire (pts (xy 317.5 177.8) (xy 312.42 177.8)) (stroke (width 0) (type default)))
 (global_label "FAVERO2_OUTER_A" (shape bidirectional) (at 312.42 177.8 180) (effects (font (size 0.9 0.9)) (justify right)) (property "Intersheetrefs" "" (at 312.42 177.8 180) (effects (font (size 1 1)) (hide yes))))
