File: packages/scoring-circuit/usb-scoring-platform/ethernet-and-remote.kicad_sch (KiCad schematic)
At the start: 6 parts, among them U12 WIZ850io, U13 TSOP38438

Commit message: feat(scoring-circuit): select exact prototype resistor parts
Parts:
- R32: MPN (none) -> RC0603FR-07100RL; Manufacturer (none) -> YAGEO

Commit message: feat(scoring-circuit): select bypass and timing capacitors
Parts:
- C29, C30: MPN (none) -> C1608X7R1H104K080AA; Manufacturer (none) -> TDK

Commit message: feat(scoring-circuit): complete nominal capacitor selections
Parts:
- C28: MPN (none) -> C1608X5R1C106M080AB; Manufacturer (none) -> TDK

Commit message: chore(scoring-circuit): bind crystal and peripheral ordering details
Parts:
- U13: MPN (none) -> TSOP38438; Manufacturer (none) -> Vishay

Commit message: chore(scoring-circuit): complete assembly BOM ordering fields
Parts:
- U12: MPN (none) -> WIZ850io; Manufacturer (none) -> WIZnet

Commit message: fix(scoring-circuit): reconcile direct Ethernet schematic draft
Parts:
- added C51: 22nF, Capacitor_SMD:C_0603_1608Metric, symbol Device:C
- added C52, C53: 6.8nF, Capacitor_SMD:C_0603_1608Metric, symbol Device:C
- added C54, C55: 10nF, Capacitor_SMD:C_0603_1608Metric, symbol Device:C
- added C56: 4.7uF, Capacitor_SMD:C_0603_1608Metric, symbol Device:C
- added C57, C58, C59, C60, C61, C62: 100nF, Capacitor_SMD:C_0603_1608Metric, symbol Device:C
- added C63: 10uF, Capacitor_SMD:C_0805_2012Metric, symbol Device:C
- added C64, C65: 18pF C0G, Capacitor_SMD:C_0603_1608Metric, symbol Device:C
- added FB1: 120R@100MHz, Inductor_SMD:L_0603_1608Metric, symbol Device:FerriteBead
- added J13: J1B1211CCD, Connector_RJ:RJ45_Cetus_J1B1211CCD_Horizontal, symbol ScoringPlatform:J1B1211CCD
- added R100, R101, R102, R99: 49.9R 1%, Resistor_SMD:R_0603_1608Metric, symbol Device:R
- added R103: 10R 1%, Resistor_SMD:R_0603_1608Metric, symbol Device:R
- added R104: 12.4k 1%, Resistor_SMD:R_0603_1608Metric, symbol Device:R
- added R105, R106: 330R 1%, Resistor_SMD:R_0603_1608Metric, symbol Device:R
- added R107: 1M 1%, Resistor_SMD:R_0603_1608Metric, symbol Device:R
- added Y2: 25MHz CL18pF, Crystal:Crystal_SMD_3225-4Pin_3.2x2.5mm, symbol Device:Crystal_GND24
- U12: value WIZ850io -> W5500; footprint ScoringPlatform:WIZ850io -> Package_QFP:LQFP-48_7x7mm_P0.5mm; symbol ScoringPlatform:WIZ850io -> Interface_Ethernet:W5500; MPN WIZ850io -> W5500
Connections:
- net APP_3V3: now also U12.28 (VDD), U12.43 (PMODE2), U12.44 (PMODE1), U12.45 (PMODE0), FB1.1, J13.10 (GREEN_A), J13.12 (YELLOW_A); no longer U12.8 (3V3), U12.9 (3V3)
- net ETH_CS_N: now also U12.32 (~{SCS}); no longer U12.5 (CS_N)
- net ETH_IRQ_N: now also U12.36 (~{INT}); no longer U12.6 (INT_N)
- net ETH_MISO: now also U12.34 (MISO); no longer U12.12 (MISO)
- net ETH_MOSI: now also U12.35 (MOSI); no longer U12.3 (MOSI)
- net ETH_RESET_N: now also U12.37 (~{RST}); no longer U12.11 (RESET_N)
- net ETH_SCLK: now also U12.33 (SCLK); no longer U12.4 (SCLK)
- net GND: now also U12.14 (AGND), U12.16 (AGND), U12.19 (AGND), U12.23 (RSVD), U12.29 (GND), U12.3 (AGND), U12.48 (AGND), U12.9 (AGND), C51.2, C54.2, C55.2, C56.2, C57.2, C58.2, C59.2, C60.2, C61.2, C62.2, C63.2, C64.2, C65.2, R104.2, Y2.2 (G), Y2.4 (G); no longer U12.1 (GND), U12.2 (GND), U12.7 (GND)
- net ETH_EXRES: now reaches U12.10 (EXRES1)
- net ETH_EXRES: now also R104.1
- new net ETH_1V2: C55.1, U12.22 (1V2O)
- new net ETH_ACT_K: J13.11 (YELLOW_K), R106.1
- new net ETH_ACT_LED: R106.2, U12.27 (ACTLED)
- new net ETH_AVDD: C57.1, C58.1, C59.1, C60.1, C61.1, C62.1, C63.1, FB1.2, R100.2, R103.1, R99.2, U12.11 (AVDD), U12.15 (AVDD), U12.17 (AVDD), U12.21 (AVDD), U12.4 (AVDD), U12.8 (AVDD)
- new net ETH_LINK_K: J13.9 (GREEN_K), R105.1
- new net ETH_LINK_LED: R105.2, U12.25 (LINKLED)
- new net ETH_RX_CT: C52.2, C53.2, J13.5 (RX_CT)
- new net ETH_RX_N: C53.1, J13.6 (RD-), R102.1, U12.5 (RXN)
- new net ETH_RX_P: C52.1, J13.4 (RD+), R101.1, U12.6 (RXP)
- new net ETH_RX_TERM: C54.1, R101.2, R102.2
- new net ETH_SHIELD: J13.13 (SHIELD), J13.8 (CHS_GND)
- new net ETH_TOCAP: C56.1, U12.20 (TOCAP)
- new net ETH_TX_CT: C51.1, J13.2 (TX_CT), R103.2
- new net ETH_TX_N: J13.3 (TD-), R100.1, U12.1 (TXN)
- new net ETH_TX_P: J13.1 (TD+), R99.1, U12.2 (TXP)
- new net ETH_XI: C64.1, R107.1, U12.30 (XI/CLKIN), Y2.1
- new net ETH_XO: C65.1, R107.2, U12.31 (XO), Y2.3
- no-connect marks 1 -> 14
Other:
- note added: "Direct W5500 Ethernet, all-mode autonegotiation. Preserve ESP32 SPI/reset/IRQ nets. J13: CETUS J1B1211CCD, matching WIZnet reference. Separate TX/RX centre taps. ETH_SHIELD is connector-local and is not a galvanic short to board ground. PCB placement, shield coupling, routing, ordering and crystal-load review IN PROGRESS; NOT FOR FABRICATION."
- note removed: "One WIZ850io Ethernet port for Cyrano/network traffic. TSOP38438 is the 38kHz IR receiver. No scoring timing is delegated to network traffic."
- note removed: "WIZ850io already contains W5500, magnetics, crystal and connector. Its module pulls are retained; do not add duplicate pulls."

Commit message: feat(scoring-circuit): route direct W5500 Ethernet checkpoint
Parts:
- J13: footprint Connector_RJ:RJ45_Cetus_J1B1211CCD_Horizontal -> ScoringPlatform:J1B1211CCD
Changed lines of the file:
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@@
 (no_connect (at 92.71 92.71))
 (no_connect (at 92.71 95.25))
-(symbol (lib_id "ScoringPlatform:J1B1211CCD") (at 185.42 105.41 0) (unit 1) (in_bom yes) (on_board yes) (dnp no) (property "Reference" "J13" (at 185.42 90.17 0) (effects (font (size 1.27 1.27)))) (property "Value" "J1B1211CCD" (at 185.42 92.71000000000001 0) (effects (font (size 1.27 1.27)))) (property "Footprint" "Connector_RJ:RJ45_Cetus_J1B1211CCD_Horizontal" (at 185.42 105.41 0) (effects (font (size 1 1)) (hide yes))) (property "MPN" "J1B1211CCD" (at 185.42 105.41 0) (effects (font (size 1 1)) (hide yes))) (property "Manufacturer" "Cetus International" (at 185.42 105.41 0) (effects (font (size 1 1)) (hide yes))) (pin "1") (pin "2") (pin "3") (pin "4") (pin "5") (pin "6") (pin "7") (pin "8") (pin "9") (pin "10") (pin "11") (pin "12") (pin "13") (instances (project "usb-scoring-platform" (path "/20cc8167-128c-446a-a106-f942323e143f/bd387e31-6da9-4a92-aed7-12491d1f9509" (reference "J13") (unit 1)))))
+(symbol (lib_id "ScoringPlatform:J1B1211CCD") (at 185.42 105.41 0) (unit 1) (in_bom yes) (on_board yes) (dnp no) (property "Reference" "J13" (at 185.42 90.17 0) (effects (font (size 1.27 1.27)))) (property "Value" "J1B1211CCD" (at 185.42 92.71000000000001 0) (effects (font (size 1.27 1.27)))) (property "Footprint" "ScoringPlatform:J1B1211CCD" (at 185.42 105.41 0) (effects (font (size 1 1)) (hide yes))) (property "MPN" "J1B1211CCD" (at 185.42 105.41 0) (effects (font (size 1 1)) (hide yes))) (property "Manufacturer" "Cetus International" (at 185.42 105.41 0) (effects (font (size 1 1)) (hide yes))) (pin "1") (pin "2") (pin "3") (pin "4") (pin "5") (pin "6") (pin "7") (pin "8") (pin "9") (pin "10") (pin "11") (pin "12") (pin "13") (instances (project "usb-scoring-platform" (path "/20cc8167-128c-446a-a106-f942323e143f/bd387e31-6da9-4a92-aed7-12491d1f9509" (reference "J13") (unit 1)))))
 (wire (pts (xy 167.64 97.79) (xy 162.56 97.79)) (stroke (width 0) (type default)))
 (global_label "ETH_TX_P" (shape bidirectional) (at 162.56 97.79 180) (effects (font (size .9 .9)) (justify right)) (property "Intersheetrefs" "" (at 162.56 97.79 0) (effects (font (size 1 1)) (hide yes))))

Commit message: fix(scoring-circuit): correct Ethernet receive coupling
Connections:
- net ETH_RX_N: no longer J13.6 (RD-)
- net ETH_RX_P: no longer J13.4 (RD+)
- net ETH_RX_TERM: now also J13.5 (RX_CT)
- removed net ETH_RX_CT: C52.2, C53.2, J13.5 (RX_CT)
- new net ETH_RX_JACK_N: C53.2, J13.6 (RD-)
- new net ETH_RX_JACK_P: C52.2, J13.4 (RD+)
Changed lines of the file:
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@@
 (global_label "ETH_TX_N" (shape bidirectional) (at 162.56 102.87 180) (effects (font (size .9 .9)) (justify right)) (property "Intersheetrefs" "" (at 162.56 102.87 0) (effects (font (size 1 1)) (hide yes))))
 (wire (pts (xy 167.64 105.41) (xy 162.56 105.41)) (stroke (width 0) (type default)))
-(global_label "ETH_RX_P" (shape bidirectional) (at 162.56 105.41 180) (effects (font (size .9 .9)) (justify right)) (property "Intersheetrefs" "" (at 162.56 105.41 0) (effects (font (size 1 1)) (hide yes))))
+(global_label "ETH_RX_JACK_P" (shape bidirectional) (at 162.56 105.41 180) (effects (font (size .9 .9)) (justify right)) (property "Intersheetrefs" "" (at 162.56 105.41 0) (effects (font (size 1 1)) (hide yes))))
 (wire (pts (xy 167.64 107.95) (xy 162.56 107.95)) (stroke (width 0) (type default)))
-(global_label "ETH_RX_CT" (shape bidirectional) (at 162.56 107.95 180) (effects (font (size .9 .9)) (justify right)) (property "Intersheetrefs" "" (at 162.56 107.95 0) (effects (font (size 1 1)) (hide yes))))
+(global_label "ETH_RX_TERM" (shape bidirectional) (at 162.56 107.95 180) (effects (font (size .9 .9)) (justify right)) (property "Intersheetrefs" "" (at 162.56 107.95 0) (effects (font (size 1 1)) (hide yes))))
 (wire (pts (xy 167.64 110.49) (xy 162.56 110.49)) (stroke (width 0) (type default)))
-(global_label "ETH_RX_N" (shape bidirectional) (at 162.56 110.49 180) (effects (font (size .9 .9)) (justify right)) (property "Intersheetrefs" "" (at 162.56 110.49 0) (effects (font (size 1 1)) (hide yes))))
+(global_label "ETH_RX_JACK_N" (shape bidirectional) (at 162.56 110.49 180) (effects (font (size .9 .9)) (justify right)) (property "Intersheetrefs" "" (at 162.56 110.49 0) (effects (font (size 1 1)) (hide yes))))
 (no_connect (at 167.64 113.03))
 (wire (pts (xy 203.2 97.79) (xy 208.28 97.79)) (stroke (width 0) (type default)))
@@
 (global_label "ETH_RX_P" (shape bidirectional) (at 97.79 254 0) (effects (font (size .9 .9)) (justify left)) (property "Intersheetrefs" "" (at 97.79 254 0) (effects (font (size 1 1)) (hide yes))))
 (wire (pts (xy 97.79 266.7) (xy 97.79 271.78)) (stroke (width 0) (type default)))
-(global_label "ETH_RX_CT" (shape bidirectional) (at 97.79 271.78 0) (effects (font (size .9 .9)) (justify left)) (property "Intersheetrefs" "" (at 97.79 271.78 0) (effects (font (size 1 1)) (hide yes))))
+(global_label "ETH_RX_JACK_P" (shape bidirectional) (at 97.79 271.78 0) (effects (font (size .9 .9)) (justify left)) (property "Intersheetrefs" "" (at 97.79 271.78 0) (effects (font (size 1 1)) (hide yes))))
 (symbol (lib_id "Device:C") (at 156.21 262.89 0) (unit 1) (in_bom yes) (on_board yes) (dnp no) (property "Reference" "C53" (at 156.21 250.27 0) (effects (font (size 1.27 1.27)))) (property "Value" "6.8nF" (at 156.21 252.81 0) (effects (font (size 1.27 1.27)))) (property "Footprint" "Capacitor_SMD:C_0603_1608Metric" (at 156.21 262.89 0) (effects (font (size 1 1)) (hide yes))) (property "MPN" "C1608X7R1H682K080AA" (at 156.21 262.89 0) (effects (font (size 1 1)) (hide yes))) (property "Manufacturer" "TDK" (at 156.21 262.89 0) (effects (font (size 1 1)) (hide yes))) (pin "1") (pin "2") (instances (project "usb-scoring-platform" (path "/20cc8167-128c-446a-a106-f942323e143f/bd387e31-6da9-4a92-aed7-12491d1f9509" (reference "C53") (unit 1)))))
 (wire (pts (xy 156.21 259.08) (xy 156.21 254)) (stroke (width 0) (type default)))
 (global_label "ETH_RX_N" (shape bidirectional) (at 156.21 254 0) (effects (font (size .9 .9)) (justify left)) (property "Intersheetrefs" "" (at 156.21 254 0) (effects (font (size 1 1)) (hide yes))))
 (wire (pts (xy 156.21 266.7) (xy 156.21 271.78)) (stroke (width 0) (type default)))
-(global_label "ETH_RX_CT" (shape bidirectional) (at 156.21 271.78 0) (effects (font (size .9 .9)) (justify left)) (property "Intersheetrefs" "" (at 156.21 271.78 0) (effects (font (size 1 1)) (hide yes))))
+(global_label "ETH_RX_JACK_N" (shape bidirectional) (at 156.21 271.78 0) (effects (font (size .9 .9)) (justify left)) (property "Intersheetrefs" "" (at 156.21 271.78 0) (effects (font (size 1 1)) (hide yes))))
 (symbol (lib_id "Device:C") (at 214.63 262.89 0) (unit 1) (in_bom yes) (on_board yes) (dnp no) (property "Reference" "C54" (at 214.63 250.27 0) (effects (font (size 1.27 1.27)))) (property "Value" "10nF" (at 214.63 252.81 0) (effects (font (size 1.27 1.27)))) (property "Footprint" "Capacitor_SMD:C_0603_1608Metric" (at 214.63 262.89 0) (effects (font (size 1 1)) (hide yes))) (property "MPN" "C1608X7R1H103K080AA" (at 214.63 262.89 0) (effects (font (size 1 1)) (hide yes))) (property "Manufacturer" "TDK" (at 214.63 262.89 0) (effects (font (size 1 1)) (hide yes))) (pin "1") (pin "2") (instances (project "usb-scoring-platform" (path "/20cc8167-128c-446a-a106-f942323e143f/bd387e31-6da9-4a92-aed7-12491d1f9509" (reference "C54") (unit 1)))))
 (wire (pts (xy 214.63 259.08) (xy 214.63 254)) (stroke (width 0) (type default)))
