File: packages/scoring-circuit/usb-scoring-platform/ethernet-and-remote.kicad_sch (KiCad schematic)
At the start: 33 parts, among them J13 J1B1211CCD, U12 W5500, U13 TSOP38438, Y2 25MHz CL18pF

Commit message: fix(scoring): select accessible crystal load capacitors
Parts:
- C64, C65: MPN C1608C0G1H180J080AA -> CC0603JRNPO9BN180; Manufacturer TDK -> YAGEO
Changed lines of the file:
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@@
 (wire (pts (xy 214.63 314.96) (xy 214.63 320.04)) (stroke (width 0) (type default)))
 (global_label "GND" (shape bidirectional) (at 214.63 320.04 0) (effects (font (size .9 .9)) (justify left)) (property "Intersheetrefs" "" (at 214.63 320.04 0) (effects (font (size 1 1)) (hide yes))))
-(symbol (lib_id "Device:C") (at 271.78 311.15 0) (unit 1) (in_bom yes) (on_board yes) (dnp no) (property "Reference" "C64" (at 271.78 298.53 0) (effects (font (size 1.27 1.27)))) (property "Value" "18pF C0G" (at 271.78 301.07 0) (effects (font (size 1.27 1.27)))) (property "Footprint" "Capacitor_SMD:C_0603_1608Metric" (at 271.78 311.15 0) (effects (font (size 1 1)) (hide yes))) (property "MPN" "C1608C0G1H180J080AA" (at 271.78 311.15 0) (effects (font (size 1 1)) (hide yes))) (property "Manufacturer" "TDK" (at 271.78 311.15 0) (effects (font (size 1 1)) (hide yes))) (pin "1") (pin "2") (instances (project "usb-scoring-platform" (path "/20cc8167-128c-446a-a106-f942323e143f/bd387e31-6da9-4a92-aed7-12491d1f9509" (reference "C64") (unit 1)))))
+(symbol (lib_id "Device:C") (at 271.78 311.15 0) (unit 1) (in_bom yes) (on_board yes) (dnp no) (property "Reference" "C64" (at 271.78 298.53 0) (effects (font (size 1.27 1.27)))) (property "Value" "18pF C0G" (at 271.78 301.07 0) (effects (font (size 1.27 1.27)))) (property "Footprint" "Capacitor_SMD:C_0603_1608Metric" (at 271.78 311.15 0) (effects (font (size 1 1)) (hide yes))) (property "MPN" "CC0603JRNPO9BN180" (at 271.78 311.15 0) (effects (font (size 1 1)) (hide yes))) (property "Manufacturer" "YAGEO" (at 271.78 311.15 0) (effects (font (size 1 1)) (hide yes))) (pin "1") (pin "2") (instances (project "usb-scoring-platform" (path "/20cc8167-128c-446a-a106-f942323e143f/bd387e31-6da9-4a92-aed7-12491d1f9509" (reference "C64") (unit 1)))))
 (wire (pts (xy 271.78 307.34) (xy 271.78 302.26)) (stroke (width 0) (type default)))
 (global_label "ETH_XI" (shape bidirectional) (at 271.78 302.26 0) (effects (font (size .9 .9)) (justify left)) (property "Intersheetrefs" "" (at 271.78 302.26 0) (effects (font (size 1 1)) (hide yes))))
 (wire (pts (xy 271.78 314.96) (xy 271.78 320.04)) (stroke (width 0) (type default)))
 (global_label "GND" (shape bidirectional) (at 271.78 320.04 0) (effects (font (size .9 .9)) (justify left)) (property "Intersheetrefs" "" (at 271.78 320.04 0) (effects (font (size 1 1)) (hide yes))))
-(symbol (lib_id "Device:C") (at 330.2 311.15 0) (unit 1) (in_bom yes) (on_board yes) (dnp no) (property "Reference" "C65" (at 330.2 298.53 0) (effects (font (size 1.27 1.27)))) (property "Value" "18pF C0G" (at 330.2 301.07 0) (effects (font (size 1.27 1.27)))) (property "Footprint" "Capacitor_SMD:C_0603_1608Metric" (at 330.2 311.15 0) (effects (font (size 1 1)) (hide yes))) (property "MPN" "C1608C0G1H180J080AA" (at 330.2 311.15 0) (effects (font (size 1 1)) (hide yes))) (property "Manufacturer" "TDK" (at 330.2 311.15 0) (effects (font (size 1 1)) (hide yes))) (pin "1") (pin "2") (instances (project "usb-scoring-platform" (path "/20cc8167-128c-446a-a106-f942323e143f/bd387e31-6da9-4a92-aed7-12491d1f9509" (reference "C65") (unit 1)))))
+(symbol (lib_id "Device:C") (at 330.2 311.15 0) (unit 1) (in_bom yes) (on_board yes) (dnp no) (property "Reference" "C65" (at 330.2 298.53 0) (effects (font (size 1.27 1.27)))) (property "Value" "18pF C0G" (at 330.2 301.07 0) (effects (font (size 1.27 1.27)))) (property "Footprint" "Capacitor_SMD:C_0603_1608Metric" (at 330.2 311.15 0) (effects (font (size 1 1)) (hide yes))) (property "MPN" "CC0603JRNPO9BN180" (at 330.2 311.15 0) (effects (font (size 1 1)) (hide yes))) (property "Manufacturer" "YAGEO" (at 330.2 311.15 0) (effects (font (size 1 1)) (hide yes))) (pin "1") (pin "2") (instances (project "usb-scoring-platform" (path "/20cc8167-128c-446a-a106-f942323e143f/bd387e31-6da9-4a92-aed7-12491d1f9509" (reference "C65") (unit 1)))))
 (wire (pts (xy 330.2 307.34) (xy 330.2 302.26)) (stroke (width 0) (type default)))
 (global_label "ETH_XO" (shape bidirectional) (at 330.2 302.26 0) (effects (font (size .9 .9)) (justify left)) (property "Intersheetrefs" "" (at 330.2 302.26 0) (effects (font (size 1 1)) (hide yes))))

Commit message: fix(scoring): replace obsolete Ethernet reference capacitor
Parts:
- C56: MPN C1608X5R1A475K080AC -> C1608X5R1C475K080AC
Changed lines of the file:
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@@
 (wire (pts (xy 271.78 266.7) (xy 271.78 271.78)) (stroke (width 0) (type default)))
 (global_label "GND" (shape bidirectional) (at 271.78 271.78 0) (effects (font (size .9 .9)) (justify left)) (property "Intersheetrefs" "" (at 271.78 271.78 0) (effects (font (size 1 1)) (hide yes))))
-(symbol (lib_id "Device:C") (at 330.2 262.89 0) (unit 1) (in_bom yes) (on_board yes) (dnp no) (property "Reference" "C56" (at 330.2 250.27 0) (effects (font (size 1.27 1.27)))) (property "Value" "4.7uF" (at 330.2 252.81 0) (effects (font (size 1.27 1.27)))) (property "Footprint" "Capacitor_SMD:C_0603_1608Metric" (at 330.2 262.89 0) (effects (font (size 1 1)) (hide yes))) (property "MPN" "C1608X5R1A475K080AC" (at 330.2 262.89 0) (effects (font (size 1 1)) (hide yes))) (property "Manufacturer" "TDK" (at 330.2 262.89 0) (effects (font (size 1 1)) (hide yes))) (pin "1") (pin "2") (instances (project "usb-scoring-platform" (path "/20cc8167-128c-446a-a106-f942323e143f/bd387e31-6da9-4a92-aed7-12491d1f9509" (reference "C56") (unit 1)))))
+(symbol (lib_id "Device:C") (at 330.2 262.89 0) (unit 1) (in_bom yes) (on_board yes) (dnp no) (property "Reference" "C56" (at 330.2 250.27 0) (effects (font (size 1.27 1.27)))) (property "Value" "4.7uF" (at 330.2 252.81 0) (effects (font (size 1.27 1.27)))) (property "Footprint" "Capacitor_SMD:C_0603_1608Metric" (at 330.2 262.89 0) (effects (font (size 1 1)) (hide yes))) (property "MPN" "C1608X5R1C475K080AC" (at 330.2 262.89 0) (effects (font (size 1 1)) (hide yes))) (property "Manufacturer" "TDK" (at 330.2 262.89 0) (effects (font (size 1 1)) (hide yes))) (pin "1") (pin "2") (instances (project "usb-scoring-platform" (path "/20cc8167-128c-446a-a106-f942323e143f/bd387e31-6da9-4a92-aed7-12491d1f9509" (reference "C56") (unit 1)))))
 (wire (pts (xy 330.2 259.08) (xy 330.2 254)) (stroke (width 0) (type default)))
 (global_label "ETH_TOCAP" (shape bidirectional) (at 330.2 254 0) (effects (font (size .9 .9)) (justify left)) (property "Intersheetrefs" "" (at 330.2 254 0) (effects (font (size 1 1)) (hide yes))))

Commit message: fix(scoring): select stocked coupling and controller capacitors
Parts:
- C52, C53: MPN C1608X7R1H682K080AA -> CC0603KRX7R9BB682; Manufacturer TDK -> Yageo
Changed lines of the file:
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@@
 (wire (pts (xy 39.37 266.7) (xy 39.37 271.78)) (stroke (width 0) (type default)))
 (global_label "GND" (shape bidirectional) (at 39.37 271.78 0) (effects (font (size .9 .9)) (justify left)) (property "Intersheetrefs" "" (at 39.37 271.78 0) (effects (font (size 1 1)) (hide yes))))
-(symbol (lib_id "Device:C") (at 97.79 262.89 0) (unit 1) (in_bom yes) (on_board yes) (dnp no) (property "Reference" "C52" (at 97.79 250.27 0) (effects (font (size 1.27 1.27)))) (property "Value" "6.8nF" (at 97.79 252.81 0) (effects (font (size 1.27 1.27)))) (property "Footprint" "Capacitor_SMD:C_0603_1608Metric" (at 97.79 262.89 0) (effects (font (size 1 1)) (hide yes))) (property "MPN" "C1608X7R1H682K080AA" (at 97.79 262.89 0) (effects (font (size 1 1)) (hide yes))) (property "Manufacturer" "TDK" (at 97.79 262.89 0) (effects (font (size 1 1)) (hide yes))) (pin "1") (pin "2") (instances (project "usb-scoring-platform" (path "/20cc8167-128c-446a-a106-f942323e143f/bd387e31-6da9-4a92-aed7-12491d1f9509" (reference "C52") (unit 1)))))
+(symbol (lib_id "Device:C") (at 97.79 262.89 0) (unit 1) (in_bom yes) (on_board yes) (dnp no) (property "Reference" "C52" (at 97.79 250.27 0) (effects (font (size 1.27 1.27)))) (property "Value" "6.8nF" (at 97.79 252.81 0) (effects (font (size 1.27 1.27)))) (property "Footprint" "Capacitor_SMD:C_0603_1608Metric" (at 97.79 262.89 0) (effects (font (size 1 1)) (hide yes))) (property "MPN" "CC0603KRX7R9BB682" (at 97.79 262.89 0) (effects (font (size 1 1)) (hide yes))) (property "Manufacturer" "Yageo" (at 97.79 262.89 0) (effects (font (size 1 1)) (hide yes))) (pin "1") (pin "2") (instances (project "usb-scoring-platform" (path "/20cc8167-128c-446a-a106-f942323e143f/bd387e31-6da9-4a92-aed7-12491d1f9509" (reference "C52") (unit 1)))))
 (wire (pts (xy 97.79 259.08) (xy 97.79 254)) (stroke (width 0) (type default)))
 (global_label "ETH_RX_P" (shape bidirectional) (at 97.79 254 0) (effects (font (size .9 .9)) (justify left)) (property "Intersheetrefs" "" (at 97.79 254 0) (effects (font (size 1 1)) (hide yes))))
 (wire (pts (xy 97.79 266.7) (xy 97.79 271.78)) (stroke (width 0) (type default)))
 (global_label "ETH_RX_JACK_P" (shape bidirectional) (at 97.79 271.78 0) (effects (font (size .9 .9)) (justify left)) (property "Intersheetrefs" "" (at 97.79 271.78 0) (effects (font (size 1 1)) (hide yes))))
-(symbol (lib_id "Device:C") (at 156.21 262.89 0) (unit 1) (in_bom yes) (on_board yes) (dnp no) (property "Reference" "C53" (at 156.21 250.27 0) (effects (font (size 1.27 1.27)))) (property "Value" "6.8nF" (at 156.21 252.81 0) (effects (font (size 1.27 1.27)))) (property "Footprint" "Capacitor_SMD:C_0603_1608Metric" (at 156.21 262.89 0) (effects (font (size 1 1)) (hide yes))) (property "MPN" "C1608X7R1H682K080AA" (at 156.21 262.89 0) (effects (font (size 1 1)) (hide yes))) (property "Manufacturer" "TDK" (at 156.21 262.89 0) (effects (font (size 1 1)) (hide yes))) (pin "1") (pin "2") (instances (project "usb-scoring-platform" (path "/20cc8167-128c-446a-a106-f942323e143f/bd387e31-6da9-4a92-aed7-12491d1f9509" (reference "C53") (unit 1)))))
+(symbol (lib_id "Device:C") (at 156.21 262.89 0) (unit 1) (in_bom yes) (on_board yes) (dnp no) (property "Reference" "C53" (at 156.21 250.27 0) (effects (font (size 1.27 1.27)))) (property "Value" "6.8nF" (at 156.21 252.81 0) (effects (font (size 1.27 1.27)))) (property "Footprint" "Capacitor_SMD:C_0603_1608Metric" (at 156.21 262.89 0) (effects (font (size 1 1)) (hide yes))) (property "MPN" "CC0603KRX7R9BB682" (at 156.21 262.89 0) (effects (font (size 1 1)) (hide yes))) (property "Manufacturer" "Yageo" (at 156.21 262.89 0) (effects (font (size 1 1)) (hide yes))) (pin "1") (pin "2") (instances (project "usb-scoring-platform" (path "/20cc8167-128c-446a-a106-f942323e143f/bd387e31-6da9-4a92-aed7-12491d1f9509" (reference "C53") (unit 1)))))
 (wire (pts (xy 156.21 259.08) (xy 156.21 254)) (stroke (width 0) (type default)))
 (global_label "ETH_RX_N" (shape bidirectional) (at 156.21 254 0) (effects (font (size .9 .9)) (justify left)) (property "Intersheetrefs" "" (at 156.21 254 0) (effects (font (size 1 1)) (hide yes))))

Commit message: fix(scoring-circuit): source stocked bypass and reservoir capacitors
Parts:
- C29, C30, C57, C58, C59, C60, C61, C62: MPN C1608X7R1H104K080AA -> CC0603KRX7R9BB104; Manufacturer TDK -> Yageo
- C63: MPN C2012X5R1A106K125AC -> GRM21BR61A106KE19L; Manufacturer TDK -> Murata
