File: packages/scoring-circuit/usb-scoring-platform/isolated-usb.kicad_sch (KiCad schematic)
At the start: 1 part, among them U18 LTM2884IY#PBF

Commit message: feat(scoring-circuit): route primary USB power controller
Connections:
- net USB_HOST_3V3: no longer U18.A3 (SPNDPWR), U18.A4 (ON)
- new net USB_ISO_EN: U18.A4 (ON)
- new net USB_SUSPEND_EN: U18.A3 (SPNDPWR)
Other:
- note added: "U18 ON and SPNDPWR are controlled by U21 on USB_GND. R112 defaults acquisition OFF; R113 defaults suspend shutdown ON. VLO supplies only primary control logic. Do not bridge USB_GND to isolated GND."
- note removed: "Internal bypass: VBUS 2.2uF, VCC 4.7uF, VLO 2.2uF, VCC2 22uF, VLO2 2.2uF. No duplicate ADuM capacitors/24R resistors."
- note removed: "SPNDPWR high powers off VCC2 after USB idle. Host resume restarts acquisition and requires enumeration; no remote wake."
- note removed: "VCC/VBUS share computer 5V. VLO drives ON + SPNDPWR only; VLO2 is unused (10mA LDO, not the STM32 supply)."
Changed lines of the file:
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@@
 (global_label "USB_HOST_DP" (shape bidirectional) (at 162.56 76.2 180) (effects (font (size 0.9 0.9)) (justify right)) (property "Intersheetrefs" "" (at 162.56 76.2 180) (effects (font (size 1 1)) (hide yes))))
 (wire (pts (xy 167.64 78.74) (xy 162.56 78.74)) (stroke (width 0) (type default)))
-(global_label "USB_HOST_3V3" (shape bidirectional) (at 162.56 78.74 180) (effects (font (size 0.9 0.9)) (justify right)) (property "Intersheetrefs" "" (at 162.56 78.74 180) (effects (font (size 1 1)) (hide yes))))
+(global_label "USB_SUSPEND_EN" (shape bidirectional) (at 162.56 78.74 180) (effects (font (size 0.9 0.9)) (justify right)) (property "Intersheetrefs" "" (at 162.56 78.74 180) (effects (font (size 1 1)) (hide yes))))
 (wire (pts (xy 167.64 81.28) (xy 162.56 81.28)) (stroke (width 0) (type default)))
-(global_label "USB_HOST_3V3" (shape bidirectional) (at 162.56 81.28 180) (effects (font (size 0.9 0.9)) (justify right)) (property "Intersheetrefs" "" (at 162.56 81.28 180) (effects (font (size 1 1)) (hide yes))))
+(global_label "USB_ISO_EN" (shape bidirectional) (at 162.56 81.28 180) (effects (font (size 0.9 0.9)) (justify right)) (property "Intersheetrefs" "" (at 162.56 81.28 180) (effects (font (size 1 1)) (hide yes))))
 (wire (pts (xy 167.64 83.82) (xy 162.56 83.82)) (stroke (width 0) (type default)))
 (global_label "USB_HOST_3V3" (shape bidirectional) (at 162.56 83.82 180) (effects (font (size 0.9 0.9)) (justify right)) (property "Intersheetrefs" "" (at 162.56 83.82 180) (effects (font (size 1 1)) (hide yes))))
@@
 (wire (pts (xy 203.2 127) (xy 208.28 127)) (stroke (width 0) (type default)))
 (global_label "USB_ISOLATED_5V" (shape bidirectional) (at 208.28 127 0) (effects (font (size 0.9 0.9)) (justify left)) (property "Intersheetrefs" "" (at 208.28 127 0) (effects (font (size 1 1)) (hide yes))))
-(text "VCC/VBUS share computer 5V. VLO drives ON + SPNDPWR only; VLO2 is unused (10mA LDO, not the STM32 supply)." (at 25 150 0) (effects (font (size 1.1 1.1)) (justify left top)))
-(text "Internal bypass: VBUS 2.2uF, VCC 4.7uF, VLO 2.2uF, VCC2 22uF, VLO2 2.2uF. No duplicate ADuM capacitors/24R resistors." (at 25 160 0) (effects (font (size 1.1 1.1)) (justify left top)))
+(text "U18 ON and SPNDPWR are controlled by U21 on USB_GND.\nR112 defaults acquisition OFF; R113 defaults suspend shutdown ON.\nVLO supplies only primary control logic. Do not bridge USB_GND to isolated GND." (at 25 150 0) (effects (font (size 1.1 1.1)) (justify left top)))
+(text "U18 ON and SPNDPWR are controlled by U21 on USB_GND.\nR112 defaults acquisition OFF; R113 defaults suspend shutdown ON.\nVLO supplies only primary control logic. Do not bridge USB_GND to isolated GND." (at 25 160 0) (effects (font (size 1.1 1.1)) (justify left top)))
 (text "VCC2 feeds D1 on the power sheet. Never connect 20V PD to this module. Keep all copper out of the isolation barrier." (at 25 170 0) (effects (font (size 1.1 1.1)) (justify left top)))
 (text "FIRMWARE REQUIRED: boot <=16MHz, excitation/comparators off. Sound and Favero stay off throughout laptop-only mode." (at 25 190 0) (effects (font (size 1.1 1.1)) (justify left top)))
@@
 (text "Measure host <=100mA before / <=500mA after configuration; output budget is NOT input proof. Reset returns to low power." (at 25 210 0) (effects (font (size 1.1 1.1)) (justify left top)))
 (text "Laptop product: no HUB75 panel connected; ESP32/Ethernet/IR supply stays off. U18 200mA rating is not an operating target." (at 25 220 0) (effects (font (size 1.1 1.1)) (justify left top)))
-(text "SPNDPWR high powers off VCC2 after USB idle. Host resume restarts acquisition and requires enumeration; no remote wake." (at 25 230 0) (effects (font (size 1.1 1.1)) (justify left top)))
+(text "U18 ON and SPNDPWR are controlled by U21 on USB_GND.\nR112 defaults acquisition OFF; R113 defaults suspend shutdown ON.\nVLO supplies only primary control logic. Do not bridge USB_GND to isolated GND." (at 25 230 0) (effects (font (size 1.1 1.1)) (justify left top)))
 (text "PB5 USB_PRESENT senses isolated 5V on the power sheet. Disable STM32 D+ pull-up while absent, including when PD stays on." (at 25 240 0) (effects (font (size 1.1 1.1)) (justify left top)))
 (text "Desktop preserves bout state but discards old capture sessions after reconnect. Timing/suspend/inrush and USB compliance need bench tests." (at 25 250 0) (effects (font (size 1.1 1.1)) (justify left top)))
