File: packages/scoring-circuit/usb-scoring-platform/display-and-sound.kicad_sch (KiCad schematic)
At the start: 29 parts, among them J7 TST-108-02-G-D - HUB75, J8 645004114822 - panel 5V, Q1 DMN2056U-7, Q2 DMN2056U-7, U14 SN74AHCT541PWR, U15 SN74AHCT541PWR

Commit message: fix(scoring-circuit): source stocked bypass and reservoir capacitors
Parts:
- C31, C32, C35: MPN C1608X7R1H104K080AA -> CC0603KRX7R9BB104; Manufacturer TDK -> Yageo
Changed lines of the file:
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@@
 (wire (pts (xy 97.79 101.6) (xy 102.87 101.6)) (stroke (width 0) (type default)))
 (global_label "PANEL_5V" (shape bidirectional) (at 102.87 101.6 0) (effects (font (size 0.9 0.9)) (justify left)) (property "Intersheetrefs" "" (at 102.87 101.6 0) (effects (font (size 1 1)) (hide yes))))
-(symbol (lib_id "Device:C") (at 74.93 144.78 0) (unit 1) (in_bom yes) (on_board yes) (dnp no) (property "Reference" "C31" (at 74.93 130.78 0) (effects (font (size 1.2 1.2)))) (property "Value" "100nF 16V" (at 74.93 132.78 0) (effects (font (size 1.1 1.1)))) (property "Footprint" "Capacitor_SMD:C_0603_1608Metric" (at 74.93 144.78 0) (effects (font (size 1 1)) (hide yes))) (pin "1") (pin "2") (property "Manufacturer" "TDK" (at 74.93 144.78 0) (effects (font (size 1 1)) (hide yes))) (property "MPN" "C1608X7R1H104K080AA" (at 74.93 144.78 0) (effects (font (size 1 1)) (hide yes))) (property "Datasheet" "https://product.tdk.com/en/search/capacitor/ceramic/mlcc/info?part_no=C1608X7R1H104K080AA" (at 74.93 144.78 0) (effects (font (size 1 1)) (hide yes))) (instances (project "usb-scoring-platform" (path "/20cc8167-128c-446a-a106-f942323e143f/8eb01a97-00e8-4fc9-a0dc-2c04f64b61fc" (reference "C31") (unit 1)))))
+(symbol (lib_id "Device:C") (at 74.93 144.78 0) (unit 1) (in_bom yes) (on_board yes) (dnp no) (property "Reference" "C31" (at 74.93 130.78 0) (effects (font (size 1.2 1.2)))) (property "Value" "100nF 16V" (at 74.93 132.78 0) (effects (font (size 1.1 1.1)))) (property "Footprint" "Capacitor_SMD:C_0603_1608Metric" (at 74.93 144.78 0) (effects (font (size 1 1)) (hide yes))) (pin "1") (pin "2") (property "Manufacturer" "Yageo" (at 74.93 144.78 0) (effects (font (size 1 1)) (hide yes))) (property "MPN" "CC0603KRX7R9BB104" (at 74.93 144.78 0) (effects (font (size 1 1)) (hide yes))) (property "Datasheet" "https://www.yageogroup.com/download/specsheet/CC0603KRX7R9BB104" (at 74.93 144.78 0) (effects (font (size 1 1)) (hide yes))) (instances (project "usb-scoring-platform" (path "/20cc8167-128c-446a-a106-f942323e143f/8eb01a97-00e8-4fc9-a0dc-2c04f64b61fc" (reference "C31") (unit 1)))))
 (wire (pts (xy 74.93 140.97) (xy 74.93 135.89)) (stroke (width 0) (type default)))
 (global_label "PANEL_5V" (shape bidirectional) (at 74.93 135.89 0) (effects (font (size 0.9 0.9)) (justify left)) (property "Intersheetrefs" "" (at 74.93 135.89 0) (effects (font (size 1 1)) (hide yes))))
@@
 (wire (pts (xy 232.41 101.6) (xy 237.49 101.6)) (stroke (width 0) (type default)))
 (global_label "PANEL_5V" (shape bidirectional) (at 237.49 101.6 0) (effects (font (size 0.9 0.9)) (justify left)) (property "Intersheetrefs" "" (at 237.49 101.6 0) (effects (font (size 1 1)) (hide yes))))
-(symbol (lib_id "Device:C") (at 209.55 144.78 0) (unit 1) (in_bom yes) (on_board yes) (dnp no) (property "Reference" "C32" (at 209.55 130.78 0) (effects (font (size 1.2 1.2)))) (property "Value" "100nF 16V" (at 209.55 132.78 0) (effects (font (size 1.1 1.1)))) (property "Footprint" "Capacitor_SMD:C_0603_1608Metric" (at 209.55 144.78 0) (effects (font (size 1 1)) (hide yes))) (pin "1") (pin "2") (property "Manufacturer" "TDK" (at 209.55 144.78 0) (effects (font (size 1 1)) (hide yes))) (property "MPN" "C1608X7R1H104K080AA" (at 209.55 144.78 0) (effects (font (size 1 1)) (hide yes))) (property "Datasheet" "https://product.tdk.com/en/search/capacitor/ceramic/mlcc/info?part_no=C1608X7R1H104K080AA" (at 209.55 144.78 0) (effects (font (size 1 1)) (hide yes))) (instances (project "usb-scoring-platform" (path "/20cc8167-128c-446a-a106-f942323e143f/8eb01a97-00e8-4fc9-a0dc-2c04f64b61fc" (reference "C32") (unit 1)))))
+(symbol (lib_id "Device:C") (at 209.55 144.78 0) (unit 1) (in_bom yes) (on_board yes) (dnp no) (property "Reference" "C32" (at 209.55 130.78 0) (effects (font (size 1.2 1.2)))) (property "Value" "100nF 16V" (at 209.55 132.78 0) (effects (font (size 1.1 1.1)))) (property "Footprint" "Capacitor_SMD:C_0603_1608Metric" (at 209.55 144.78 0) (effects (font (size 1 1)) (hide yes))) (pin "1") (pin "2") (property "Manufacturer" "Yageo" (at 209.55 144.78 0) (effects (font (size 1 1)) (hide yes))) (property "MPN" "CC0603KRX7R9BB104" (at 209.55 144.78 0) (effects (font (size 1 1)) (hide yes))) (property "Datasheet" "https://www.yageogroup.com/download/specsheet/CC0603KRX7R9BB104" (at 209.55 144.78 0) (effects (font (size 1 1)) (hide yes))) (instances (project "usb-scoring-platform" (path "/20cc8167-128c-446a-a106-f942323e143f/8eb01a97-00e8-4fc9-a0dc-2c04f64b61fc" (reference "C32") (unit 1)))))
 (wire (pts (xy 209.55 140.97) (xy 209.55 135.89)) (stroke (width 0) (type default)))
 (global_label "PANEL_5V" (shape bidirectional) (at 209.55 135.89 0) (effects (font (size 0.9 0.9)) (justify left)) (property "Intersheetrefs" "" (at 209.55 135.89 0) (effects (font (size 1 1)) (hide yes))))
@@
 (wire (pts (xy 228.6 214.63) (xy 228.6 219.71)) (stroke (width 0) (type default)))
 (global_label "BUZZER_LOW" (shape bidirectional) (at 228.6 219.71 0) (effects (font (size .9 .9)) (justify left)) (property "Intersheetrefs" "" (at 228.6 219.71 0) (effects (font (size 1 1)) (hide yes))))
-(symbol (lib_id "Device:C") (at 193.04 250.19 0) (unit 1) (in_bom yes) (on_board yes) (dnp no) (property "Reference" "C35" (at 193.04 236.19 0) (effects (font (size 1.2 1.2)))) (property "Value" "100nF" (at 193.04 238.19 0) (effects (font (size 1.1 1.1)))) (property "Footprint" "Capacitor_SMD:C_0603_1608Metric" (at 193.04 250.19 0) (effects (font (size 1 1)) (hide yes))) (pin "1") (pin "2") (property "Manufacturer" "TDK" (at 193.04 250.19 0) (effects (font (size 1 1)) (hide yes))) (property "MPN" "C1608X7R1H104K080AA" (at 193.04 250.19 0) (effects (font (size 1 1)) (hide yes))) (property "Datasheet" "https://product.tdk.com/en/search/capacitor/ceramic/mlcc/info?part_no=C1608X7R1H104K080AA" (at 193.04 250.19 0) (effects (font (size 1 1)) (hide yes))) (instances (project "usb-scoring-platform" (path "/20cc8167-128c-446a-a106-f942323e143f/8eb01a97-00e8-4fc9-a0dc-2c04f64b61fc" (reference "C35") (unit 1)))))
+(symbol (lib_id "Device:C") (at 193.04 250.19 0) (unit 1) (in_bom yes) (on_board yes) (dnp no) (property "Reference" "C35" (at 193.04 236.19 0) (effects (font (size 1.2 1.2)))) (property "Value" "100nF" (at 193.04 238.19 0) (effects (font (size 1.1 1.1)))) (property "Footprint" "Capacitor_SMD:C_0603_1608Metric" (at 193.04 250.19 0) (effects (font (size 1 1)) (hide yes))) (pin "1") (pin "2") (property "Manufacturer" "Yageo" (at 193.04 250.19 0) (effects (font (size 1 1)) (hide yes))) (property "MPN" "CC0603KRX7R9BB104" (at 193.04 250.19 0) (effects (font (size 1 1)) (hide yes))) (property "Datasheet" "https://www.yageogroup.com/download/specsheet/CC0603KRX7R9BB104" (at 193.04 250.19 0) (effects (font (size 1 1)) (hide yes))) (instances (project "usb-scoring-platform" (path "/20cc8167-128c-446a-a106-f942323e143f/8eb01a97-00e8-4fc9-a0dc-2c04f64b61fc" (reference "C35") (unit 1)))))
 (wire (pts (xy 193.04 246.38) (xy 193.04 241.3)) (stroke (width 0) (type default)))
 (global_label "CORE_3V3" (shape bidirectional) (at 193.04 241.3 0) (effects (font (size .9 .9)) (justify left)) (property "Intersheetrefs" "" (at 193.04 241.3 0) (effects (font (size 1 1)) (hide yes))))
