File: packages/scoring-circuit/usb-scoring-platform/usb-pd-power.kicad_sch (KiCad schematic)
At the start: 39 parts, among them J12 PD service: GND SDA SCL, Q4 DMN2056U-7, Q5 DMN2056U-7, U19 LTC3115IDHD-1#PBF, U20 TPS259470LRPWR, U5 STUSB4500QTR, U6 REC30K-2405SZ

Commit message: feat(scoring-circuit): route primary USB power controller
Parts:
- added C69, C71: 100nF 50V, Capacitor_SMD:C_0603_1608Metric, symbol Device:C
- added C70: 1uF 10V, Capacitor_SMD:C_0603_1608Metric, symbol Device:C
- added J14: PRIMARY SWD PADS: 3V3 GND DIO CLK RESET, ScoringPlatform:Primary_SWD_Pads, symbol Connector_Generic:Conn_01x05
- added Q6: DMN2056U-7, Package_TO_SOT_SMD:SOT-23, symbol Transistor_FET:BSS138
- added R111, R112, R113: 100k 1%, Resistor_SMD:R_0603_1608Metric, symbol Device:R
- added R114, R115: 4.7k 1%, Resistor_SMD:R_0603_1608Metric, symbol Device:R
- added R116: 47k 1%, Resistor_SMD:R_0603_1608Metric, symbol Device:R
- added U21: STM32C011F6P6, Package_SO:TSSOP-20_4.4x6.5mm_P0.65mm, symbol MCU_ST_STM32C0:STM32C011F6Px
Connections:
- net PD_EFUSE_EN: now also Q6.3 (D)
- net PD_SCL: now also R115.2, U21.20 (PB6)
- net PD_SDA: now also R114.2, U21.1 (PB7)
- net USB_GND: now also C69.2, C70.2, C71.2, J14.2 (Pin_2), Q6.2 (S), R112.2, U21.5 (VSS)
- net PD_ALERT_N: now reaches U5.19 (ALERT)
- net PD_ALERT_N: now also R116.2, U21.13 (PA6)
- new net APP_INHIBIT: Q6.1 (G), R111.2, U21.12 (PA5)
- new net PWR_NRST: C71.1, J14.5 (Pin_5), U21.6 (PF2)
- new net PWR_SWCLK: J14.4 (Pin_4), U21.19 (PA14)
- new net PWR_SWDIO: J14.3 (Pin_3), U21.18 (PA13)
- new net USB_HOST_3V3: C69.1, C70.1, J14.1 (Pin_1), R111.1, R113.1, R114.1, R115.1, R116.1, U21.4 (VDD)
- new net USB_ISO_EN: R112.1, U21.11 (PA4)
- new net USB_SUSPEND_EN: R113.2, U21.16 (PA9/PA11)
- no-connect marks 11 -> 19
Other:
- note added: "U21 controls power only; primary USB_GND domain, 6MHz internal clock. Reset defaults: U18 OFF, suspend shutdown enabled, Q6 inhibits application power. J14 is primary-side service access: do not connect a grounded debugger to the isolated side. Firmware and STUSB4500 NVM provisioning are required before operation."

Commit message: fix(scoring): migrate primary supply to automatic-mode regulator
Parts:
- removed C67: 3300pF 50V C0G, Capacitor_SMD:C_0603_1608Metric, symbol Device:C
- removed C68: 33pF 50V C0G, Capacitor_SMD:C_0603_1608Metric, symbol Device:C
- removed R108: 47.5k 1%, Resistor_SMD:R_0603_1608Metric, symbol Device:R
- removed R109: 60.4k 1%, Resistor_SMD:R_0603_1608Metric, symbol Device:R
- removed R110: 15k 1%, Resistor_SMD:R_0603_1608Metric, symbol Device:R
- removed R90: 1M 1%, Resistor_SMD:R_0603_1608Metric, symbol Device:R
- removed R91: 249k 1%, Resistor_SMD:R_0603_1608Metric, symbol Device:R
- C40: value 100nF 50V -> 1uF 50V X7R; MPN C2012X7R1H104K085AA -> C2012X7R1H105K125AB
- C42, C66: value 100nF 50V X7R -> 22nF 50V X7R; MPN C1608X7R1H104K080AA -> C1608X7R1H223K080AA
- U19: value LTC3115IDHD-1#PBF -> LTC3130IMSE-1#PBF; footprint Package_DFN_QFN:DFN-16-1EP_4x5mm_P0.5mm_EP2.44x4.34mm -> ScoringPlatform:LTC3130_MSE; symbol ScoringPlatform:LTC3115IDHD-1 -> ScoringPlatform:LTC3130IMSE-1; MPN LTC3115IDHD-1#PBF -> LTC3130IMSE-1#PBF
Connections:
- net USB_REG_FB is gone; now on net USB_REG_VCC: U19.7 (VCC)
- net USB_REG_RT is gone; now on net USB_REG_VCC: U19.8 (MPPC)
- net USB_REG_VC is gone; now on net USB_VBUS: U19.6 (RUN)
- net USB_GND: now also U19.1 (GND), U19.10 (VS1), U19.11 (MODE); no longer U19.16 (PWM_SYNC), U19.4 (GND), U19.5 (GND)
- net USB_PRIMARY_5V: now also U19.12 (EXTVCC), U19.14 (VOUT); no longer U19.3 (PVOUT)
- net USB_REG_BST1: now also U19.2 (BST1); no longer U19.13 (BST1)
- net USB_REG_BST2: now also U19.15 (BST2); no longer U19.12 (BST2)
- net USB_REG_SW1: now also U19.3 (SW1); no longer U19.15 (SW1)
- net USB_REG_SW2: now also U19.16 (SW2); no longer U19.2 (SW2)
- net USB_REG_VCC: no longer U19.11 (PVCC)
- net USB_VBUS: now also U19.4 (PVIN), U19.5 (VIN); no longer U19.1 (RUN), U19.10 (VIN), U19.14 (PVIN)
- no-connect marks 19 -> 20
Other:
- note added: "U19: LTC3130-1 fixed 5V buck-boost; MODE low selects automatic Burst/PWM. VS1=GND, VS2=VCC; 1uF VIN Kelvin bypass and 22nF bootstraps. U21 controls acquisition/application power; U18 remains LTM2884. Fixed-5V primary supply; no external compensation network."
- note removed: "U19: LTC3115-1 5V buck-boost; ADI Rev E front-page 750kHz reference network. Burst mode selected; no physical selector. Isolator U18 remains LTM2884. Input source qualification and automatic application-power control remain unfinished."

Commit message: fix(scoring): select stocked coupling and controller capacitors
Parts:
- C70: MPN C1608X5R1A105K080AC -> GRM188R61A105KA61D; Manufacturer TDK -> Murata
Changed lines of the file:
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@@
 (symbol (lib_id "Device:R") (at 341.63 260.35 0) (unit 1) (in_bom yes) (on_board yes) (dnp no) (property "Reference" "R116" (at 341.63 251.46000000000004 0) (effects (font (size 1 1)))) (property "Value" "47k 1%" (at 341.63 254.00000000000003 0) (effects (font (size 1 1)))) (property "Footprint" "Resistor_SMD:R_0603_1608Metric" (at 341.63 260.35 0) (effects (font (size 1 1)) (hide yes))) (property "Datasheet" "" (at 341.63 260.35 0) (effects (font (size 1 1)) (hide yes))) (property "Manufacturer" "YAGEO" (at 341.63 260.35 0) (effects (font (size 1 1)) (hide yes))) (property "MPN" "RC0603FR-0747KL" (at 341.63 260.35 0) (effects (font (size 1 1)) (hide yes))) (instances (project "usb-scoring-platform" (path "/20cc8167-128c-446a-a106-f942323e143f/972b77fe-bd38-49a7-88fc-3c741d64cdb1" (reference "R116") (unit 1)))) (pin "1") (pin "2"))
 (symbol (lib_id "Device:C") (at 391.16 260.35 0) (unit 1) (in_bom yes) (on_board yes) (dnp no) (property "Reference" "C69" (at 391.16 251.46000000000004 0) (effects (font (size 1 1)))) (property "Value" "100nF 50V" (at 391.16 254.00000000000003 0) (effects (font (size 1 1)))) (property "Footprint" "Capacitor_SMD:C_0603_1608Metric" (at 391.16 260.35 0) (effects (font (size 1 1)) (hide yes))) (property "Datasheet" "" (at 391.16 260.35 0) (effects (font (size 1 1)) (hide yes))) (property "Manufacturer" "TDK" (at 391.16 260.35 0) (effects (font (size 1 1)) (hide yes))) (property "MPN" "C1608X7R1H104K080AA" (at 391.16 260.35 0) (effects (font (size 1 1)) (hide yes))) (instances (project "usb-scoring-platform" (path "/20cc8167-128c-446a-a106-f942323e143f/972b77fe-bd38-49a7-88fc-3c741d64cdb1" (reference "C69") (unit 1)))) (pin "1") (pin "2"))
-(symbol (lib_id "Device:C") (at 391.16 299.72 0) (unit 1) (in_bom yes) (on_board yes) (dnp no) (property "Reference" "C70" (at 391.16 290.83000000000004 0) (effects (font (size 1 1)))) (property "Value" "1uF 10V" (at 391.16 293.37 0) (effects (font (size 1 1)))) (property "Footprint" "Capacitor_SMD:C_0603_1608Metric" (at 391.16 299.72 0) (effects (font (size 1 1)) (hide yes))) (property "Datasheet" "" (at 391.16 299.72 0) (effects (font (size 1 1)) (hide yes))) (property "Manufacturer" "TDK" (at 391.16 299.72 0) (effects (font (size 1 1)) (hide yes))) (property "MPN" "C1608X5R1A105K080AC" (at 391.16 299.72 0) (effects (font (size 1 1)) (hide yes))) (instances (project "usb-scoring-platform" (path "/20cc8167-128c-446a-a106-f942323e143f/972b77fe-bd38-49a7-88fc-3c741d64cdb1" (reference "C70") (unit 1)))) (pin "1") (pin "2"))
+(symbol (lib_id "Device:C") (at 391.16 299.72 0) (unit 1) (in_bom yes) (on_board yes) (dnp no) (property "Reference" "C70" (at 391.16 290.83000000000004 0) (effects (font (size 1 1)))) (property "Value" "1uF 10V" (at 391.16 293.37 0) (effects (font (size 1 1)))) (property "Footprint" "Capacitor_SMD:C_0603_1608Metric" (at 391.16 299.72 0) (effects (font (size 1 1)) (hide yes))) (property "Datasheet" "" (at 391.16 299.72 0) (effects (font (size 1 1)) (hide yes))) (property "Manufacturer" "Murata" (at 391.16 299.72 0) (effects (font (size 1 1)) (hide yes))) (property "MPN" "GRM188R61A105KA61D" (at 391.16 299.72 0) (effects (font (size 1 1)) (hide yes))) (instances (project "usb-scoring-platform" (path "/20cc8167-128c-446a-a106-f942323e143f/972b77fe-bd38-49a7-88fc-3c741d64cdb1" (reference "C70") (unit 1)))) (pin "1") (pin "2"))
 (symbol (lib_id "Device:C") (at 341.63 299.72 0) (unit 1) (in_bom yes) (on_board yes) (dnp no) (property "Reference" "C71" (at 341.63 290.83000000000004 0) (effects (font (size 1 1)))) (property "Value" "100nF 50V" (at 341.63 293.37 0) (effects (font (size 1 1)))) (property "Footprint" "Capacitor_SMD:C_0603_1608Metric" (at 341.63 299.72 0) (effects (font (size 1 1)) (hide yes))) (property "Datasheet" "" (at 341.63 299.72 0) (effects (font (size 1 1)) (hide yes))) (property "Manufacturer" "TDK" (at 341.63 299.72 0) (effects (font (size 1 1)) (hide yes))) (property "MPN" "C1608X7R1H104K080AA" (at 341.63 299.72 0) (effects (font (size 1 1)) (hide yes))) (instances (project "usb-scoring-platform" (path "/20cc8167-128c-446a-a106-f942323e143f/972b77fe-bd38-49a7-88fc-3c741d64cdb1" (reference "C71") (unit 1)))) (pin "1") (pin "2"))
 (symbol (lib_id "Connector_Generic:Conn_01x05") (at 457.2 275.59 0) (unit 1) (in_bom no) (on_board yes) (dnp no) (property "Reference" "J14" (at 457.2 253.58999999999997 0) (effects (font (size 1 1)))) (property "Value" "PRIMARY SWD PADS: 3V3 GND DIO CLK RESET" (at 457.2 256.09 0) (effects (font (size 1 1)))) (property "Footprint" "ScoringPlatform:Primary_SWD_Pads" (at 457.2 275.59 0) (effects (font (size 1 1)) (hide yes))) (property "Datasheet" "" (at 457.2 275.59 0) (effects (font (size 1 1)) (hide yes))) (property "Manufacturer" "PCB fabrication" (at 457.2 275.59 0) (effects (font (size 1 1)) (hide yes))) (property "MPN" "Not populated - service pads" (at 457.2 275.59 0) (effects (font (size 1 1)) (hide yes))) (instances (project "usb-scoring-platform" (path "/20cc8167-128c-446a-a106-f942323e143f/972b77fe-bd38-49a7-88fc-3c741d64cdb1" (reference "J14") (unit 1)))) (pin "1") (pin "2") (pin "3") (pin "4") (pin "5"))

Commit message: fix(scoring-circuit): source stocked bypass and reservoir capacitors
Parts:
- C48, C69, C71: MPN C1608X7R1H104K080AA -> CC0603KRX7R9BB104; Manufacturer TDK -> Yageo
