File: packages/scoring-circuit/virtual-scoring-box/left-weapon-inputs.kicad_sch (KiCad schematic)
At the start: 15 parts, among them J3 LEFT WEAPON A B C, U8 74LVC125APW

Commit message: feat(scoring-circuit): place virtual scoring box input and controller circuits
Parts:
- J3: footprint ScoringPlatform:Samtec_HTSW-103-07-L-S -> ScoringPlatform:Wire_Solder_3; MPN HTSW-103-07-L-S -> PCB solder termination; Manufacturer Samtec -> PCB; now left out of the parts list
