File: packages/scoring-circuit/virtual-scoring-box/right-and-piste-inputs.kicad_sch (KiCad schematic)
At the start: 20 parts, among them J4 RIGHT WEAPON A B C, J5 PISTE - NOT protective earth, U9 74LVC125APW

Commit message: feat(scoring-circuit): place virtual scoring box input and controller circuits
Parts:
- J4: footprint ScoringPlatform:Samtec_HTSW-103-07-L-S -> ScoringPlatform:Wire_Solder_3; MPN HTSW-103-07-L-S -> PCB solder termination; Manufacturer Samtec -> PCB; now left out of the parts list
- J5: footprint ScoringPlatform:Samtec_HTSW-101-07-L-S -> ScoringPlatform:Wire_Solder_1; MPN HTSW-101-07-L-S -> PCB solder termination; Manufacturer Samtec -> PCB; now left out of the parts list
