File: packages/scoring-circuit/virtual-scoring-box/acquisition-controller.kicad_sch (KiCad schematic)
At the start: 19 parts, among them J2 STM SWD 3.3V, SW1 STM RESET, U1 STM32G474RET6, Y1 ABM3B-8.000MHZ-B2-T

Commit message: feat(scoring-circuit): place virtual scoring box input and controller circuits
Connections:
- net FAVERO_TX: no longer names the net of U1.14 (PA2)
- net SOUNDER_PWM: no longer names the net of U1.42 (PA8)
- no-connect marks 18 -> 20

Commit message: feat(scoring-circuit): add suspend-aware isolated serial interface
Connections:
- net LAPTOP_UART_TX: now reaches U1.14 (PA2)
- net LAPTOP_UART_RX: now reaches U1.51 (PA15)
- net USB_DM: no longer names the net of U1.45 (PA11)
- net USB_DP: no longer names the net of U1.46 (PA12)
- net USB_PRESENT: no longer names the net of U1.58 (PB5)
- no-connect marks 20 -> 21
Other:
- note added: "Virtual box laptop link: USART2 PA2(TX) / PA15(RX), AF7, through U19 to U18. USB PA11/PA12 are not used. SWD and USART1 PA9/PA10 to ESP32 are unchanged."

Commit message: fix(scoring-circuit): correct virtual-box assembly part matching
Parts:
- C15, C33: JLCPCB (none) -> C45537494
Changed lines of the file:
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@@
 (wire (pts (xy 180.34 133.35) (xy 180.34 138.43)) (stroke (width 0) (type default)))
 (global_label "GND" (shape bidirectional) (at 180.34 138.43 0) (effects (font (size 0.9 0.9)) (justify left)) (property "Intersheetrefs" "" (at 180.34 138.43 0) (effects (font (size 1 1)) (hide yes))))
-(symbol (lib_id "Device:C") (at 240.03 129.54 0) (unit 1) (in_bom yes) (on_board yes) (dnp no) (property "Reference" "C15" (at 240.03 115.54 0) (effects (font (size 1.2 1.2)))) (property "Value" "1uF 10V" (at 240.03 117.54 0) (effects (font (size 1.1 1.1)))) (property "Footprint" "Capacitor_SMD:C_0603_1608Metric" (at 240.03 129.54 0) (effects (font (size 1 1)) (hide yes))) (pin "1") (pin "2") (property "Manufacturer" "TDK" (at 240.03 129.54 0) (effects (font (size 1 1)) (hide yes))) (property "MPN" "C1608X7R1H105K080AB" (at 240.03 129.54 0) (effects (font (size 1 1)) (hide yes))) (property "Datasheet" "https://product.tdk.com/en/search/capacitor/ceramic/mlcc/info?part_no=C1608X7R1H105K080AB" (at 240.03 129.54 0) (effects (font (size 1 1)) (hide yes))) (instances (project "virtual-scoring-box" (path "/20cc8167-128c-446a-a106-f942323e143f/edc47c5d-79f6-4e87-a428-cb43ded9ee70" (reference "C15") (unit 1)))))
+(symbol (lib_id "Device:C") (at 240.03 129.54 0) (unit 1) (in_bom yes) (on_board yes) (dnp no) (property "Reference" "C15" (at 240.03 115.54 0) (effects (font (size 1.2 1.2)))) (property "Value" "1uF 10V" (at 240.03 117.54 0) (effects (font (size 1.1 1.1)))) (property "Footprint" "Capacitor_SMD:C_0603_1608Metric" (at 240.03 129.54 0) (effects (font (size 1 1)) (hide yes))) (pin "1") (pin "2") (property "Manufacturer" "TDK" (at 240.03 129.54 0) (effects (font (size 1 1)) (hide yes))) (property "MPN" "C1608X7R1H105K080AB" (at 240.03 129.54 0) (effects (font (size 1 1)) (hide yes))) (property "JLCPCB" "C45537494" (at 240.03 129.54 0) (effects (font (size 1 1)) (hide yes))) (property "Datasheet" "https://product.tdk.com/en/search/capacitor/ceramic/mlcc/info?part_no=C1608X7R1H105K080AB" (at 240.03 129.54 0) (effects (font (size 1 1)) (hide yes))) (instances (project "virtual-scoring-box" (path "/20cc8167-128c-446a-a106-f942323e143f/edc47c5d-79f6-4e87-a428-cb43ded9ee70" (reference "C15") (unit 1)))))
 (wire (pts (xy 240.03 125.73) (xy 240.03 120.65)) (stroke (width 0) (type default)))
 (global_label "CORE_3V3" (shape bidirectional) (at 240.03 120.65 0) (effects (font (size 0.9 0.9)) (justify left)) (property "Intersheetrefs" "" (at 240.03 120.65 0) (effects (font (size 1 1)) (hide yes))))
@@
 (text "Continuity characterization: COMP1/2/3/4/5/6/7 = PA1/PA3/PA0/PB0/PB13/PB11/PB14.\nUse internal VREFINT/2 and HYST=1; allow 205us startup before observations.\nSwitch drives with observation blanking and active-low cable discharge. Full weapon scan/timing remains open." (at 180 240 0) (effects (font (size 1.1 1.1)) (justify left top)))
 (text "STM32 acquisition, USB and standalone scoring" (at 20 15 0) (effects (font (size 2 2)) (justify left top)))
-(symbol (lib_id "Device:C") (at 299.72 129.54 0) (unit 1) (in_bom yes) (on_board yes) (dnp no) (property "Reference" "C33" (at 299.72 115.54 0) (effects (font (size 1.2 1.2)))) (property "Value" "1uF 10V" (at 299.72 117.54 0) (effects (font (size 1.1 1.1)))) (property "Footprint" "Capacitor_SMD:C_0603_1608Metric" (at 299.72 129.54 0) (effects (font (size 1 1)) (hide yes))) (pin "1") (pin "2") (property "Manufacturer" "TDK" (at 299.72 129.54 0) (effects (font (size 1 1)) (hide yes))) (property "MPN" "C1608X7R1H105K080AB" (at 299.72 129.54 0) (effects (font (size 1 1)) (hide yes))) (property "Datasheet" "https://product.tdk.com/en/search/capacitor/ceramic/mlcc/info?part_no=C1608X7R1H105K080AB" (at 299.72 129.54 0) (effects (font (size 1 1)) (hide yes))) (instances (project "virtual-scoring-box" (path "/20cc8167-128c-446a-a106-f942323e143f/edc47c5d-79f6-4e87-a428-cb43ded9ee70" (reference "C33") (unit 1)))))
+(symbol (lib_id "Device:C") (at 299.72 129.54 0) (unit 1) (in_bom yes) (on_board yes) (dnp no) (property "Reference" "C33" (at 299.72 115.54 0) (effects (font (size 1.2 1.2)))) (property "Value" "1uF 10V" (at 299.72 117.54 0) (effects (font (size 1.1 1.1)))) (property "Footprint" "Capacitor_SMD:C_0603_1608Metric" (at 299.72 129.54 0) (effects (font (size 1 1)) (hide yes))) (pin "1") (pin "2") (property "Manufacturer" "TDK" (at 299.72 129.54 0) (effects (font (size 1 1)) (hide yes))) (property "MPN" "C1608X7R1H105K080AB" (at 299.72 129.54 0) (effects (font (size 1 1)) (hide yes))) (property "JLCPCB" "C45537494" (at 299.72 129.54 0) (effects (font (size 1 1)) (hide yes))) (property "Datasheet" "https://product.tdk.com/en/search/capacitor/ceramic/mlcc/info?part_no=C1608X7R1H105K080AB" (at 299.72 129.54 0) (effects (font (size 1 1)) (hide yes))) (instances (project "virtual-scoring-box" (path "/20cc8167-128c-446a-a106-f942323e143f/edc47c5d-79f6-4e87-a428-cb43ded9ee70" (reference "C33") (unit 1)))))
 (wire (pts (xy 299.72 125.73) (xy 299.72 120.65)) (stroke (width 0) (type default)))
 (global_label "CORE_3V3" (shape bidirectional) (at 299.72 120.65 0) (effects (font (size 0.9 0.9)) (justify left)) (property "Intersheetrefs" "" (at 299.72 120.65 0) (effects (font (size 1 1)) (hide yes))))

Commit message: fix(scoring-circuit): resolve prototype sourcing gaps
Parts:
- C12: JLCPCB (none) -> C100042; MPN C1608X7R1H103K080AA -> CC0603KRX7R9BB103; Manufacturer TDK -> YAGEO
- C14: JLCPCB (none) -> C342959; MPN C1608X7S1A475K080AC -> C1608X7S1A475KT000E
- C15, C33: JLCPCB C45537494 -> C559769; MPN C1608X7R1H105K080AB -> CC0603KRX7R9BB105; Manufacturer TDK -> YAGEO
- C17, C18: JLCPCB (none) -> C107045; MPN CGA3E2C0G1H270J080AA -> CC0603JRNPO9BN270; Manufacturer TDK -> YAGEO
- J2: JLCPCB (none) -> C3337223; MPN HTSW-105-07-L-S -> HTSW-105-07-G-S
