File: packages/scoring-circuit/virtual-scoring-box/application-controller.kicad_sch (KiCad schematic)
At the start: 19 parts, among them J6 ESP 3.3V UART recovery, SW2 ESP RESET, SW3 ESP BOOT, U10 SN74AXC1T45DCKR, U11 SN74AXC1T45DCKR, U2 ESP32-S3-WROOM-1-N8R8

Commit message: feat(scoring-circuit): place virtual scoring box input and controller circuits
Connections:
- net DISPLAY_ENABLE: no longer names the net of U2.23 (IO21)
- net ETH_CS_N: no longer names the net of U2.32 (IO39)
- net ETH_IRQ_N: no longer names the net of U2.33 (IO40)
- net ETH_MISO: no longer names the net of U2.31 (IO38)
- net ETH_MOSI: no longer names the net of U2.21 (IO13)
- net ETH_RESET_N: no longer names the net of U2.34 (IO41)
- net ETH_SCLK: no longer names the net of U2.22 (IO14)
- net RGB_A: no longer names the net of U2.10 (IO17)
- net RGB_B: no longer names the net of U2.11 (IO18)
- net RGB_B1: no longer names the net of U2.6 (IO6)
- net RGB_B2: no longer names the net of U2.9 (IO16)
- net RGB_C: no longer names the net of U2.12 (IO8)
- net RGB_CLK: no longer names the net of U2.18 (IO10)
- net RGB_D: no longer names the net of U2.17 (IO9)
- net RGB_G1: no longer names the net of U2.5 (IO5)
- net RGB_G2: no longer names the net of U2.8 (IO15)
- net RGB_LAT: no longer names the net of U2.19 (IO11)
- net RGB_OE: no longer names the net of U2.20 (IO12)
- net RGB_R1: no longer names the net of U2.4 (IO4)
- net RGB_R2: no longer names the net of U2.7 (IO7)
- no-connect marks 10 -> 30
Changed lines of the file:
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@@
 (wire (pts (xy 64.77 77.47) (xy 59.69 77.47)) (stroke (width 0) (type default)))
 (global_label "ESP_EN" (shape bidirectional) (at 59.69 77.47 180) (effects (font (size 0.9 0.9)) (justify right)) (property "Intersheetrefs" "" (at 59.69 77.47 180) (effects (font (size 1 1)) (hide yes))))
-(wire (pts (xy 64.77 92.71) (xy 59.69 92.71)) (stroke (width 0) (type default)))
-(global_label "RGB_R1" (shape bidirectional) (at 59.69 92.71 180) (effects (font (size 0.9 0.9)) (justify right)) (property "Intersheetrefs" "" (at 59.69 92.71 180) (effects (font (size 1 1)) (hide yes))))
-(wire (pts (xy 64.77 95.25) (xy 59.69 95.25)) (stroke (width 0) (type default)))
-(global_label "RGB_G1" (shape bidirectional) (at 59.69 95.25 180) (effects (font (size 0.9 0.9)) (justify right)) (property "Intersheetrefs" "" (at 59.69 95.25 180) (effects (font (size 1 1)) (hide yes))))
-(wire (pts (xy 64.77 97.79) (xy 59.69 97.79)) (stroke (width 0) (type default)))
-(global_label "RGB_B1" (shape bidirectional) (at 59.69 97.79 180) (effects (font (size 0.9 0.9)) (justify right)) (property "Intersheetrefs" "" (at 59.69 97.79 180) (effects (font (size 1 1)) (hide yes))))
-(wire (pts (xy 64.77 100.33) (xy 59.69 100.33)) (stroke (width 0) (type default)))
-(global_label "RGB_R2" (shape bidirectional) (at 59.69 100.33 180) (effects (font (size 0.9 0.9)) (justify right)) (property "Intersheetrefs" "" (at 59.69 100.33 180) (effects (font (size 1 1)) (hide yes))))
-(wire (pts (xy 64.77 120.65) (xy 59.69 120.65)) (stroke (width 0) (type default)))
-(global_label "RGB_G2" (shape bidirectional) (at 59.69 120.65 180) (effects (font (size 0.9 0.9)) (justify right)) (property "Intersheetrefs" "" (at 59.69 120.65 180) (effects (font (size 1 1)) (hide yes))))
-(wire (pts (xy 64.77 123.19) (xy 59.69 123.19)) (stroke (width 0) (type default)))
-(global_label "RGB_B2" (shape bidirectional) (at 59.69 123.19 180) (effects (font (size 0.9 0.9)) (justify right)) (property "Intersheetrefs" "" (at 59.69 123.19 180) (effects (font (size 1 1)) (hide yes))))
-(wire (pts (xy 95.25 82.55) (xy 100.33 82.55)) (stroke (width 0) (type default)))
-(global_label "RGB_A" (shape bidirectional) (at 100.33 82.55 0) (effects (font (size 0.9 0.9)) (justify left)) (property "Intersheetrefs" "" (at 100.33 82.55 0) (effects (font (size 1 1)) (hide yes))))
-(wire (pts (xy 95.25 85.09) (xy 100.33 85.09)) (stroke (width 0) (type default)))
-(global_label "RGB_B" (shape bidirectional) (at 100.33 85.09 0) (effects (font (size 0.9 0.9)) (justify left)) (property "Intersheetrefs" "" (at 100.33 85.09 0) (effects (font (size 1 1)) (hide yes))))
-(wire (pts (xy 64.77 102.87) (xy 59.69 102.87)) (stroke (width 0) (type default)))
-(global_label "RGB_C" (shape bidirectional) (at 59.69 102.87 180) (effects (font (size 0.9 0.9)) (justify right)) (property "Intersheetrefs" "" (at 59.69 102.87 180) (effects (font (size 1 1)) (hide yes))))
+(no_connect (at 64.77 92.71))
+(no_connect (at 64.77 95.25))
+(no_connect (at 64.77 97.79))
+(no_connect (at 64.77 100.33))
+(no_connect (at 64.77 120.65))
+(no_connect (at 64.77 123.19))
+(no_connect (at 95.25 82.55))
+(no_connect (at 95.25 85.09))
+(no_connect (at 64.77 102.87))
 (no_connect (at 95.25 87.63))
 (no_connect (at 95.25 90.17))
 (no_connect (at 64.77 90.17))
 (no_connect (at 95.25 118.11))
-(wire (pts (xy 64.77 105.41) (xy 59.69 105.41)) (stroke (width 0) (type default)))
-(global_label "RGB_D" (shape bidirectional) (at 59.69 105.41 180) (effects (font (size 0.9 0.9)) (justify right)) (property "Intersheetrefs" "" (at 59.69 105.41 180) (effects (font (size 1 1)) (hide yes))))
-(wire (pts (xy 64.77 107.95) (xy 59.69 107.95)) (stroke (width 0) (type default)))
-(global_label "RGB_CLK" (shape bidirectional) (at 59.69 107.95 180) (effects (font (size 0.9 0.9)) (justify right)) (property "Intersheetrefs" "" (at 59.69 107.95 180) (effects (font (size 1 1)) (hide yes))))
-(wire (pts (xy 64.77 110.49) (xy 59.69 110.49)) (stroke (width 0) (type default)))
-(global_label "RGB_LAT" (shape bidirectional) (at 59.69 110.49 180) (effects (font (size 0.9 0.9)) (justify right)) (property "Intersheetrefs" "" (at 59.69 110.49 180) (effects (font (size 1 1)) (hide yes))))
-(wire (pts (xy 64.77 113.03) (xy 59.69 113.03)) (stroke (width 0) (type default)))
-(global_label "RGB_OE" (shape bidirectional) (at 59.69 113.03 180) (effects (font (size 0.9 0.9)) (justify right)) (property "Intersheetrefs" "" (at 59.69 113.03 180) (effects (font (size 1 1)) (hide yes))))
-(wire (pts (xy 64.77 115.57) (xy 59.69 115.57)) (stroke (width 0) (type default)))
-(global_label "ETH_MOSI" (shape bidirectional) (at 59.69 115.57 180) (effects (font (size 0.9 0.9)) (justify right)) (property "Intersheetrefs" "" (at 59.69 115.57 180) (effects (font (size 1 1)) (hide yes))))
-(wire (pts (xy 64.77 118.11) (xy 59.69 118.11)) (stroke (width 0) (type default)))
-(global_label "ETH_SCLK" (shape bidirectional) (at 59.69 118.11 180) (effects (font (size 0.9 0.9)) (justify right)) (property "Intersheetrefs" "" (at 59.69 118.11 180) (effects (font (size 1 1)) (hide yes))))
-(wire (pts (xy 95.25 92.71) (xy 100.33 92.71)) (stroke (width 0) (type default)))
-(global_label "DISPLAY_ENABLE" (shape bidirectional) (at 100.33 92.71 0) (effects (font (size 0.9 0.9)) (justify left)) (property "Intersheetrefs" "" (at 100.33 92.71 0) (effects (font (size 1 1)) (hide yes))))
+(no_connect (at 64.77 105.41))
+(no_connect (at 64.77 107.95))
+(no_connect (at 64.77 110.49))
+(no_connect (at 64.77 113.03))
+(no_connect (at 64.77 115.57))
+(no_connect (at 64.77 118.11))
+(no_connect (at 95.25 92.71))
 (wire (pts (xy 95.25 120.65) (xy 100.33 120.65)) (stroke (width 0) (type default)))
 (global_label "ESP_TX" (shape bidirectional) (at 100.33 120.65 0) (effects (font (size 0.9 0.9)) (justify left)) (property "Intersheetrefs" "" (at 100.33 120.65 0) (effects (font (size 1 1)) (hide yes))))
@@
 (no_connect (at 95.25 97.79))
 (no_connect (at 95.25 100.33))
-(wire (pts (xy 95.25 102.87) (xy 100.33 102.87)) (stroke (width 0) (type default)))
-(global_label "ETH_MISO" (shape bidirectional) (at 100.33 102.87 0) (effects (font (size 0.9 0.9)) (justify left)) (property "Intersheetrefs" "" (at 100.33 102.87 0) (effects (font (size 1 1)) (hide yes))))
-(wire (pts (xy 95.25 105.41) (xy 100.33 105.41)) (stroke (width 0) (type default)))
-(global_label "ETH_CS_N" (shape bidirectional) (at 100.33 105.41 0) (effects (font (size 0.9 0.9)) (justify left)) (property "Intersheetrefs" "" (at 100.33 105.41 0) (effects (font (size 1 1)) (hide yes))))
-(wire (pts (xy 95.25 107.95) (xy 100.33 107.95)) (stroke (width 0) (type default)))
-(global_label "ETH_IRQ_N" (shape bidirectional) (at 100.33 107.95 0) (effects (font (size 0.9 0.9)) (justify left)) (property "Intersheetrefs" "" (at 100.33 107.95 0) (effects (font (size 1 1)) (hide yes))))
-(wire (pts (xy 95.25 110.49) (xy 100.33 110.49)) (stroke (width 0) (type default)))
-(global_label "ETH_RESET_N" (shape bidirectional) (at 100.33 110.49 0) (effects (font (size 0.9 0.9)) (justify left)) (property "Intersheetrefs" "" (at 100.33 110.49 0) (effects (font (size 1 1)) (hide yes))))
+(no_connect (at 95.25 102.87))
+(no_connect (at 95.25 105.41))
+(no_connect (at 95.25 107.95))
+(no_connect (at 95.25 110.49))
 (wire (pts (xy 95.25 113.03) (xy 100.33 113.03)) (stroke (width 0) (type default)))
 (global_label "IR_RX" (shape bidirectional) (at 100.33 113.03 0) (effects (font (size 0.9 0.9)) (justify left)) (property "Intersheetrefs" "" (at 100.33 113.03 0) (effects (font (size 1 1)) (hide yes))))

Commit message: feat(scoring-circuit): add virtual box USB interface and signal routing checkpoint
Parts:
- U2: footprint RF_Module:ESP32-S3-WROOM-1 -> ScoringPlatform:ESP32-S3-WROOM-1_Edge
Changed lines of the file:
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@@
 (paper "A3")
 (title_block (title "ESP32 wireless and remote controller") (rev "Engineering draft") (comment 1 "NOT FOR FABRICATION"))
-(symbol (lib_id "RF_Module:ESP32-S3-WROOM-1") (at 80.01 100.33 0) (unit 1) (in_bom yes) (on_board yes) (dnp no) (property "Reference" "U2" (at 80.01 63.39 0) (effects (font (size 1.2 1.2)))) (property "Value" "ESP32-S3-WROOM-1-N8R8" (at 80.01 65.39 0) (effects (font (size 1.1 1.1)))) (property "Footprint" "RF_Module:ESP32-S3-WROOM-1" (at 80.01 100.33 0) (effects (font (size 1 1)) (hide yes))) (pin "1") (pin "2") (pin "3") (pin "4") (pin "5") (pin "6") (pin "7") (pin "8") (pin "9") (pin "10") (pin "11") (pin "12") (pin "13") (pin "14") (pin "15") (pin "16") (pin "17") (pin "18") (pin "19") (pin "20") (pin "21") (pin "22") (pin "23") (pin "24") (pin "25") (pin "26") (pin "27") (pin "28") (pin "29") (pin "30") (pin "31") (pin "32") (pin "33") (pin "34") (pin "35") (pin "36") (pin "37") (pin "38") (pin "39") (pin "40") (pin "41") (instances (project "virtual-scoring-box" (path "/20cc8167-128c-446a-a106-f942323e143f/97185045-65e6-4b5b-a06d-6bdd67041229" (reference "U2") (unit 1)))) (property "Manufacturer" "Espressif Systems" (at 0 0 0) (effects (font (size 1 1)) (hide yes))) (property "MPN" "ESP32-S3-WROOM-1-N8R8" (at 0 0 0) (effects (font (size 1 1)) (hide yes))))
+(symbol (lib_id "RF_Module:ESP32-S3-WROOM-1") (at 80.01 100.33 0) (unit 1) (in_bom yes) (on_board yes) (dnp no) (property "Reference" "U2" (at 80.01 63.39 0) (effects (font (size 1.2 1.2)))) (property "Value" "ESP32-S3-WROOM-1-N8R8" (at 80.01 65.39 0) (effects (font (size 1.1 1.1)))) (property "Footprint" "ScoringPlatform:ESP32-S3-WROOM-1_Edge" (at 80.01 100.33 0) (effects (font (size 1 1)) (hide yes))) (pin "1") (pin "2") (pin "3") (pin "4") (pin "5") (pin "6") (pin "7") (pin "8") (pin "9") (pin "10") (pin "11") (pin "12") (pin "13") (pin "14") (pin "15") (pin "16") (pin "17") (pin "18") (pin "19") (pin "20") (pin "21") (pin "22") (pin "23") (pin "24") (pin "25") (pin "26") (pin "27") (pin "28") (pin "29") (pin "30") (pin "31") (pin "32") (pin "33") (pin "34") (pin "35") (pin "36") (pin "37") (pin "38") (pin "39") (pin "40") (pin "41") (instances (project "virtual-scoring-box" (path "/20cc8167-128c-446a-a106-f942323e143f/97185045-65e6-4b5b-a06d-6bdd67041229" (reference "U2") (unit 1)))) (property "Manufacturer" "Espressif Systems" (at 0 0 0) (effects (font (size 1 1)) (hide yes))) (property "MPN" "ESP32-S3-WROOM-1-N8R8" (at 0 0 0) (effects (font (size 1 1)) (hide yes))))
 (wire (pts (xy 80.01 128.27) (xy 80.01 133.35)) (stroke (width 0) (type default)))
 (global_label "GND" (shape bidirectional) (at 80.01 133.35 0) (effects (font (size 0.9 0.9)) (justify left)) (property "Intersheetrefs" "" (at 80.01 133.35 0) (effects (font (size 1 1)) (hide yes))))

Commit message: feat(scoring-circuit): integrate isolated virtual-box processor supply
Connections:
- net APP_3V3 is gone; now on net CORE_3V3: C22.1, C23.1, C25.1, C27.1, J6.1 (Pin_1), R28.1, R29.1, R31.1, R73.1, U10.6 (VCCB), U11.6 (VCCB), U2.2 (3V3)

Commit message: feat(scoring-circuit): simplify virtual-box UART and export assembly handoff
Parts:
- removed C23, C24, C25, C26: 100nF 10V, Capacitor_SMD:C_0603_1608Metric, symbol Device:C
- removed R30, R31: 47k, Resistor_SMD:R_0603_1608Metric, symbol Device:R
- removed U10, U11: SN74AXC1T45DCKR, ScoringPlatform:SN74AXC1T45DCKR, symbol ScoringPlatform:SN74AXC1T45DCKR
Connections:
- net ESP_RX is gone; now on net STM_TX: U2.25 (IO48)
- net ESP_TX is gone; now on net STM_RX: R73.2, U2.24 (IO47)
Other:
- note added: "ESP32-S3-WROOM-1-N8R8: GPIO35/36/37 reserved for octal PSRAM. STM32 owns contact timing. Both processors share CORE_3V3; the UART is connected directly."
- note added: "R72/R73 hold the two UART lines high during reset. C22/C27 decouple ESP32 supply. Do not inject programmer power into either processor rail."
- note removed: "ESP32-S3-WROOM-1-N8R8: GPIO35/36/37 reserved for octal PSRAM. STM32 owns contact timing. UART parts prevent powered-off domain backfeeding, not galvanic isolation."
- note removed: "R72/R73 hold each transmitter high during reset; R30/R31 keep receivers idle when the opposite rail is off. Each pull references its own processor supply."
- moved on the sheet: C27

Commit message: fix(scoring-circuit): correct virtual-box assembly part matching
Parts:
- C21: JLCPCB (none) -> C45537494
Changed lines of the file:
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@@
 (wire (pts (xy 160.02 48.26) (xy 160.02 53.34)) (stroke (width 0) (type default)))
 (global_label "ESP_EN" (shape bidirectional) (at 160.02 53.34 0) (effects (font (size 0.9 0.9)) (justify left)) (property "Intersheetrefs" "" (at 160.02 53.34 0) (effects (font (size 1 1)) (hide yes))))
-(symbol (lib_id "Device:C") (at 199.39 44.45 0) (unit 1) (in_bom yes) (on_board yes) (dnp no) (property "Reference" "C21" (at 199.39 30.45 0) (effects (font (size 1.2 1.2)))) (property "Value" "1uF 10V" (at 199.39 32.45 0) (effects (font (size 1.1 1.1)))) (property "Footprint" "Capacitor_SMD:C_0603_1608Metric" (at 199.39 44.45 0) (effects (font (size 1 1)) (hide yes))) (pin "1") (pin "2") (property "Manufacturer" "TDK" (at 199.39 44.45 0) (effects (font (size 1 1)) (hide yes))) (property "MPN" "C1608X7R1H105K080AB" (at 199.39 44.45 0) (effects (font (size 1 1)) (hide yes))) (property "Datasheet" "https://product.tdk.com/en/search/capacitor/ceramic/mlcc/info?part_no=C1608X7R1H105K080AB" (at 199.39 44.45 0) (effects (font (size 1 1)) (hide yes))) (instances (project "virtual-scoring-box" (path "/20cc8167-128c-446a-a106-f942323e143f/97185045-65e6-4b5b-a06d-6bdd67041229" (reference "C21") (unit 1)))))
+(symbol (lib_id "Device:C") (at 199.39 44.45 0) (unit 1) (in_bom yes) (on_board yes) (dnp no) (property "Reference" "C21" (at 199.39 30.45 0) (effects (font (size 1.2 1.2)))) (property "Value" "1uF 10V" (at 199.39 32.45 0) (effects (font (size 1.1 1.1)))) (property "Footprint" "Capacitor_SMD:C_0603_1608Metric" (at 199.39 44.45 0) (effects (font (size 1 1)) (hide yes))) (pin "1") (pin "2") (property "Manufacturer" "TDK" (at 199.39 44.45 0) (effects (font (size 1 1)) (hide yes))) (property "MPN" "C1608X7R1H105K080AB" (at 199.39 44.45 0) (effects (font (size 1 1)) (hide yes))) (property "JLCPCB" "C45537494" (at 199.39 44.45 0) (effects (font (size 1 1)) (hide yes))) (property "Datasheet" "https://product.tdk.com/en/search/capacitor/ceramic/mlcc/info?part_no=C1608X7R1H105K080AB" (at 199.39 44.45 0) (effects (font (size 1 1)) (hide yes))) (instances (project "virtual-scoring-box" (path "/20cc8167-128c-446a-a106-f942323e143f/97185045-65e6-4b5b-a06d-6bdd67041229" (reference "C21") (unit 1)))))
 (wire (pts (xy 199.39 40.64) (xy 199.39 35.56)) (stroke (width 0) (type default)))
 (global_label "ESP_EN" (shape bidirectional) (at 199.39 35.56 0) (effects (font (size 0.9 0.9)) (justify left)) (property "Intersheetrefs" "" (at 199.39 35.56 0) (effects (font (size 1 1)) (hide yes))))
