File: packages/scoring-circuit/virtual-scoring-box/application-controller.kicad_sch (KiCad schematic)
At the start: 11 parts, among them J6 ESP 3.3V UART recovery, SW2 ESP RESET, SW3 ESP BOOT, U2 ESP32-S3-WROOM-1-N8R8

Commit message: fix(scoring-circuit): resolve prototype sourcing gaps
Parts:
- C21: JLCPCB C45537494 -> C559769; MPN C1608X7R1H105K080AB -> CC0603KRX7R9BB105; Manufacturer TDK -> YAGEO
- C22: JLCPCB (none) -> C342854; MPN C1608X5R1C106M080AB -> C1608X5R1C106MT000N
- J6: JLCPCB (none) -> C3334125; MPN HTSW-106-07-L-S -> HTSW-106-07-G-S
Changed lines of the file:
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@@
 (wire (pts (xy 160.02 48.26) (xy 160.02 53.34)) (stroke (width 0) (type default)))
 (global_label "ESP_EN" (shape bidirectional) (at 160.02 53.34 0) (effects (font (size 0.9 0.9)) (justify left)) (property "Intersheetrefs" "" (at 160.02 53.34 0) (effects (font (size 1 1)) (hide yes))))
-(symbol (lib_id "Device:C") (at 199.39 44.45 0) (unit 1) (in_bom yes) (on_board yes) (dnp no) (property "Reference" "C21" (at 199.39 30.45 0) (effects (font (size 1.2 1.2)))) (property "Value" "1uF 10V" (at 199.39 32.45 0) (effects (font (size 1.1 1.1)))) (property "Footprint" "Capacitor_SMD:C_0603_1608Metric" (at 199.39 44.45 0) (effects (font (size 1 1)) (hide yes))) (pin "1") (pin "2") (property "Manufacturer" "TDK" (at 199.39 44.45 0) (effects (font (size 1 1)) (hide yes))) (property "MPN" "C1608X7R1H105K080AB" (at 199.39 44.45 0) (effects (font (size 1 1)) (hide yes))) (property "JLCPCB" "C45537494" (at 199.39 44.45 0) (effects (font (size 1 1)) (hide yes))) (property "Datasheet" "https://product.tdk.com/en/search/capacitor/ceramic/mlcc/info?part_no=C1608X7R1H105K080AB" (at 199.39 44.45 0) (effects (font (size 1 1)) (hide yes))) (instances (project "virtual-scoring-box" (path "/20cc8167-128c-446a-a106-f942323e143f/97185045-65e6-4b5b-a06d-6bdd67041229" (reference "C21") (unit 1)))))
+(symbol (lib_id "Device:C") (at 199.39 44.45 0) (unit 1) (in_bom yes) (on_board yes) (dnp no) (property "Reference" "C21" (at 199.39 30.45 0) (effects (font (size 1.2 1.2)))) (property "Value" "1uF 10V" (at 199.39 32.45 0) (effects (font (size 1.1 1.1)))) (property "Footprint" "Capacitor_SMD:C_0603_1608Metric" (at 199.39 44.45 0) (effects (font (size 1 1)) (hide yes))) (pin "1") (pin "2") (property "Manufacturer" "YAGEO" (at 199.39 44.45 0) (effects (font (size 1 1)) (hide yes))) (property "MPN" "CC0603KRX7R9BB105" (at 199.39 44.45 0) (effects (font (size 1 1)) (hide yes))) (property "JLCPCB" "C559769" (at 199.39 44.45 0) (effects (font (size 1 1)) (hide yes))) (property "Datasheet" "https://yageogroup.com/download/specsheet/CC0603KRX7R9BB105" (at 199.39 44.45 0) (effects (font (size 1 1)) (hide yes))) (instances (project "virtual-scoring-box" (path "/20cc8167-128c-446a-a106-f942323e143f/97185045-65e6-4b5b-a06d-6bdd67041229" (reference "C21") (unit 1)))))
 (wire (pts (xy 199.39 40.64) (xy 199.39 35.56)) (stroke (width 0) (type default)))
 (global_label "ESP_EN" (shape bidirectional) (at 199.39 35.56 0) (effects (font (size 0.9 0.9)) (justify left)) (property "Intersheetrefs" "" (at 199.39 35.56 0) (effects (font (size 1 1)) (hide yes))))
@@
 (wire (pts (xy 240.03 48.26) (xy 240.03 53.34)) (stroke (width 0) (type default)))
 (global_label "ESP_BOOT0" (shape bidirectional) (at 240.03 53.34 0) (effects (font (size 0.9 0.9)) (justify left)) (property "Intersheetrefs" "" (at 240.03 53.34 0) (effects (font (size 1 1)) (hide yes))))
-(symbol (lib_id "Device:C") (at 160.02 90.17 0) (unit 1) (in_bom yes) (on_board yes) (dnp no) (property "Reference" "C22" (at 160.02 76.17 0) (effects (font (size 1.2 1.2)))) (property "Value" "10uF 10V" (at 160.02 78.17 0) (effects (font (size 1.1 1.1)))) (property "Footprint" "Capacitor_SMD:C_0603_1608Metric" (at 160.02 90.17 0) (effects (font (size 1 1)) (hide yes))) (pin "1") (pin "2") (property "Manufacturer" "TDK" (at 0 0 0) (effects (font (size 1 1)) (hide yes))) (property "MPN" "C1608X5R1C106M080AB" (at 0 0 0) (effects (font (size 1 1)) (hide yes))) (property "Datasheet" "https://product.tdk.com/en/search/capacitor/ceramic/mlcc/info?part_no=C1608X5R1C106M080AB" (at 0 0 0) (effects (font (size 1 1)) (hide yes))) (instances (project "virtual-scoring-box" (path "/20cc8167-128c-446a-a106-f942323e143f/97185045-65e6-4b5b-a06d-6bdd67041229" (reference "C22") (unit 1)))))
+(symbol (lib_id "Device:C") (at 160.02 90.17 0) (unit 1) (in_bom yes) (on_board yes) (dnp no) (property "Reference" "C22" (at 160.02 76.17 0) (effects (font (size 1.2 1.2)))) (property "Value" "10uF 10V" (at 160.02 78.17 0) (effects (font (size 1.1 1.1)))) (property "Footprint" "Capacitor_SMD:C_0603_1608Metric" (at 160.02 90.17 0) (effects (font (size 1 1)) (hide yes))) (pin "1") (pin "2") (property "Manufacturer" "TDK" (at 0 0 0) (effects (font (size 1 1)) (hide yes))) (property "MPN" "C1608X5R1C106MT000N" (at 0 0 0) (effects (font (size 1 1)) (hide yes))) (property "JLCPCB" "C342854" (at 0 0 0) (effects (font (size 1 1)) (hide yes))) (property "Datasheet" "https://product.tdk.com/en/search/capacitor/ceramic/mlcc/info?part_no=C1608X5R1C106M080AB" (at 0 0 0) (effects (font (size 1 1)) (hide yes))) (instances (project "virtual-scoring-box" (path "/20cc8167-128c-446a-a106-f942323e143f/97185045-65e6-4b5b-a06d-6bdd67041229" (reference "C22") (unit 1)))))
 (wire (pts (xy 160.02 86.36) (xy 160.02 81.28)) (stroke (width 0) (type default)))
 (global_label "CORE_3V3" (shape bidirectional) (at 160.02 81.28 0) (effects (font (size 0.9 0.9)) (justify left)) (property "Intersheetrefs" "" (at 160.02 81.28 0) (effects (font (size 1 1)) (hide yes))))
@@
 (wire (pts (xy 355.6 74.93) (xy 360.68 74.93)) (stroke (width 0) (type default)))
 (global_label "GND" (shape bidirectional) (at 360.68 74.93 0) (effects (font (size 0.9 0.9)) (justify left)) (property "Intersheetrefs" "" (at 360.68 74.93 0) (effects (font (size 1 1)) (hide yes))))
-(symbol (lib_id "Connector_Generic:Conn_01x06") (at 320.04 129.54 0) (unit 1) (in_bom yes) (on_board yes) (dnp no) (property "Reference" "J6" (at 320.04 115.46 0) (effects (font (size 1.2 1.2)))) (property "Value" "ESP 3.3V UART recovery" (at 320.04 117.46 0) (effects (font (size 1.1 1.1)))) (property "Footprint" "ScoringPlatform:Samtec_HTSW-106-07-L-S" (at 320.04 129.54 0) (effects (font (size 1 1)) (hide yes))) (pin "1") (pin "2") (pin "3") (pin "4") (pin "5") (pin "6") (instances (project "virtual-scoring-box" (path "/20cc8167-128c-446a-a106-f942323e143f/97185045-65e6-4b5b-a06d-6bdd67041229" (reference "J6") (unit 1)))) (property "Datasheet" "https://suddendocs.samtec.com/prints/htsw-xxx-xx-xxx-x-xx-xx-xx-mkt.pdf" (at 0 0 0) (effects (font (size 1 1)) (hide yes))) (property "Manufacturer" "Samtec" (at 0 0 0) (effects (font (size 1 1)) (hide yes))) (property "MPN" "HTSW-106-07-L-S" (at 0 0 0) (effects (font (size 1 1)) (hide yes))))
+(symbol (lib_id "Connector_Generic:Conn_01x06") (at 320.04 129.54 0) (unit 1) (in_bom yes) (on_board yes) (dnp no) (property "Reference" "J6" (at 320.04 115.46 0) (effects (font (size 1.2 1.2)))) (property "Value" "ESP 3.3V UART recovery" (at 320.04 117.46 0) (effects (font (size 1.1 1.1)))) (property "Footprint" "ScoringPlatform:Samtec_HTSW-106-07-L-S" (at 320.04 129.54 0) (effects (font (size 1 1)) (hide yes))) (pin "1") (pin "2") (pin "3") (pin "4") (pin "5") (pin "6") (instances (project "virtual-scoring-box" (path "/20cc8167-128c-446a-a106-f942323e143f/97185045-65e6-4b5b-a06d-6bdd67041229" (reference "J6") (unit 1)))) (property "Datasheet" "https://www.samtec.com/products/htsw-106-07-g-s" (at 0 0 0) (effects (font (size 1 1)) (hide yes))) (property "Manufacturer" "Samtec" (at 0 0 0) (effects (font (size 1 1)) (hide yes))) (property "MPN" "HTSW-106-07-G-S" (at 0 0 0) (effects (font (size 1 1)) (hide yes))) (property "JLCPCB" "C3334125" (at 0 0 0) (effects (font (size 1 1)) (hide yes))))
 (wire (pts (xy 314.96 124.46) (xy 309.88 124.46)) (stroke (width 0) (type default)))
 (global_label "CORE_3V3" (shape bidirectional) (at 309.88 124.46 180) (effects (font (size 0.9 0.9)) (justify right)) (property "Intersheetrefs" "" (at 309.88 124.46 180) (effects (font (size 1 1)) (hide yes))))
