File: packages/scoring-circuit/virtual-scoring-box/isolated-power.kicad_sch (KiCad schematic)
At the start: 15 parts, among them T1 750315371, U21 SN6505BDBVR, U22 TPS62162DSGR

Commit message: fix(scoring-circuit): resolve prototype sourcing gaps
Parts:
- C41, C42, C43, C44, C45, C46: JLCPCB (none) -> C342827; MPN C3216X7R1C106K160AC -> C3216X7R1C106KT000N
