File: packages/scoring-circuit/virtual-scoring-box/usb-interface.kicad_sch (KiCad schematic)
At the start: 17 parts, among them J1 GCT USB4105-GF-A, U18 CP2102N-A02-GQFN20R, U19 ISO7021DR, U20 TPS70933DBVR, U3 TPD2E2U06DCKR

Commit message: fix(scoring-circuit): correct virtual-box assembly part matching
Parts:
- C1, C39: JLCPCB (none) -> C45537494
Changed lines of the file:
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@@
 (global_label "LAPTOP_UART_TX" (shape bidirectional) (at 317.5 77.47 0) (effects (font (size .9 .9)) (justify left)) (property "Intersheetrefs" "" (at 317.5 77.47 0) (effects (font (size 1 1)) (hide yes))))
 (global_label "CORE_3V3" (shape bidirectional) (at 317.5 74.93 0) (effects (font (size .9 .9)) (justify left)) (property "Intersheetrefs" "" (at 317.5 74.93 0) (effects (font (size 1 1)) (hide yes))))
-(symbol (lib_id "Device:C") (at 91.44 144.78 0) (unit 1) (in_bom yes) (on_board yes) (dnp no) (property "Reference" "C1" (at 91.44 139.7 0) (effects (font (size 1 1)))) (property "Value" "1uF" (at 91.44 142.24 0) (effects (font (size 1 1)))) (property "Footprint" "Capacitor_SMD:C_0603_1608Metric" (at 91.44 142.24 0) (effects (font (size 1 1)) (hide yes))) (property "Datasheet" "" (at 91.44 142.24 0) (effects (font (size 1 1)) (hide yes))) (property "MPN" "C1608X7R1H105K080AB" (at 91.44 142.24 0) (effects (font (size 1 1)) (hide yes))) (property "Manufacturer" "TDK" (at 91.44 142.24 0) (effects (font (size 1 1)) (hide yes))) (pin "1") (pin "2") (instances (project "virtual-scoring-box" (path "/20cc8167-128c-446a-a106-f942323e143f/61355932-9259-454d-8754-8e339f213535" (reference "C1") (unit 1)))))
+(symbol (lib_id "Device:C") (at 91.44 144.78 0) (unit 1) (in_bom yes) (on_board yes) (dnp no) (property "Reference" "C1" (at 91.44 139.7 0) (effects (font (size 1 1)))) (property "Value" "1uF" (at 91.44 142.24 0) (effects (font (size 1 1)))) (property "Footprint" "Capacitor_SMD:C_0603_1608Metric" (at 91.44 142.24 0) (effects (font (size 1 1)) (hide yes))) (property "Datasheet" "" (at 91.44 142.24 0) (effects (font (size 1 1)) (hide yes))) (property "MPN" "C1608X7R1H105K080AB" (at 91.44 142.24 0) (effects (font (size 1 1)) (hide yes))) (property "JLCPCB" "C45537494" (at 91.44 142.24 0) (effects (font (size 1 1)) (hide yes))) (property "Manufacturer" "TDK" (at 91.44 142.24 0) (effects (font (size 1 1)) (hide yes))) (pin "1") (pin "2") (instances (project "virtual-scoring-box" (path "/20cc8167-128c-446a-a106-f942323e143f/61355932-9259-454d-8754-8e339f213535" (reference "C1") (unit 1)))))
 (global_label "USB_VBUS" (shape bidirectional) (at 91.44 140.97 0) (effects (font (size .9 .9)) (justify left)) (property "Intersheetrefs" "" (at 91.44 140.97 0) (effects (font (size 1 1)) (hide yes))))
 (global_label "USB_GND" (shape bidirectional) (at 91.44 148.59 0) (effects (font (size .9 .9)) (justify left)) (property "Intersheetrefs" "" (at 91.44 148.59 0) (effects (font (size 1 1)) (hide yes))))
@@
 (global_label "CORE_3V3" (shape bidirectional) (at 335.28 113.03 0) (effects (font (size .9 .9)) (justify left)) (property "Intersheetrefs" "" (at 335.28 113.03 0) (effects (font (size 1 1)) (hide yes))))
 (global_label "GND" (shape bidirectional) (at 335.28 120.65 0) (effects (font (size .9 .9)) (justify left)) (property "Intersheetrefs" "" (at 335.28 120.65 0) (effects (font (size 1 1)) (hide yes))))
-(symbol (lib_id "Device:C") (at 25.4 144.78 0) (unit 1) (in_bom yes) (on_board yes) (dnp no) (property "Reference" "C39" (at 25.4 139.7 0) (effects (font (size 1 1)))) (property "Value" "1uF" (at 25.4 142.24 0) (effects (font (size 1 1)))) (property "Footprint" "Capacitor_SMD:C_0603_1608Metric" (at 25.4 142.24 0) (effects (font (size 1 1)) (hide yes))) (property "Datasheet" "" (at 25.4 142.24 0) (effects (font (size 1 1)) (hide yes))) (property "MPN" "C1608X7R1H105K080AB" (at 25.4 142.24 0) (effects (font (size 1 1)) (hide yes))) (property "Manufacturer" "TDK" (at 25.4 142.24 0) (effects (font (size 1 1)) (hide yes))) (pin "1") (pin "2") (instances (project "virtual-scoring-box" (path "/20cc8167-128c-446a-a106-f942323e143f/61355932-9259-454d-8754-8e339f213535" (reference "C39") (unit 1)))))
+(symbol (lib_id "Device:C") (at 25.4 144.78 0) (unit 1) (in_bom yes) (on_board yes) (dnp no) (property "Reference" "C39" (at 25.4 139.7 0) (effects (font (size 1 1)))) (property "Value" "1uF" (at 25.4 142.24 0) (effects (font (size 1 1)))) (property "Footprint" "Capacitor_SMD:C_0603_1608Metric" (at 25.4 142.24 0) (effects (font (size 1 1)) (hide yes))) (property "Datasheet" "" (at 25.4 142.24 0) (effects (font (size 1 1)) (hide yes))) (property "MPN" "C1608X7R1H105K080AB" (at 25.4 142.24 0) (effects (font (size 1 1)) (hide yes))) (property "JLCPCB" "C45537494" (at 25.4 142.24 0) (effects (font (size 1 1)) (hide yes))) (property "Manufacturer" "TDK" (at 25.4 142.24 0) (effects (font (size 1 1)) (hide yes))) (pin "1") (pin "2") (instances (project "virtual-scoring-box" (path "/20cc8167-128c-446a-a106-f942323e143f/61355932-9259-454d-8754-8e339f213535" (reference "C39") (unit 1)))))
 (global_label "USB_VBUS" (shape bidirectional) (at 25.4 140.97 0) (effects (font (size .9 .9)) (justify left)) (property "Intersheetrefs" "" (at 25.4 140.97 0) (effects (font (size 1 1)) (hide yes))))
 (global_label "USB_GND" (shape bidirectional) (at 25.4 148.59 0) (effects (font (size .9 .9)) (justify left)) (property "Intersheetrefs" "" (at 25.4 148.59 0) (effects (font (size 1 1)) (hide yes))))

Commit message: fix(scoring-circuit): resolve prototype sourcing gaps
Parts:
- C1, C39: JLCPCB C45537494 -> C559769; MPN C1608X7R1H105K080AB -> CC0603KRX7R9BB105; Manufacturer TDK -> YAGEO
Changed lines of the file:
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@@
 (global_label "LAPTOP_UART_TX" (shape bidirectional) (at 317.5 77.47 0) (effects (font (size .9 .9)) (justify left)) (property "Intersheetrefs" "" (at 317.5 77.47 0) (effects (font (size 1 1)) (hide yes))))
 (global_label "CORE_3V3" (shape bidirectional) (at 317.5 74.93 0) (effects (font (size .9 .9)) (justify left)) (property "Intersheetrefs" "" (at 317.5 74.93 0) (effects (font (size 1 1)) (hide yes))))
-(symbol (lib_id "Device:C") (at 91.44 144.78 0) (unit 1) (in_bom yes) (on_board yes) (dnp no) (property "Reference" "C1" (at 91.44 139.7 0) (effects (font (size 1 1)))) (property "Value" "1uF" (at 91.44 142.24 0) (effects (font (size 1 1)))) (property "Footprint" "Capacitor_SMD:C_0603_1608Metric" (at 91.44 142.24 0) (effects (font (size 1 1)) (hide yes))) (property "Datasheet" "" (at 91.44 142.24 0) (effects (font (size 1 1)) (hide yes))) (property "MPN" "C1608X7R1H105K080AB" (at 91.44 142.24 0) (effects (font (size 1 1)) (hide yes))) (property "JLCPCB" "C45537494" (at 91.44 142.24 0) (effects (font (size 1 1)) (hide yes))) (property "Manufacturer" "TDK" (at 91.44 142.24 0) (effects (font (size 1 1)) (hide yes))) (pin "1") (pin "2") (instances (project "virtual-scoring-box" (path "/20cc8167-128c-446a-a106-f942323e143f/61355932-9259-454d-8754-8e339f213535" (reference "C1") (unit 1)))))
+(symbol (lib_id "Device:C") (at 91.44 144.78 0) (unit 1) (in_bom yes) (on_board yes) (dnp no) (property "Reference" "C1" (at 91.44 139.7 0) (effects (font (size 1 1)))) (property "Value" "1uF" (at 91.44 142.24 0) (effects (font (size 1 1)))) (property "Footprint" "Capacitor_SMD:C_0603_1608Metric" (at 91.44 142.24 0) (effects (font (size 1 1)) (hide yes))) (property "Datasheet" "https://yageogroup.com/download/specsheet/CC0603KRX7R9BB105" (at 91.44 142.24 0) (effects (font (size 1 1)) (hide yes))) (property "MPN" "CC0603KRX7R9BB105" (at 91.44 142.24 0) (effects (font (size 1 1)) (hide yes))) (property "JLCPCB" "C559769" (at 91.44 142.24 0) (effects (font (size 1 1)) (hide yes))) (property "Manufacturer" "YAGEO" (at 91.44 142.24 0) (effects (font (size 1 1)) (hide yes))) (pin "1") (pin "2") (instances (project "virtual-scoring-box" (path "/20cc8167-128c-446a-a106-f942323e143f/61355932-9259-454d-8754-8e339f213535" (reference "C1") (unit 1)))))
 (global_label "USB_VBUS" (shape bidirectional) (at 91.44 140.97 0) (effects (font (size .9 .9)) (justify left)) (property "Intersheetrefs" "" (at 91.44 140.97 0) (effects (font (size 1 1)) (hide yes))))
 (global_label "USB_GND" (shape bidirectional) (at 91.44 148.59 0) (effects (font (size .9 .9)) (justify left)) (property "Intersheetrefs" "" (at 91.44 148.59 0) (effects (font (size 1 1)) (hide yes))))
@@
 (global_label "CORE_3V3" (shape bidirectional) (at 335.28 113.03 0) (effects (font (size .9 .9)) (justify left)) (property "Intersheetrefs" "" (at 335.28 113.03 0) (effects (font (size 1 1)) (hide yes))))
 (global_label "GND" (shape bidirectional) (at 335.28 120.65 0) (effects (font (size .9 .9)) (justify left)) (property "Intersheetrefs" "" (at 335.28 120.65 0) (effects (font (size 1 1)) (hide yes))))
-(symbol (lib_id "Device:C") (at 25.4 144.78 0) (unit 1) (in_bom yes) (on_board yes) (dnp no) (property "Reference" "C39" (at 25.4 139.7 0) (effects (font (size 1 1)))) (property "Value" "1uF" (at 25.4 142.24 0) (effects (font (size 1 1)))) (property "Footprint" "Capacitor_SMD:C_0603_1608Metric" (at 25.4 142.24 0) (effects (font (size 1 1)) (hide yes))) (property "Datasheet" "" (at 25.4 142.24 0) (effects (font (size 1 1)) (hide yes))) (property "MPN" "C1608X7R1H105K080AB" (at 25.4 142.24 0) (effects (font (size 1 1)) (hide yes))) (property "JLCPCB" "C45537494" (at 25.4 142.24 0) (effects (font (size 1 1)) (hide yes))) (property "Manufacturer" "TDK" (at 25.4 142.24 0) (effects (font (size 1 1)) (hide yes))) (pin "1") (pin "2") (instances (project "virtual-scoring-box" (path "/20cc8167-128c-446a-a106-f942323e143f/61355932-9259-454d-8754-8e339f213535" (reference "C39") (unit 1)))))
+(symbol (lib_id "Device:C") (at 25.4 144.78 0) (unit 1) (in_bom yes) (on_board yes) (dnp no) (property "Reference" "C39" (at 25.4 139.7 0) (effects (font (size 1 1)))) (property "Value" "1uF" (at 25.4 142.24 0) (effects (font (size 1 1)))) (property "Footprint" "Capacitor_SMD:C_0603_1608Metric" (at 25.4 142.24 0) (effects (font (size 1 1)) (hide yes))) (property "Datasheet" "https://yageogroup.com/download/specsheet/CC0603KRX7R9BB105" (at 25.4 142.24 0) (effects (font (size 1 1)) (hide yes))) (property "MPN" "CC0603KRX7R9BB105" (at 25.4 142.24 0) (effects (font (size 1 1)) (hide yes))) (property "JLCPCB" "C559769" (at 25.4 142.24 0) (effects (font (size 1 1)) (hide yes))) (property "Manufacturer" "YAGEO" (at 25.4 142.24 0) (effects (font (size 1 1)) (hide yes))) (pin "1") (pin "2") (instances (project "virtual-scoring-box" (path "/20cc8167-128c-446a-a106-f942323e143f/61355932-9259-454d-8754-8e339f213535" (reference "C39") (unit 1)))))
 (global_label "USB_VBUS" (shape bidirectional) (at 25.4 140.97 0) (effects (font (size .9 .9)) (justify left)) (property "Intersheetrefs" "" (at 25.4 140.97 0) (effects (font (size 1 1)) (hide yes))))
 (global_label "USB_GND" (shape bidirectional) (at 25.4 148.59 0) (effects (font (size .9 .9)) (justify left)) (property "Intersheetrefs" "" (at 25.4 148.59 0) (effects (font (size 1 1)) (hide yes))))
