File: packages/scoring-circuit/virtual-scoring-box/usb-power-control.kicad_sch (KiCad schematic)
At the start: 32 parts, among them J7 PRIMARY SWD PADS, U23 STUSB4500QTR, U24 STM32C011F6P6, U25 TPS259470ARPWR, U26 SN74LVC1G3208DBVR, U27 SN74LVC1T45DBVR

Commit message: fix(scoring-circuit): correct virtual-box assembly part matching
Parts:
- C49, C50, C52: JLCPCB (none) -> C45537494
- R82, R84: JLCPCB (none) -> C190610; MPN ERA3AEB1002V -> ERA3AEB103V

Commit message: fix(scoring-circuit): source stocked virtual-box signal pullups
Parts:
- R88, R92: JLCPCB (none) -> C144107; MPN RC0603FR-0747KL -> AF0603FR-0747KL
Changed lines of the file:
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@@
 (global_label "USB_HOST_3V3" (shape bidirectional) (at 193.04 34.29 0) (effects (font (size .9 .9)) (justify left)) (property "Intersheetrefs" "" (at 193.04 34.29 0) (effects (font (size 1 1)) (hide yes))))
 (global_label "PD_SDA" (shape bidirectional) (at 193.04 41.91 0) (effects (font (size .9 .9)) (justify left)) (property "Intersheetrefs" "" (at 193.04 41.91 0) (effects (font (size 1 1)) (hide yes))))
-(symbol (lib_id "Device:R") (at 223.52 38.1 0) (unit 1) (in_bom yes) (on_board yes) (dnp no) (property "Reference" "R88" (at 223.52 33.02 0) (effects (font (size 1 1)))) (property "Value" "47k" (at 223.52 35.56 0) (effects (font (size 1 1)))) (property "Footprint" "Resistor_SMD:R_0603_1608Metric" (at 223.52 35.56 0) (effects (font (size 1 1)) (hide yes))) (property "Datasheet" "" (at 223.52 35.56 0) (effects (font (size 1 1)) (hide yes))) (property "MPN" "RC0603FR-0747KL" (at 223.52 35.56 0) (effects (font (size 1 1)) (hide yes))) (property "Manufacturer" "Yageo" (at 223.52 35.56 0) (effects (font (size 1 1)) (hide yes))) (pin "1") (pin "2") (instances (project "virtual-scoring-box" (path "/20cc8167-128c-446a-a106-f942323e143f/60912ca6-e883-4081-9dc0-30579f3da31f" (reference "R88") (unit 1)))))
+(symbol (lib_id "Device:R") (at 223.52 38.1 0) (unit 1) (in_bom yes) (on_board yes) (dnp no) (property "Reference" "R88" (at 223.52 33.02 0) (effects (font (size 1 1)))) (property "Value" "47k" (at 223.52 35.56 0) (effects (font (size 1 1)))) (property "Footprint" "Resistor_SMD:R_0603_1608Metric" (at 223.52 35.56 0) (effects (font (size 1 1)) (hide yes))) (property "Datasheet" "https://yageogroup.com/content/datasheet/asset/file/pyu-af_51_rohs_l" (at 223.52 35.56 0) (effects (font (size 1 1)) (hide yes))) (property "MPN" "AF0603FR-0747KL" (at 223.52 35.56 0) (effects (font (size 1 1)) (hide yes))) (property "Manufacturer" "Yageo" (at 223.52 35.56 0) (effects (font (size 1 1)) (hide yes))) (property "JLCPCB" "C144107" (at 0 0 0) (effects (font (size 1 1)) (hide yes))) (pin "1") (pin "2") (instances (project "virtual-scoring-box" (path "/20cc8167-128c-446a-a106-f942323e143f/60912ca6-e883-4081-9dc0-30579f3da31f" (reference "R88") (unit 1)))))
 (global_label "USB_HOST_3V3" (shape bidirectional) (at 223.52 34.29 0) (effects (font (size .9 .9)) (justify left)) (property "Intersheetrefs" "" (at 223.52 34.29 0) (effects (font (size 1 1)) (hide yes))))
 (global_label "PD_ALERT_N" (shape bidirectional) (at 223.52 41.91 0) (effects (font (size .9 .9)) (justify left)) (property "Intersheetrefs" "" (at 223.52 41.91 0) (effects (font (size 1 1)) (hide yes))))
@@
 (global_label "USB_SUSPEND_EXEMPT" (shape bidirectional) (at 167.64 265.43 0) (effects (font (size .9 .9)) (justify left)) (property "Intersheetrefs" "" (at 167.64 265.43 0) (effects (font (size 1 1)) (hide yes))))
 (global_label "USB_GND" (shape bidirectional) (at 167.64 273.05 0) (effects (font (size .9 .9)) (justify left)) (property "Intersheetrefs" "" (at 167.64 273.05 0) (effects (font (size 1 1)) (hide yes))))
-(symbol (lib_id "Device:R") (at 389.89 132.08 0) (unit 1) (in_bom yes) (on_board yes) (dnp no) (property "Reference" "R92" (at 389.89 127.0 0) (effects (font (size 1 1)))) (property "Value" "47k" (at 389.89 129.54 0) (effects (font (size 1 1)))) (property "Footprint" "Resistor_SMD:R_0603_1608Metric" (at 389.89 129.54 0) (effects (font (size 1 1)) (hide yes))) (property "Datasheet" "" (at 389.89 129.54 0) (effects (font (size 1 1)) (hide yes))) (property "MPN" "RC0603FR-0747KL" (at 389.89 129.54 0) (effects (font (size 1 1)) (hide yes))) (property "Manufacturer" "Yageo" (at 389.89 129.54 0) (effects (font (size 1 1)) (hide yes))) (pin "1") (pin "2") (instances (project "virtual-scoring-box" (path "/20cc8167-128c-446a-a106-f942323e143f/60912ca6-e883-4081-9dc0-30579f3da31f" (reference "R92") (unit 1)))))
+(symbol (lib_id "Device:R") (at 389.89 132.08 0) (unit 1) (in_bom yes) (on_board yes) (dnp no) (property "Reference" "R92" (at 389.89 127.0 0) (effects (font (size 1 1)))) (property "Value" "47k" (at 389.89 129.54 0) (effects (font (size 1 1)))) (property "Footprint" "Resistor_SMD:R_0603_1608Metric" (at 389.89 129.54 0) (effects (font (size 1 1)) (hide yes))) (property "Datasheet" "https://yageogroup.com/content/datasheet/asset/file/pyu-af_51_rohs_l" (at 389.89 129.54 0) (effects (font (size 1 1)) (hide yes))) (property "MPN" "AF0603FR-0747KL" (at 389.89 129.54 0) (effects (font (size 1 1)) (hide yes))) (property "Manufacturer" "Yageo" (at 389.89 129.54 0) (effects (font (size 1 1)) (hide yes))) (property "JLCPCB" "C144107" (at 0 0 0) (effects (font (size 1 1)) (hide yes))) (pin "1") (pin "2") (instances (project "virtual-scoring-box" (path "/20cc8167-128c-446a-a106-f942323e143f/60912ca6-e883-4081-9dc0-30579f3da31f" (reference "R92") (unit 1)))))
 (global_label "USB_HOST_3V3" (shape bidirectional) (at 389.89 128.27 0) (effects (font (size .9 .9)) (justify left)) (property "Intersheetrefs" "" (at 390 128.27 0) (effects (font (size 1 1)) (hide yes))))
 (global_label "FUSE_FAULT_N" (shape bidirectional) (at 389.89 135.89 0) (effects (font (size .9 .9)) (justify left)) (property "Intersheetrefs" "" (at 390 135.89 0) (effects (font (size 1 1)) (hide yes))))

Commit message: fix(scoring-circuit): resolve prototype sourcing gaps
Parts:
- C49, C50, C52: JLCPCB C45537494 -> C559769; MPN C1608X7R1H105K080AB -> CC0603KRX7R9BB105; Manufacturer TDK -> YAGEO
- R81: JLCPCB (none) -> C861245; MPN ERA3AEB2372V -> RT0603BRD0723K7L; Manufacturer Panasonic -> Yageo
- R83: JLCPCB (none) -> C861338; MPN ERA3AEB3482V -> RT0603BRD0734K8L; Manufacturer Panasonic -> Yageo
