File: packages/scoring-circuit/standalone-scoring-box/acquisition-controller.kicad_sch (KiCad schematic)
At the start: 19 parts, among them J2 STM SWD 3.3V, SW1 STM RESET, U1 STM32G474RET6, Y1 ABM3B-8.000MHZ-B2-T

Commit message: fix(scoring-circuit): resolve standalone assembly sourcing matches
Parts:
- C12: LCSC (none) -> C100042; MPN C1608X7R1H103K080AA -> CC0603KRX7R9BB103; Manufacturer TDK -> YAGEO
- C14: LCSC (none) -> C342959; MPN C1608X7S1A475K080AC -> C1608X7S1A475KT000E
- C15, C33: LCSC (none) -> C559769; MPN C1608X7R1H105K080AB -> CC0603KRX7R9BB105; Manufacturer TDK -> YAGEO
- C17, C18: LCSC (none) -> C107045; MPN CGA3E2C0G1H270J080AA -> CC0603JRNPO9BN270; Manufacturer TDK -> YAGEO
- J2: LCSC (none) -> C3337223; MPN HTSW-105-07-L-S -> HTSW-105-07-G-S
