File: packages/scoring-circuit/standalone-scoring-box/application-controller.kicad_sch (KiCad schematic)
At the start: 19 parts, among them J6 ESP 3.3V UART recovery, SW2 ESP RESET, SW3 ESP BOOT, U10 SN74AXC1T45DCKR, U11 SN74AXC1T45DCKR, U2 ESP32-S3-WROOM-1-N8R8

Commit message: feat(scoring-circuit): route standalone HUB75 board
Organize power, ground and signal routing; preserve the isolated boundary and reserve continuous panel power copper. Keep crystals and Ethernet pairs on the top layer. Refine USB and antenna placement and remove dead-end routing.

Verified with KiCad 10.0.6: ERC 0, DRC 0, unconnected 0, schematic parity 0. Inspected native 3D and all four copper layers. pnpm verify passes repository checks and all 969 scoring tests but fails the existing scoring coverage threshold (95.44 statements, 93.78 branches, 99.79 functions, 96.09 lines vs 100). Power qualification, factory NVM handoff and manufacturing review remain open; not order-ready.
Parts:
- U2: footprint RF_Module:ESP32-S3-WROOM-1 -> ScoringPlatform:ESP32-S3-WROOM-1_EdgeMount
Changed lines of the file:
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@@
 (paper "A3")
 (title_block (title "ESP32 display, IR and network controller") (rev "Engineering draft") (comment 1 "NOT FOR FABRICATION"))
-(symbol (lib_id "RF_Module:ESP32-S3-WROOM-1") (at 80.01 100.33 0) (unit 1) (in_bom yes) (on_board yes) (dnp no) (property "Reference" "U2" (at 80.01 63.39 0) (effects (font (size 1.2 1.2)))) (property "Value" "ESP32-S3-WROOM-1-N8R8" (at 80.01 65.39 0) (effects (font (size 1.1 1.1)))) (property "Footprint" "RF_Module:ESP32-S3-WROOM-1" (at 80.01 100.33 0) (effects (font (size 1 1)) (hide yes))) (pin "1") (pin "2") (pin "3") (pin "4") (pin "5") (pin "6") (pin "7") (pin "8") (pin "9") (pin "10") (pin "11") (pin "12") (pin "13") (pin "14") (pin "15") (pin "16") (pin "17") (pin "18") (pin "19") (pin "20") (pin "21") (pin "22") (pin "23") (pin "24") (pin "25") (pin "26") (pin "27") (pin "28") (pin "29") (pin "30") (pin "31") (pin "32") (pin "33") (pin "34") (pin "35") (pin "36") (pin "37") (pin "38") (pin "39") (pin "40") (pin "41") (instances (project "standalone-scoring-box" (path "/95251ad8-e338-4d8f-a50b-ff3c23d840b3/97185045-65e6-4b5b-a06d-6bdd67041229" (reference "U2") (unit 1)))) (property "Manufacturer" "Espressif Systems" (at 0 0 0) (effects (font (size 1 1)) (hide yes))) (property "MPN" "ESP32-S3-WROOM-1-N8R8" (at 0 0 0) (effects (font (size 1 1)) (hide yes))))
+(symbol (lib_id "RF_Module:ESP32-S3-WROOM-1") (at 80.01 100.33 0) (unit 1) (in_bom yes) (on_board yes) (dnp no) (property "Reference" "U2" (at 80.01 63.39 0) (effects (font (size 1.2 1.2)))) (property "Value" "ESP32-S3-WROOM-1-N8R8" (at 80.01 65.39 0) (effects (font (size 1.1 1.1)))) (property "Footprint" "ScoringPlatform:ESP32-S3-WROOM-1_EdgeMount" (at 80.01 100.33 0) (effects (font (size 1 1)) (hide yes))) (pin "1") (pin "2") (pin "3") (pin "4") (pin "5") (pin "6") (pin "7") (pin "8") (pin "9") (pin "10") (pin "11") (pin "12") (pin "13") (pin "14") (pin "15") (pin "16") (pin "17") (pin "18") (pin "19") (pin "20") (pin "21") (pin "22") (pin "23") (pin "24") (pin "25") (pin "26") (pin "27") (pin "28") (pin "29") (pin "30") (pin "31") (pin "32") (pin "33") (pin "34") (pin "35") (pin "36") (pin "37") (pin "38") (pin "39") (pin "40") (pin "41") (instances (project "standalone-scoring-box" (path "/95251ad8-e338-4d8f-a50b-ff3c23d840b3/97185045-65e6-4b5b-a06d-6bdd67041229" (reference "U2") (unit 1)))) (property "Manufacturer" "Espressif Systems" (at 0 0 0) (effects (font (size 1 1)) (hide yes))) (property "MPN" "ESP32-S3-WROOM-1-N8R8" (at 0 0 0) (effects (font (size 1 1)) (hide yes))))
 (wire (pts (xy 80.01 128.27) (xy 80.01 133.35)) (stroke (width 0) (type default)))
 (global_label "GND" (shape bidirectional) (at 80.01 133.35 0) (effects (font (size 0.9 0.9)) (justify left)) (property "Intersheetrefs" "" (at 80.01 133.35 0) (effects (font (size 1 1)) (hide yes))))

Commit message: fix(scoring-circuit): resolve standalone assembly sourcing matches
Parts:
- C21: LCSC (none) -> C559769; MPN C1608X7R1H105K080AB -> CC0603KRX7R9BB105; Manufacturer TDK -> YAGEO
- C22: LCSC (none) -> C342854; MPN C1608X5R1C106M080AB -> C1608X5R1C106MT000N
- J6: LCSC (none) -> C3334125; MPN HTSW-106-07-L-S -> HTSW-106-07-G-S
- R30, R31: LCSC (none) -> C844929; MPN RC0603FR-0747KL -> CRCW060347K0FKEA; Manufacturer YAGEO -> Vishay
