File: packages/scoring-circuit/standalone-scoring-box/ethernet-and-remote.kicad_sch (KiCad schematic)
At the start: 33 parts, among them J13 J1B1211CCD, U12 W5500, U13 TSOP38438, Y2 25MHz CL18pF

Commit message: fix(scoring-circuit): resolve standalone assembly sourcing matches
Parts:
- C28: LCSC (none) -> C342854; MPN C1608X5R1C106M080AB -> C1608X5R1C106MT000N
- C51: LCSC (none) -> C106222; MPN C1608X7R1H223K080AA -> CC0603KRX7R9BB223; Manufacturer TDK -> YAGEO
- C54, C55: LCSC (none) -> C100042; MPN C1608X7R1H103K080AA -> CC0603KRX7R9BB103; Manufacturer TDK -> YAGEO
- C56: LCSC (none) -> C277476; MPN C1608X5R1C475K080AC -> CC0603KRX5R7BB475; Manufacturer TDK -> YAGEO
