File: packages/scoring-circuit/standalone-scoring-box/secondary-power.kicad_sch (KiCad schematic)
At the start: 11 parts, among them J1 GCT USB4105-GF-A, U4 AP2112K-3.3TRG1, U7 AP63203WU-7

Commit message: fix(scoring-circuit): resolve standalone assembly sourcing matches
Parts:
- C1, C2, C3: LCSC (none) -> C559769; MPN C1608X7R1H105K080AB -> CC0603KRX7R9BB105; Manufacturer TDK -> YAGEO
- C5: LCSC (none) -> C342854; MPN C1608X5R1C106M080AB -> C1608X5R1C106MT000N
- J1: LCSC (none) -> C3020560
