File: packages/scoring-circuit/standalone-scoring-box/standalone-scoring-box.kicad_pcb (KiCad board)
At the start: 4 copper layers, 165 x 100 mm, 202 parts, among them J1 GCT USB4105-GF-A, J10 5520250-2, J12 PD service: GND SDA SCL, J13 J1B1211CCD, J2 STM SWD 3.3V, J3 LEFT WEAPON A B C, J4 RIGHT WEAPON A B C, J5 PISTE - NOT protective earth, J6 ESP 3.3V UART recovery, J7 TST-108-02-G-D - HUB75, J8 645004114822 - panel 5V, J9 5520250-2, Q1 DMN2056U-7, Q2 DMN2056U-7, Q3 DMN2056U-7, Q4 DMN2056U-7, Q5 DMN2056U-7, SW1 STM RESET, SW2 ESP RESET, SW3 ESP BOOT, U1 STM32G474RET6, U10 SN74AXC1T45DCKR, U11 SN74AXC1T45DCKR, U12 W5500, U13 TSOP38438, U14 SN74AHCT541PWR, U15 SN74AHCT541PWR, U16 4N32M, U17 4N32M, U2 ESP32-S3-WROOM-1-N8R8, U20 TPS259470LRPWR, U22 TPS70933DBVR, U4 AP2112K-3.3TRG1, U5 STUSB4500QTR, U6 REC30K-2405SZ, U7 AP63203WU-7, U8 74LVC125APW, U9 74LVC125APW, Y1 ABM3B-8.000MHZ-B2-T, Y2 25MHz CL18pF

Commit message: feat(scoring-circuit): route standalone HUB75 board
Organize power, ground and signal routing; preserve the isolated boundary and reserve continuous panel power copper. Keep crystals and Ethernet pairs on the top layer. Refine USB and antenna placement and remove dead-end routing.

Verified with KiCad 10.0.6: ERC 0, DRC 0, unconnected 0, schematic parity 0. Inspected native 3D and all four copper layers. pnpm verify passes repository checks and all 969 scoring tests but fails the existing scoring coverage threshold (95.44 statements, 93.78 branches, 99.79 functions, 96.09 lines vs 100). Power qualification, factory NVM handoff and manufacturing review remain open; not order-ready.
Parts:
- U2: footprint RF_Module:ESP32-S3-WROOM-1 -> ScoringPlatform:ESP32-S3-WROOM-1_EdgeMount
- moved J1 75.7 mm to (49.0, 73.0), turned to -90 degrees
- moved C1 64.7 mm to (58.5, 71.3)
- moved R114 42.1 mm to (53.0, 84.0), turned to 0 degrees
- moved R115 37.0 mm to (56.8, 84.0), turned to 0 degrees
- moved C72 13.2 mm to (61.0, 68.0), turned to 0 degrees
- moved J12 11.5 mm to (51.5, 88.0), turned to 90 degrees
- moved C22 11.5 mm to (134.0, 52.5)
- moved U2 11.5 mm to (146.0, 56.5)
- moved C21 7.30 mm to (132.5, 59.0)
- moved R28 7.30 mm to (130.1, 59.0)
- moved C27 7.15 mm to (134.0, 55.0)
- moved U22 5.39 mm to (57.0, 68.0)
- moved Q4 4.00 mm to (57.0, 77.0)
- moved Q5 4.00 mm to (62.0, 77.0)
- moved R93 3.64 mm to (62.0, 73.5)
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Routing:
- net APP_3V3: track 0.00 -> 362.3 mm, vias 0 -> 13
- net CORE_3V3: track 0.00 -> 360.7 mm, vias 0 -> 52
- net GND: track 0.00 -> 197.0 mm, vias 0 -> 125
- net RIGHT_A: track 0.00 -> 192.1 mm, vias 0 -> 3
- net RIGHT_B: track 0.00 -> 178.0 mm, vias 0 -> 4
- net RIGHT_C: track 0.00 -> 151.8 mm, vias 0 -> 3
- net RIGHT_A_SENSE: track 0.00 -> 130.6 mm, vias 0 -> 12
- net RIGHT_B_SENSE: track 0.00 -> 122.6 mm, vias 0 -> 7
- net PISTE_SENSE: track 0.00 -> 119.9 mm, vias 0 -> 12
- net LEFT_B_SENSE: track 0.00 -> 118.4 mm, vias 0 -> 4
- net PANEL_5V: track 0.00 -> 115.8 mm, vias 0 -> 8
- net FAVERO_TX: track 0.00 -> 112.9 mm, vias 0 -> 2
- net LEFT_A_SENSE: track 0.00 -> 103.5 mm, vias 0 -> 5
- net LEFT_C_SENSE: track 0.00 -> 101.9 mm, vias 0 -> 9
- net SOUNDER_PWM: track 0.00 -> 100.5 mm, vias 0 -> 2
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- added copper zone on In2.Cu, net APP_3V3
- added copper zone on In2.Cu, net CORE_3V3
- added copper zone on In2.Cu, net ETH_AVDD
- added copper zone on B.Cu, net GND
- added copper zone on F.Cu, net GND
- added copper zone on In1.Cu, net GND
- added copper zone on In2.Cu, net GND
- added copper zone on In2.Cu, net PANEL_5V
- added copper zone on B.Cu, net PD_ISO_INPUT
- added copper zone on F.Cu, net PD_ISO_INPUT
- added copper zone on B.Cu, net USB_GND
- added copper zone on F.Cu, net USB_GND
- added copper zone on In1.Cu, net USB_GND
- added copper zone on B.Cu, net USB_VBUS
- added copper zone on F.Cu, net USB_VBUS
Other:
- board text added: "USB-C PD POWER"
- board text removed: "USB HOST / ISOLATION"

Commit message: feat(scoring-circuit): prepare standalone power and assembly handoff
Parts:
- C45: value 10nF 50V -> 1nF 50V C0G 5%
Changed lines of the file:
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@@
 	(title_block
 		(title "Fencing Club standalone scoring box")
-		(rev "Placement draft")
+		(rev "Routed review")
 	)
 	(layers
@@
 			(layer "F.Mask"
 				(type "Top Solder Mask")
-				(color "Black")
+				(color "Green")
 				(thickness 0.01)
 			)
@@
 			(layer "B.Mask"
 				(type "Bottom Solder Mask")
-				(color "Black")
+				(color "Green")
 				(thickness 0.01)
 			)
@@
 		(capping no)
 		(filling no)
+		(aux_axis_origin 45 150)
 		(pcbplotparams
 			(layerselection 0x00000000_00000000_55555555_5755f5ff)
@@
 			(layer "F.Fab")
 		)
+		(fp_text user "${REFERENCE}"
+			(at 0 0 0)
+			(layer "F.Fab")
+			(effects
+				(font
+					(size 0.4 0.4)
+					(thickness 0.06)
+				)
+			)
+		)
 		(pad "" smd roundrect
 			(at -0.25 -0.63)
@@
 			)
 		)
+		(fp_text user "${REFERENCE}"
+			(at 0 5 0)
+			(layer "F.Fab")
+			(effects
+				(font
+					(size 1 1)
+					(thickness 0.15)
+				)
+			)
+		)
 		(pad "" np_thru_hole circle
 			(at -5.08 3.9825)
@@
 			(layer "F.CrtYd")
 		)
+		(fp_text user "${REFERENCE}"
+			(at 0 -3 0)
+			(layer "F.Fab")
+			(effects
+				(font
+					(size 0.8 0.8)
+					(thickness 0.12)
+				)
+			)
+		)
 		(pad "1" thru_hole rect
 			(at -2.54 0 180)
@@
 			(layer "F.CrtYd")
 		)
+		(fp_text user "${REFERENCE}"
+			(at 0 0 0)
+			(layer "F.Fab")
+			(effects
+				(font
+					(size 1 1)
+					(thickness 0.15)
+				)
+			)
+		)
 		(pad "1" thru_hole rect
 			(at -2.5 0)
@@
 			(layer "F.CrtYd")
 		)
+		(fp_text user "${REFERENCE}"
+			(at 0 0 0)
+			(layer "F.Fab")
+			(effects
+				(font
+					(size 0.8 0.8)
+					(thickness 0.12)
+				)
+			)
+		)
 		(pad "1" thru_hole rect
 			(at -3.81 -2.54 90)
@@
 			(layer "F.CrtYd")
 		)
+		(fp_text user "${REFERENCE}"
+			(at 0 0 0)
+			(layer "F.Fab")
+			(effects
+				(font
+					(size 0.8 0.8)
+					(thickness 0.12)
+				)
+			)
+		)
 		(pad "1" thru_hole rect
 			(at -3.81 -2.54 90)
@@
 			)
 		)
-		(property "Value" "10nF 50V"
+		(property "Value" "1nF 50V C0G 5%"
 			(at 0 1.43 0)
 			(layer "F.Fab")
@@
 			)
 		)
-		(property "Datasheet" "https://product.tdk.com/en/search/capacitor/ceramic/mlcc/info?part_no=C1608X7R1H103K080AA"
+		(property "Datasheet" "https://product.tdk.com/en/search/capacitor/ceramic/mlcc/info?part_no=C1608C0G1H102J080AA"
 			(at 0 0 0)
 			(layer "F.Fab")
@@
 			)
 		)
-		(property "MPN" "C1608X7R1H103K080AA"
+		(property "MPN" "C1608C0G1H102J080AA"
 			(at 0 0 0)
 			(layer "F.SilkS")
@@
 			)
 		)
+		(fp_text user "${REFERENCE}"
+			(at 0 0 90)
+			(layer "F.Fab")
+			(effects
+				(font
+					(size 0.65 0.65)
+					(thickness 0.0975)
+				)
+			)
+		)
 		(pad "1" thru_hole rect
 			(at -1.27 -8.89)
@@
 			)
 		)
+		(fp_text user "${REFERENCE}"
+			(at 0 -3 0)
+			(layer "F.Fab")
+			(effects
+				(font
+					(size 0.8 0.8)
+					(thickness 0.12)
+				)
+			)
+		)
 		(pad "1" thru_hole rect
 			(at -5.94 0)
@@
 			(layer "F.Fab")
 		)
+		(fp_text user "${REFERENCE}"
+			(at 0 0 0)
+			(layer "F.Fab")
+			(effects
+				(font
+					(size 1.2 1.2)
+					(thickness 0.18)
+				)
+			)
+		)
 		(pad "1" thru_hole rect
 			(at -10.16 2.54)
@@
 					(thickness 0.15)
 				)
+			)
+		)
+		(fp_text user "${REFERENCE}"
+			(at 0 5 0)
+			(layer "F.Fab")
+			(effects
+				(font
+					(size 1 1)
+					(thickness 0.15)
+				)

Commit message: feat(scoring-circuit): add standalone mounting and assembly draft handoff
Parts:
- added H1: M3 nylon mounting, MountingHole_3.2mm_M3, F.Cu at (49.0, 54.0)
- added H2: M3 nylon mounting, MountingHole_3.2mm_M3, F.Cu at (49.0, 146.0)
- added H3: M3 nylon mounting, MountingHole_3.2mm_M3, F.Cu at (205.0, 146.5)
- added H4: M3 nylon mounting, MountingHole_3.2mm_M3, F.Cu at (182.0, 95.0)
